File: FMC_2.sch (KiCad schematic (older format))
At the start: 16 parts, among them P2 SAMTEC_ASP-134603-01, U44 MIC2090-1YM5TR

Commit message: Convert "~" and "~~" in .sch and .lib files to " "
Parts:
- C10, C11, C12, C13, C5, C6, C7, C8, C9: ComponentHeight ~~ -> (none); PackageDescription ~~ -> (none); PressFit ~~ -> (none); Sense Comment ~~ -> (none); Status Comment ~~ -> (none)
- P2: Case ~~ -> (none); Comment ~~ -> (none); ComponentLink1Description ~~ -> (none); ComponentLink1URL ~~ -> (none); ComponentLink2Description ~~ -> (none); ComponentLink2URL ~~ -> (none); Device ~~ -> (none); PackageDescription ~~ -> (none); SCEM ~~ -> (none); Sense Comment ~~ -> (none); Status Comment ~~ -> (none)
- R205, R258, R259: ComponentHeight ~~ -> (none); PackageDescription ~~ -> (none); Sense Comment ~~ -> (none); Status Comment ~~ -> (none); Voltage ~~ -> (none)

Commit message: Sanitize pin counts in schematics
A lot of them were listed as 2.0000000000000000e+00
Parts:
- C10, C11, C12, C13, C5, C6, C7, C8, C9: Pin Count 2.0000000000000000e+00 -> 2
Changed lines of the file:
@@
 F 9 "Standard" H 7400 4910 60  0001 L CNN "Component Kind"
 F 10 "Standard" H 7400 4820 60  0001 L CNN "Component Type"
-F 11 "2.0000000000000000e+00" H 7400 4640 60  0001 L CNN "Pin Count"
+F 11 "2" H 7400 4640 60  0001 L CNN "Pin Count"
 F 12 "PcbLib\\Capacitors SMD.PcbLib" H 7400 4550 60  0001 L CNN "Footprint Path"
 F 13 "CAPC0603X33N" H 7400 4460 60  0001 L CNN "Footprint Ref"
@@
 F 9 "Standard" H 3000 4460 60  0001 L CNN "Component Kind"
 F 10 "Standard" H 3000 4370 60  0001 L CNN "Component Type"
-F 11 "2.0000000000000000e+00" H 3000 4190 60  0001 L CNN "Pin Count"
+F 11 "2" H 3000 4190 60  0001 L CNN "Pin Count"
 F 12 "PcbLib\\Capacitors SMD.PcbLib" H 3000 4100 60  0001 L CNN "Footprint Path"
 F 13 "CAPC3216X140N" H 3000 4010 60  0001 L CNN "Footprint Ref"
@@
 F 9 "Standard" H 4700 5110 60  0001 L CNN "Component Kind"
 F 10 "Standard" H 4700 5020 60  0001 L CNN "Component Type"
-F 11 "2.0000000000000000e+00" H 4700 4840 60  0001 L CNN "Pin Count"
+F 11 "2" H 4700 4840 60  0001 L CNN "Pin Count"
 F 12 "PcbLib\\Capacitors SMD.PcbLib" H 4700 4750 60  0001 L CNN "Footprint Path"
 F 13 "CAPC0603X33N" H 4700 4660 60  0001 L CNN "Footprint Ref"
@@
 F 9 "Standard" H 8300 5210 60  0001 L CNN "Component Kind"
 F 10 "Standard" H 8300 5120 60  0001 L CNN "Component Type"
-F 11 "2.0000000000000000e+00" H 8300 4940 60  0001 L CNN "Pin Count"
+F 11 "2" H 8300 4940 60  0001 L CNN "Pin Count"
 F 12 "PcbLib\\Capacitors SMD.PcbLib" H 8300 4850 60  0001 L CNN "Footprint Path"
 F 13 "CAPC1608X87N" H 8300 4760 60  0001 L CNN "Footprint Ref"
@@
 F 9 "Standard" H 2500 4460 60  0001 L CNN "Component Kind"
 F 10 "Standard" H 2500 4370 60  0001 L CNN "Component Type"
-F 11 "2.0000000000000000e+00" H 2500 4190 60  0001 L CNN "Pin Count"
+F 11 "2" H 2500 4190 60  0001 L CNN "Pin Count"
 F 12 "PcbLib\\Capacitors SMD.PcbLib" H 2500 4100 60  0001 L CNN "Footprint Path"
 F 13 "CAPC1005X55N" H 2500 4010 60  0001 L CNN "Footprint Ref"
@@
 F 9 "Standard" H 5150 5110 60  0001 L CNN "Component Kind"
 F 10 "Standard" H 5150 5020 60  0001 L CNN "Component Type"
-F 11 "2.0000000000000000e+00" H 5150 4840 60  0001 L CNN "Pin Count"
+F 11 "2" H 5150 4840 60  0001 L CNN "Pin Count"
 F 12 "PcbLib\\Capacitors SMD.PcbLib" H 5150 4750 60  0001 L CNN "Footprint Path"
 F 13 "CAPC0603X33N" H 5150 4660 60  0001 L CNN "Footprint Ref"
@@
 F 9 "Standard" H 5950 6010 60  0001 L CNN "Component Kind"
 F 10 "Standard" H 5950 5920 60  0001 L CNN "Component Type"
-F 11 "2.0000000000000000e+00" H 5950 5740 60  0001 L CNN "Pin Count"
+F 11 "2" H 5950 5740 60  0001 L CNN "Pin Count"
 F 12 "PcbLib\\Capacitors SMD.PcbLib" H 5950 5650 60  0001 L CNN "Footprint Path"
 F 13 "CAPC0603X33N" H 5950 5560 60  0001 L CNN "Footprint Ref"
@@
 F 9 "Standard" H 6400 6010 60  0001 L CNN "Component Kind"
 F 10 "Standard" H 6400 5920 60  0001 L CNN "Component Type"
-F 11 "2.0000000000000000e+00" H 6400 5740 60  0001 L CNN "Pin Count"
+F 11 "2" H 6400 5740 60  0001 L CNN "Pin Count"
 F 12 "PcbLib\\Capacitors SMD.PcbLib" H 6400 5650 60  0001 L CNN "Footprint Path"
 F 13 "CAPC0603X33N" H 6400 5560 60  0001 L CNN "Footprint Ref"
@@
 F 9 "Standard" H 7900 5210 60  0001 L CNN "Component Kind"
 F 10 "Standard" H 7900 5120 60  0001 L CNN "Component Type"
-F 11 "2.0000000000000000e+00" H 7900 4940 60  0001 L CNN "Pin Count"
+F 11 "2" H 7900 4940 60  0001 L CNN "Pin Count"
 F 12 "PcbLib\\Capacitors SMD.PcbLib" H 7900 4850 60  0001 L CNN "Footprint Path"
 F 13 "CAPC1608X87N" H 7900 4760 60  0001 L CNN "Footprint Ref"

Commit message: Trash HelpURL ComponentLink1URL ComponentLink2URL attributes
Removes 1056 useless and library-mismatched attributes
Parts:
- C10, C11, C7, C8, C9: HelpURL \\\\cern.ch\\dfs\\Applications\\Altium\\Datasheets\\CC0201_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 -> (none)
- C12, C13: HelpURL \\\\cern.ch\\dfs\\Applications\\Altium\\Datasheets\\CC0603_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 -> (none)
- C5: HelpURL \\\\cern.ch\\dfs\\Applications\\Altium\\Datasheets\\CC0402_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 -> (none)
- C6: HelpURL \\\\cern.ch\\dfs\\Applications\\Altium\\Datasheets\\CC1206_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 -> (none)
- P2: ComponentLink1URL (none) -> (none); ComponentLink2URL (none) -> (none); HelpURL \\\\cern.ch\\dfs\\Applications\\Altium\\Datasheets\\SAMTEC_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 -> (none)
- R205, R258, R259: HelpURL \\\\cern.ch\\dfs\\Applications\\Altium\\Datasheets\\R0402_P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 -> (none)
Changed lines of the file:
@@
 F 33 "232270671003L" H 10650 -1680 60  0001 L CNN "Manufacturer1 Part Number"
 F 34 "0.4mm" H 10650 -1770 60  0001 L CNN "Manufacturer1 ComponentHeight"
-F 35 "\\\\cern.ch\\dfs\\Applications\\Altium\\Datasheets\\R0402_Phycomp_RC0402.pdf" H 10650 -1860 60  0001 L CNN "HelpURL"
 F 36 "CERN DEM JLC" H 10650 -1950 60  0001 L CNN "Author"
 F 37 "12/03/07 00:00:00" H 10650 -2040 60  0001 L CNN "CreateDate"
@@
 F 32 "02016D104KAT2A" H 7400 2660 60  0001 L CNN "Manufacturer1 Part Number"
 F 33 "0.33mm" H 7400 2570 60  0001 L CNN "Manufacturer1 ComponentHeight"
-F 34 "\\\\cern.ch\\dfs\\Applications\\Altium\\Datasheets\\CC0201_X5R_AVX.pdf" H 7400 2480 60  0001 L CNN "HelpURL"
 F 35 "CERN DEM JLC" H 7400 2390 60  0001 L CNN "Author"
 F 36 "12/03/07 00:00:00" H 7400 2300 60  0001 L CNN "CreateDate"
@@
 F 32 "C1206C106K4RAC" H 3000 2210 60  0001 L CNN "Manufacturer1 Part Number"
 F 33 "1.8mm" H 3000 2120 60  0001 L CNN "Manufacturer1 ComponentHeight"
-F 34 "\\\\cern.ch\\dfs\\Applications\\Altium\\Datasheets\\CC1206_X7R_KEMET.pdf" H 3000 2030 60  0001 L CNN "HelpURL"
 F 35 "CERN DEM JLC" H 3000 1940 60  0001 L CNN "Author"
 F 36 "04/28/09 00:00:00" H 3000 1850 60  0001 L CNN "CreateDate"
@@
 F 32 "02016D104KAT2A" H 4700 2860 60  0001 L CNN "Manufacturer1 Part Number"
 F 33 "0.33mm" H 4700 2770 60  0001 L CNN "Manufacturer1 ComponentHeight"
-F 34 "\\\\cern.ch\\dfs\\Applications\\Altium\\Datasheets\\CC0201_X5R_AVX.pdf" H 4700 2680 60  0001 L CNN "HelpURL"
 F 35 "CERN DEM JLC" H 4700 2590 60  0001 L CNN "Author"
 F 36 "12/03/07 00:00:00" H 4700 2500 60  0001 L CNN "CreateDate"
@@
 F 32 "C0603C106M9PAC" H 8300 2960 60  0001 L CNN "Manufacturer1 Part Number"
 F 33 "0.95mm" H 8300 2870 60  0001 L CNN "Manufacturer1 ComponentHeight"
-F 34 "\\\\cern.ch\\dfs\\Applications\\Altium\\Datasheets\\CC0603_X5R_KEMET.pdf" H 8300 2780 60  0001 L CNN "HelpURL"
 F 35 "CERN DEM JLC" H 8300 2690 60  0001 L CNN "Author"
 F 36 "12/03/07 00:00:00" H 8300 2600 60  0001 L CNN "CreateDate"
@@
 F 32 "GRM155R61C104KA88D" H 2500 2210 60  0001 L CNN "Manufacturer1 Part Number"
 F 33 "0.55mm" H 2500 2120 60  0001 L CNN "Manufacturer1 ComponentHeight"
-F 34 "\\\\cern.ch\\dfs\\Applications\\Altium\\Datasheets\\CC0402_X5R_MURATA_GRM.pdf" H 2500 2030 60  0001 L CNN "HelpURL"
 F 35 "CERN DEM JLC" H 2500 1940 60  0001 L CNN "Author"
 F 36 "12/10/13 00:00:00" H 2500 1850 60  0001 L CNN "CreateDate"
@@
 F 29 "ASP-134603-01" H 4050 -4860 60  0001 L CNN "Manufacturer Part Number"
 F 30 "6.55mm" H 4050 -4950 60  0001 L CNN "ComponentHeight"
-F 31 "\\\\cern.ch\\dfs\\Applications\\Altium\\Datasheets\\SAMTEC_ASP-134603-01.pdf" H 4050 -5040 60  0001 L CNN "HelpURL"
-F 32 " " H 4050 -5130 60  0001 L CNN "ComponentLink1URL"
 F 33 " " H 4050 -5220 60  0001 L CNN "ComponentLink1Description"
-F 34 " " H 4050 -5310 60  0001 L CNN "ComponentLink2URL"
 F 35 " " H 4050 -5400 60  0001 L CNN "ComponentLink2Description"
 F 36 "CERN DEM JLC" H 4050 -5490 60  0001 L CNN "Author"
@@
 F 29 "ASP-134603-01" H 6350 -4860 60  0001 L CNN "Manufacturer Part Number"
 F 30 "6.55mm" H 6350 -4950 60  0001 L CNN "ComponentHeight"
-F 31 "\\\\cern.ch\\dfs\\Applications\\Altium\\Datasheets\\SAMTEC_ASP-134603-01.pdf" H 6350 -5040 60  0001 L CNN "HelpURL"
-F 32 " " H 6350 -5130 60  0001 L CNN "ComponentLink1URL"
 F 33 " " H 6350 -5220 60  0001 L CNN "ComponentLink1Description"
-F 34 " " H 6350 -5310 60  0001 L CNN "ComponentLink2URL"
 F 35 " " H 6350 -5400 60  0001 L CNN "ComponentLink2Description"
 F 36 "CERN DEM JLC" H 6350 -5490 60  0001 L CNN "Author"
@@
 F 29 "ASP-134603-01" H 9100 -4860 60  0001 L CNN "Manufacturer Part Number"
 F 30 "6.55mm" H 9100 -4950 60  0001 L CNN "ComponentHeight"
-F 31 "\\\\cern.ch\\dfs\\Applications\\Altium\\Datasheets\\SAMTEC_ASP-134603-01.pdf" H 9100 -5040 60  0001 L CNN "HelpURL"
-F 32 " " H 9100 -5130 60  0001 L CNN "ComponentLink1URL"
 F 33 " " H 9100 -5220 60  0001 L CNN "ComponentLink1Description"
-F 34 " " H 9100 -5310 60  0001 L CNN "ComponentLink2URL"
 F 35 " " H 9100 -5400 60  0001 L CNN "ComponentLink2Description"
 F 36 "CERN DEM JLC" H 9100 -5490 60  0001 L CNN "Author"
@@
 F 29 "ASP-134603-01" H 11750 -4860 60  0001 L CNN "Manufacturer Part Number"
 F 30 "6.55mm" H 11750 -4950 60  0001 L CNN "ComponentHeight"
-F 31 "\\\\cern.ch\\dfs\\Applications\\Altium\\Datasheets\\SAMTEC_ASP-134603-01.pdf" H 11750 -5040 60  0001 L CNN "HelpURL"
-F 32 " " H 11750 -5130 60  0001 L CNN "ComponentLink1URL"
 F 33 " " H 11750 -5220 60  0001 L CNN "ComponentLink1Description"
-F 34 " " H 11750 -5310 60  0001 L CNN "ComponentLink2URL"
 F 35 " " H 11750 -5400 60  0001 L CNN "ComponentLink2Description"
 F 36 "CERN DEM JLC" H 11750 -5490 60  0001 L CNN "Author"
@@
 F 33 "232270671003L" H 8400 3720 60  0001 L CNN "Manufacturer1 Part Number"
 F 34 "0.4mm" H 8400 3630 60  0001 L CNN "Manufacturer1 ComponentHeight"
-F 35 "\\\\cern.ch\\dfs\\Applications\\Altium\\Datasheets\\R0402_Phycomp_RC0402.pdf" H 8400 3540 60  0001 L CNN "HelpURL"
 F 36 "CERN DEM JLC" H 8400 3450 60  0001 L CNN "Author"
 F 37 "12/03/07 00:00:00" H 8400 3360 60  0001 L CNN "CreateDate"
@@
 F 33 "232270671002L" H 8250 3870 60  0001 L CNN "Manufacturer1 Part Number"
 F 34 "0.4mm" H 8250 3780 60  0001 L CNN "Manufacturer1 ComponentHeight"
-F 35 "\\\\cern.ch\\dfs\\Applications\\Altium\\Datasheets\\R0402_Phycomp_RC0402.pdf" H 8250 3690 60  0001 L CNN "HelpURL"
 F 36 "CERN DEM JLC" H 8250 3600 60  0001 L CNN "Author"
 F 37 "12/03/07 00:00:00" H 8250 3510 60  0001 L CNN "CreateDate"
@@
 F 32 "02016D104KAT2A" H 5150 2860 60  0001 L CNN "Manufacturer1 Part Number"
 F 33 "0.33mm" H 5150 2770 60  0001 L CNN "Manufacturer1 ComponentHeight"
-F 34 "\\\\cern.ch\\dfs\\Applications\\Altium\\Datasheets\\CC0201_X5R_AVX.pdf" H 5150 2680 60  0001 L CNN "HelpURL"
 F 35 "CERN DEM JLC" H 5150 2590 60  0001 L CNN "Author"
 F 36 "12/03/07 00:00:00" H 5150 2500 60  0001 L CNN "CreateDate"
@@
 F 32 "02016D104KAT2A" H 5950 3760 60  0001 L CNN "Manufacturer1 Part Number"
 F 33 "0.33mm" H 5950 3670 60  0001 L CNN "Manufacturer1 ComponentHeight"
-F 34 "\\\\cern.ch\\dfs\\Applications\\Altium\\Datasheets\\CC0201_X5R_AVX.pdf" H 5950 3580 60  0001 L CNN "HelpURL"
 F 35 "CERN DEM JLC" H 5950 3490 60  0001 L CNN "Author"
 F 36 "12/03/07 00:00:00" H 5950 3400 60  0001 L CNN "CreateDate"
@@
 F 32 "02016D104KAT2A" H 6400 3760 60  0001 L CNN "Manufacturer1 Part Number"
 F 33 "0.33mm" H 6400 3670 60  0001 L CNN "Manufacturer1 ComponentHeight"
-F 34 "\\\\cern.ch\\dfs\\Applications\\Altium\\Datasheets\\CC0201_X5R_AVX.pdf" H 6400 3580 60  0001 L CNN "HelpURL"
 F 35 "CERN DEM JLC" H 6400 3490 60  0001 L CNN "Author"
 F 36 "12/03/07 00:00:00" H 6400 3400 60  0001 L CNN "CreateDate"
@@
 F 32 "C0603C106M9PAC" H 7900 2960 60  0001 L CNN "Manufacturer1 Part Number"
 F 33 "0.95mm" H 7900 2870 60  0001 L CNN "Manufacturer1 ComponentHeight"
-F 34 "\\\\cern.ch\\dfs\\Applications\\Altium\\Datasheets\\CC0603_X5R_KEMET.pdf" H 7900 2780 60  0001 L CNN "HelpURL"
 F 35 "CERN DEM JLC" H 7900 2690 60  0001 L CNN "Author"
 F 36 "12/03/07 00:00:00" H 7900 2600 60  0001 L CNN "CreateDate"

Commit message: Trash "Footprint Library" and "Database Table Name" attributes
Takes 100 attributes out of schematic, 174 out of library
Parts:
- R299, R300: Database Table Name Resistors SMD -> (none); Footprint Library Resistors SMD -> (none)
Changed lines of the file:
@@
 F 36 "12/03/07 00:00:00" H 3100 2505 50  0001 L CNN "CreateDate"
 F 37 "10/17/12 00:00:00" H 3100 2430 50  0001 L CNN "LatestRevisionDate"
-F 38 "Resistors SMD" H 3100 2355 50  0001 L CNN "Database Table Name"
 F 39 "Resistors SMD" H 3100 2280 50  0001 L CNN "Library Name"
-F 40 "Resistors SMD" H 3100 2205 50  0001 L CNN "Footprint Library"
 F 41 "This work is licensed under the Creative Commons CC-BY-SA 4.0 License. To the extent that circuit schematics that use Licensed Material can be considered to be ‘Adapted Material’, then the copyright holder waives article 3.b of the license with respect to these schematics." H 3100 2130 50  0001 L CNN "License"
 	1    3100 5250
@@
 F 36 "12/03/07 00:00:00" H 5150 2605 50  0001 L CNN "CreateDate"
 F 37 "10/17/12 00:00:00" H 5150 2530 50  0001 L CNN "LatestRevisionDate"
-F 38 "Resistors SMD" H 5150 2455 50  0001 L CNN "Database Table Name"
 F 39 "Resistors SMD" H 5150 2380 50  0001 L CNN "Library Name"
-F 40 "Resistors SMD" H 5150 2305 50  0001 L CNN "Footprint Library"
 F 41 "This work is licensed under the Creative Commons CC-BY-SA 4.0 License. To the extent that circuit schematics that use Licensed Material can be considered to be ‘Adapted Material’, then the copyright holder waives article 3.b of the license with respect to these schematics." H 5150 2230 50  0001 L CNN "License"
 	1    5150 5350

Commit message: Trash SCEM attribute
Parts:
- P2: SCEM (none) -> (none)
Changed lines of the file:
@@
 F 24 " " H 4050 -4410 60  0001 L CNN "Status Comment"
 F 25 "None" H 4050 -4500 60  0001 L CNN "Status"
-F 26 " " H 4050 -4590 60  0001 L CNN "SCEM"
 F 27 "160 contacts (4 rows cdgh) Surface Mount Female Connector, VITA 57 (CC-LPC-10)" H 4050 -4680 60  0001 L CNN "Part Description"
 F 28 "SAMTEC" H 4050 -4770 60  0001 L CNN "Manufacturer"
@@
 F 24 " " H 6350 -4410 60  0001 L CNN "Status Comment"
 F 25 "None" H 6350 -4500 60  0001 L CNN "Status"
-F 26 " " H 6350 -4590 60  0001 L CNN "SCEM"
 F 27 "160 contacts (4 rows cdgh) Surface Mount Female Connector, VITA 57 (CC-LPC-10)" H 6350 -4680 60  0001 L CNN "Part Description"
 F 28 "SAMTEC" H 6350 -4770 60  0001 L CNN "Manufacturer"
@@
 F 24 " " H 9100 -4410 60  0001 L CNN "Status Comment"
 F 25 "None" H 9100 -4500 60  0001 L CNN "Status"
-F 26 " " H 9100 -4590 60  0001 L CNN "SCEM"
 F 27 "160 contacts (4 rows cdgh) Surface Mount Female Connector, VITA 57 (CC-LPC-10)" H 9100 -4680 60  0001 L CNN "Part Description"
 F 28 "SAMTEC" H 9100 -4770 60  0001 L CNN "Manufacturer"
@@
 F 24 " " H 11750 -4410 60  0001 L CNN "Status Comment"
 F 25 "None" H 11750 -4500 60  0001 L CNN "Status"
-F 26 " " H 11750 -4590 60  0001 L CNN "SCEM"
 F 27 "160 contacts (4 rows cdgh) Surface Mount Female Connector, VITA 57 (CC-LPC-10)" H 11750 -4680 60  0001 L CNN "Part Description"
 F 28 "SAMTEC" H 11750 -4770 60  0001 L CNN "Manufacturer"

Commit message: Touch up a few symbols and instances
Add attribute names to MIC2090
Fix spelling error in XRP7724 description
Remove stray AMC_FMC_Carrier-PcbDoc-cache.lib
Parts:
- U44: Case (none) -> SOT-23-5; Field4 MIC2090-1YM5TR -> (none); Field6 SOT-23-5 -> (none); Field7 MICREL SEMICONDUCTOR -> (none); Manufacturer (none) -> MICREL SEMICONDUCTOR; Part Number (none) -> MIC2090-1YM5TR
Changed lines of the file:
@@
 F 2 "ICs And Semiconductors SMD:SOT95P280X145-5N" H 7550 6500 50  0001 L BNN
 F 3 "58T4896" H 7550 6200 50  0001 L BNN
-F 4 "MIC2090-1YM5TR" H 7550 6400 50  0001 L BNN "Field4"
+F 4 "MIC2090-1YM5TR" H 7550 6400 50  0001 L BNN "Part Number"
 F 5 "1924707" H 7550 6100 50  0001 L BNN "Field5"
-F 6 "SOT-23-5" H 7550 6300 50  0001 L BNN "Field6"
-F 7 "MICREL SEMICONDUCTOR" H 7550 6600 50  0001 L BNN "Field7"
+F 6 "SOT-23-5" H 7550 6300 50  0001 L BNN "Case"
+F 7 "MICREL SEMICONDUCTOR" H 7550 6600 50  0001 L BNN "Manufacturer"
 	1    7550 7100
 	-1   0    0    -1
