File: FMC_1.sch (KiCad schematic (older format))
At the start: 16 parts, among them P1 SAMTEC_ASP-134603-01, U45 MIC2090-1YM5TR

Commit message: Convert "~" and "~~" in .sch and .lib files to " "
Parts:
- C61, C62, C63, C64, C65, C66, C67, C68, C69: ComponentHeight ~~ -> (none); PackageDescription ~~ -> (none); PressFit ~~ -> (none); Sense Comment ~~ -> (none); Status Comment ~~ -> (none)
- P1: Case ~~ -> (none); Comment ~~ -> (none); ComponentLink1Description ~~ -> (none); ComponentLink1URL ~~ -> (none); ComponentLink2Description ~~ -> (none); ComponentLink2URL ~~ -> (none); Device ~~ -> (none); PackageDescription ~~ -> (none); SCEM ~~ -> (none); Sense Comment ~~ -> (none); Status Comment ~~ -> (none)
- R234, R260, R261: ComponentHeight ~~ -> (none); PackageDescription ~~ -> (none); Sense Comment ~~ -> (none); Status Comment ~~ -> (none); Voltage ~~ -> (none)

Commit message: Sanitize pin counts in schematics
A lot of them were listed as 2.0000000000000000e+00
Parts:
- C61, C62, C63, C64, C65, C66, C67, C68, C69: Pin Count 2.0000000000000000e+00 -> 2
Changed lines of the file:
@@
 F 9 "Standard" H 7600 4910 60  0001 L CNN "Component Kind"
 F 10 "Standard" H 7600 4820 60  0001 L CNN "Component Type"
-F 11 "2.0000000000000000e+00" H 7600 4640 60  0001 L CNN "Pin Count"
+F 11 "2" H 7600 4640 60  0001 L CNN "Pin Count"
 F 12 "PcbLib\\Capacitors SMD.PcbLib" H 7600 4550 60  0001 L CNN "Footprint Path"
 F 13 "CAPC1608X87N" H 7600 4460 60  0001 L CNN "Footprint Ref"
@@
 F 9 "Standard" H 7100 4610 60  0001 L CNN "Component Kind"
 F 10 "Standard" H 7100 4520 60  0001 L CNN "Component Type"
-F 11 "2.0000000000000000e+00" H 7100 4340 60  0001 L CNN "Pin Count"
+F 11 "2" H 7100 4340 60  0001 L CNN "Pin Count"
 F 12 "PcbLib\\Capacitors SMD.PcbLib" H 7100 4250 60  0001 L CNN "Footprint Path"
 F 13 "CAPC0603X33N" H 7100 4160 60  0001 L CNN "Footprint Ref"
@@
 F 9 "Standard" H 8000 4910 60  0001 L CNN "Component Kind"
 F 10 "Standard" H 8000 4820 60  0001 L CNN "Component Type"
-F 11 "2.0000000000000000e+00" H 8000 4640 60  0001 L CNN "Pin Count"
+F 11 "2" H 8000 4640 60  0001 L CNN "Pin Count"
 F 12 "PcbLib\\Capacitors SMD.PcbLib" H 8000 4550 60  0001 L CNN "Footprint Path"
 F 13 "CAPC1608X87N" H 8000 4460 60  0001 L CNN "Footprint Ref"
@@
 F 9 "Standard" H 5650 5710 60  0001 L CNN "Component Kind"
 F 10 "Standard" H 5650 5620 60  0001 L CNN "Component Type"
-F 11 "2.0000000000000000e+00" H 5650 5440 60  0001 L CNN "Pin Count"
+F 11 "2" H 5650 5440 60  0001 L CNN "Pin Count"
 F 12 "PcbLib\\Capacitors SMD.PcbLib" H 5650 5350 60  0001 L CNN "Footprint Path"
 F 13 "CAPC0603X33N" H 5650 5260 60  0001 L CNN "Footprint Ref"
@@
 F 9 "Standard" H 6100 5710 60  0001 L CNN "Component Kind"
 F 10 "Standard" H 6100 5620 60  0001 L CNN "Component Type"
-F 11 "2.0000000000000000e+00" H 6100 5440 60  0001 L CNN "Pin Count"
+F 11 "2" H 6100 5440 60  0001 L CNN "Pin Count"
 F 12 "PcbLib\\Capacitors SMD.PcbLib" H 6100 5350 60  0001 L CNN "Footprint Path"
 F 13 "CAPC0603X33N" H 6100 5260 60  0001 L CNN "Footprint Ref"
@@
 F 9 "Standard" H 4400 4810 60  0001 L CNN "Component Kind"
 F 10 "Standard" H 4400 4720 60  0001 L CNN "Component Type"
-F 11 "2.0000000000000000e+00" H 4400 4540 60  0001 L CNN "Pin Count"
+F 11 "2" H 4400 4540 60  0001 L CNN "Pin Count"
 F 12 "PcbLib\\Capacitors SMD.PcbLib" H 4400 4450 60  0001 L CNN "Footprint Path"
 F 13 "CAPC0603X33N" H 4400 4360 60  0001 L CNN "Footprint Ref"
@@
 F 9 "Standard" H 4850 4810 60  0001 L CNN "Component Kind"
 F 10 "Standard" H 4850 4720 60  0001 L CNN "Component Type"
-F 11 "2.0000000000000000e+00" H 4850 4540 60  0001 L CNN "Pin Count"
+F 11 "2" H 4850 4540 60  0001 L CNN "Pin Count"
 F 12 "PcbLib\\Capacitors SMD.PcbLib" H 4850 4450 60  0001 L CNN "Footprint Path"
 F 13 "CAPC0603X33N" H 4850 4360 60  0001 L CNN "Footprint Ref"
@@
 F 9 "Standard" H 2700 4160 60  0001 L CNN "Component Kind"
 F 10 "Standard" H 2700 4070 60  0001 L CNN "Component Type"
-F 11 "2.0000000000000000e+00" H 2700 3890 60  0001 L CNN "Pin Count"
+F 11 "2" H 2700 3890 60  0001 L CNN "Pin Count"
 F 12 "PcbLib\\Capacitors SMD.PcbLib" H 2700 3800 60  0001 L CNN "Footprint Path"
 F 13 "CAPC3216X140N" H 2700 3710 60  0001 L CNN "Footprint Ref"
@@
 F 9 "Standard" H 2200 4160 60  0001 L CNN "Component Kind"
 F 10 "Standard" H 2200 4070 60  0001 L CNN "Component Type"
-F 11 "2.0000000000000000e+00" H 2200 3890 60  0001 L CNN "Pin Count"
+F 11 "2" H 2200 3890 60  0001 L CNN "Pin Count"
 F 12 "PcbLib\\Capacitors SMD.PcbLib" H 2200 3800 60  0001 L CNN "Footprint Path"
 F 13 "CAPC1005X55N" H 2200 3710 60  0001 L CNN "Footprint Ref"

Commit message: Trash HelpURL ComponentLink1URL ComponentLink2URL attributes
Removes 1056 useless and library-mismatched attributes
Parts:
- C61: HelpURL \\\\cern.ch\\dfs\\Applications\\Altium\\Datasheets\\CC0402_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 -> (none)
- C62: HelpURL \\\\cern.ch\\dfs\\Applications\\Altium\\Datasheets\\CC1206_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 -> (none)
- C63, C64, C65, C66, C67: HelpURL \\\\cern.ch\\dfs\\Applications\\Altium\\Datasheets\\CC0201_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 -> (none)
- C68, C69: HelpURL \\\\cern.ch\\dfs\\Applications\\Altium\\Datasheets\\CC0603_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 -> (none)
- P1: ComponentLink1URL (none) -> (none); ComponentLink2URL (none) -> (none); HelpURL \\\\cern.ch\\dfs\\Applications\\Altium\\Datasheets\\SAMTEC_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 -> (none)
- R234, R260, R261: HelpURL \\\\cern.ch\\dfs\\Applications\\Altium\\Datasheets\\R0402_P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 -> (none)
Changed lines of the file:
@@
 F 33 "232270671003L" H 10350 -1980 60  0001 L CNN "Manufacturer1 Part Number"
 F 34 "0.4mm" H 10350 -2070 60  0001 L CNN "Manufacturer1 ComponentHeight"
-F 35 "\\\\cern.ch\\dfs\\Applications\\Altium\\Datasheets\\R0402_Phycomp_RC0402.pdf" H 10350 -2160 60  0001 L CNN "HelpURL"
 F 36 "CERN DEM JLC" H 10350 -2250 60  0001 L CNN "Author"
 F 37 "12/03/07 00:00:00" H 10350 -2340 60  0001 L CNN "CreateDate"
@@
 F 32 "C0603C106M9PAC" H 7600 2660 60  0001 L CNN "Manufacturer1 Part Number"
 F 33 "0.95mm" H 7600 2570 60  0001 L CNN "Manufacturer1 ComponentHeight"
-F 34 "\\\\cern.ch\\dfs\\Applications\\Altium\\Datasheets\\CC0603_X5R_KEMET.pdf" H 7600 2480 60  0001 L CNN "HelpURL"
 F 35 "CERN DEM JLC" H 7600 2390 60  0001 L CNN "Author"
 F 36 "12/03/07 00:00:00" H 7600 2300 60  0001 L CNN "CreateDate"
@@
 F 32 "02016D104KAT2A" H 7100 2360 60  0001 L CNN "Manufacturer1 Part Number"
 F 33 "0.33mm" H 7100 2270 60  0001 L CNN "Manufacturer1 ComponentHeight"
-F 34 "\\\\cern.ch\\dfs\\Applications\\Altium\\Datasheets\\CC0201_X5R_AVX.pdf" H 7100 2180 60  0001 L CNN "HelpURL"
 F 35 "CERN DEM JLC" H 7100 2090 60  0001 L CNN "Author"
 F 36 "12/03/07 00:00:00" H 7100 2000 60  0001 L CNN "CreateDate"
@@
 F 32 "C0603C106M9PAC" H 8000 2660 60  0001 L CNN "Manufacturer1 Part Number"
 F 33 "0.95mm" H 8000 2570 60  0001 L CNN "Manufacturer1 ComponentHeight"
-F 34 "\\\\cern.ch\\dfs\\Applications\\Altium\\Datasheets\\CC0603_X5R_KEMET.pdf" H 8000 2480 60  0001 L CNN "HelpURL"
 F 35 "CERN DEM JLC" H 8000 2390 60  0001 L CNN "Author"
 F 36 "12/03/07 00:00:00" H 8000 2300 60  0001 L CNN "CreateDate"
@@
 F 32 "02016D104KAT2A" H 5650 3460 60  0001 L CNN "Manufacturer1 Part Number"
 F 33 "0.33mm" H 5650 3370 60  0001 L CNN "Manufacturer1 ComponentHeight"
-F 34 "\\\\cern.ch\\dfs\\Applications\\Altium\\Datasheets\\CC0201_X5R_AVX.pdf" H 5650 3280 60  0001 L CNN "HelpURL"
 F 35 "CERN DEM JLC" H 5650 3190 60  0001 L CNN "Author"
 F 36 "12/03/07 00:00:00" H 5650 3100 60  0001 L CNN "CreateDate"
@@
 F 32 "02016D104KAT2A" H 6100 3460 60  0001 L CNN "Manufacturer1 Part Number"
 F 33 "0.33mm" H 6100 3370 60  0001 L CNN "Manufacturer1 ComponentHeight"
-F 34 "\\\\cern.ch\\dfs\\Applications\\Altium\\Datasheets\\CC0201_X5R_AVX.pdf" H 6100 3280 60  0001 L CNN "HelpURL"
 F 35 "CERN DEM JLC" H 6100 3190 60  0001 L CNN "Author"
 F 36 "12/03/07 00:00:00" H 6100 3100 60  0001 L CNN "CreateDate"
@@
 F 32 "02016D104KAT2A" H 4400 2560 60  0001 L CNN "Manufacturer1 Part Number"
 F 33 "0.33mm" H 4400 2470 60  0001 L CNN "Manufacturer1 ComponentHeight"
-F 34 "\\\\cern.ch\\dfs\\Applications\\Altium\\Datasheets\\CC0201_X5R_AVX.pdf" H 4400 2380 60  0001 L CNN "HelpURL"
 F 35 "CERN DEM JLC" H 4400 2290 60  0001 L CNN "Author"
 F 36 "12/03/07 00:00:00" H 4400 2200 60  0001 L CNN "CreateDate"
@@
 F 32 "02016D104KAT2A" H 4850 2560 60  0001 L CNN "Manufacturer1 Part Number"
 F 33 "0.33mm" H 4850 2470 60  0001 L CNN "Manufacturer1 ComponentHeight"
-F 34 "\\\\cern.ch\\dfs\\Applications\\Altium\\Datasheets\\CC0201_X5R_AVX.pdf" H 4850 2380 60  0001 L CNN "HelpURL"
 F 35 "CERN DEM JLC" H 4850 2290 60  0001 L CNN "Author"
 F 36 "12/03/07 00:00:00" H 4850 2200 60  0001 L CNN "CreateDate"
@@
 F 32 "C1206C106K4RAC" H 2700 1910 60  0001 L CNN "Manufacturer1 Part Number"
 F 33 "1.8mm" H 2700 1820 60  0001 L CNN "Manufacturer1 ComponentHeight"
-F 34 "\\\\cern.ch\\dfs\\Applications\\Altium\\Datasheets\\CC1206_X7R_KEMET.pdf" H 2700 1730 60  0001 L CNN "HelpURL"
 F 35 "CERN DEM JLC" H 2700 1640 60  0001 L CNN "Author"
 F 36 "04/28/09 00:00:00" H 2700 1550 60  0001 L CNN "CreateDate"
@@
 F 32 "GRM155R61C104KA88D" H 2200 1910 60  0001 L CNN "Manufacturer1 Part Number"
 F 33 "0.55mm" H 2200 1820 60  0001 L CNN "Manufacturer1 ComponentHeight"
-F 34 "\\\\cern.ch\\dfs\\Applications\\Altium\\Datasheets\\CC0402_X5R_MURATA_GRM.pdf" H 2200 1730 60  0001 L CNN "HelpURL"
 F 35 "CERN DEM JLC" H 2200 1640 60  0001 L CNN "Author"
 F 36 "12/10/13 00:00:00" H 2200 1550 60  0001 L CNN "CreateDate"
@@
 F 29 "ASP-134603-01" H 3750 -5160 60  0001 L CNN "Manufacturer Part Number"
 F 30 "6.55mm" H 3750 -5250 60  0001 L CNN "ComponentHeight"
-F 31 "\\\\cern.ch\\dfs\\Applications\\Altium\\Datasheets\\SAMTEC_ASP-134603-01.pdf" H 3750 -5340 60  0001 L CNN "HelpURL"
-F 32 " " H 3750 -5430 60  0001 L CNN "ComponentLink1URL"
 F 33 " " H 3750 -5520 60  0001 L CNN "ComponentLink1Description"
-F 34 " " H 3750 -5610 60  0001 L CNN "ComponentLink2URL"
 F 35 " " H 3750 -5700 60  0001 L CNN "ComponentLink2Description"
 F 36 "CERN DEM JLC" H 3750 -5790 60  0001 L CNN "Author"
@@
 F 29 "ASP-134603-01" H 6050 -5160 60  0001 L CNN "Manufacturer Part Number"
 F 30 "6.55mm" H 6050 -5250 60  0001 L CNN "ComponentHeight"
-F 31 "\\\\cern.ch\\dfs\\Applications\\Altium\\Datasheets\\SAMTEC_ASP-134603-01.pdf" H 6050 -5340 60  0001 L CNN "HelpURL"
-F 32 " " H 6050 -5430 60  0001 L CNN "ComponentLink1URL"
 F 33 " " H 6050 -5520 60  0001 L CNN "ComponentLink1Description"
-F 34 " " H 6050 -5610 60  0001 L CNN "ComponentLink2URL"
 F 35 " " H 6050 -5700 60  0001 L CNN "ComponentLink2Description"
 F 36 "CERN DEM JLC" H 6050 -5790 60  0001 L CNN "Author"
@@
 F 29 "ASP-134603-01" H 8800 -5160 60  0001 L CNN "Manufacturer Part Number"
 F 30 "6.55mm" H 8800 -5250 60  0001 L CNN "ComponentHeight"
-F 31 "\\\\cern.ch\\dfs\\Applications\\Altium\\Datasheets\\SAMTEC_ASP-134603-01.pdf" H 8800 -5340 60  0001 L CNN "HelpURL"
-F 32 " " H 8800 -5430 60  0001 L CNN "ComponentLink1URL"
 F 33 " " H 8800 -5520 60  0001 L CNN "ComponentLink1Description"
-F 34 " " H 8800 -5610 60  0001 L CNN "ComponentLink2URL"
 F 35 " " H 8800 -5700 60  0001 L CNN "ComponentLink2Description"
 F 36 "CERN DEM JLC" H 8800 -5790 60  0001 L CNN "Author"
@@
 F 29 "ASP-134603-01" H 11450 -5160 60  0001 L CNN "Manufacturer Part Number"
 F 30 "6.55mm" H 11450 -5250 60  0001 L CNN "ComponentHeight"
-F 31 "\\\\cern.ch\\dfs\\Applications\\Altium\\Datasheets\\SAMTEC_ASP-134603-01.pdf" H 11450 -5340 60  0001 L CNN "HelpURL"
-F 32 " " H 11450 -5430 60  0001 L CNN "ComponentLink1URL"
 F 33 " " H 11450 -5520 60  0001 L CNN "ComponentLink1Description"
-F 34 " " H 11450 -5610 60  0001 L CNN "ComponentLink2URL"
 F 35 " " H 11450 -5700 60  0001 L CNN "ComponentLink2Description"
 F 36 "CERN DEM JLC" H 11450 -5790 60  0001 L CNN "Author"
@@
 F 33 "232270671003L" H 8150 3420 60  0001 L CNN "Manufacturer1 Part Number"
 F 34 "0.4mm" H 8150 3330 60  0001 L CNN "Manufacturer1 ComponentHeight"
-F 35 "\\\\cern.ch\\dfs\\Applications\\Altium\\Datasheets\\R0402_Phycomp_RC0402.pdf" H 8150 3240 60  0001 L CNN "HelpURL"
 F 36 "CERN DEM JLC" H 8150 3150 60  0001 L CNN "Author"
 F 37 "12/03/07 00:00:00" H 8150 3060 60  0001 L CNN "CreateDate"
@@
 F 33 "232270671002L" H 7950 3570 60  0001 L CNN "Manufacturer1 Part Number"
 F 34 "0.4mm" H 7950 3480 60  0001 L CNN "Manufacturer1 ComponentHeight"
-F 35 "\\\\cern.ch\\dfs\\Applications\\Altium\\Datasheets\\R0402_Phycomp_RC0402.pdf" H 7950 3390 60  0001 L CNN "HelpURL"
 F 36 "CERN DEM JLC" H 7950 3300 60  0001 L CNN "Author"
 F 37 "12/03/07 00:00:00" H 7950 3210 60  0001 L CNN "CreateDate"

Commit message: Trash "Footprint Library" and "Database Table Name" attributes
Takes 100 attributes out of schematic, 174 out of library
Parts:
- R297, R298: Database Table Name Resistors SMD -> (none); Footprint Library Resistors SMD -> (none)
Changed lines of the file:
@@
 F 36 "12/03/07 00:00:00" H 2800 2205 50  0001 L CNN "CreateDate"
 F 37 "10/17/12 00:00:00" H 2800 2130 50  0001 L CNN "LatestRevisionDate"
-F 38 "Resistors SMD" H 2800 2055 50  0001 L CNN "Database Table Name"
 F 39 "Resistors SMD" H 2800 1980 50  0001 L CNN "Library Name"
-F 40 "Resistors SMD" H 2800 1905 50  0001 L CNN "Footprint Library"
 F 41 "This work is licensed under the Creative Commons CC-BY-SA 4.0 License. To the extent that circuit schematics that use Licensed Material can be considered to be ‘Adapted Material’, then the copyright holder waives article 3.b of the license with respect to these schematics." H 2800 1830 50  0001 L CNN "License"
 	1    2800 4950
@@
 F 36 "12/03/07 00:00:00" H 4850 2305 50  0001 L CNN "CreateDate"
 F 37 "10/17/12 00:00:00" H 4850 2230 50  0001 L CNN "LatestRevisionDate"
-F 38 "Resistors SMD" H 4850 2155 50  0001 L CNN "Database Table Name"
 F 39 "Resistors SMD" H 4850 2080 50  0001 L CNN "Library Name"
-F 40 "Resistors SMD" H 4850 2005 50  0001 L CNN "Footprint Library"
 F 41 "This work is licensed under the Creative Commons CC-BY-SA 4.0 License. To the extent that circuit schematics that use Licensed Material can be considered to be ‘Adapted Material’, then the copyright holder waives article 3.b of the license with respect to these schematics." H 4850 1930 50  0001 L CNN "License"
 	1    4850 5050

Commit message: Trash SCEM attribute
Parts:
- P1: SCEM (none) -> (none)
Changed lines of the file:
@@
 F 24 " " H 3750 -4710 60  0001 L CNN "Status Comment"
 F 25 "None" H 3750 -4800 60  0001 L CNN "Status"
-F 26 " " H 3750 -4890 60  0001 L CNN "SCEM"
 F 27 "160 contacts (4 rows cdgh) Surface Mount Female Connector, VITA 57 (CC-LPC-10)" H 3750 -4980 60  0001 L CNN "Part Description"
 F 28 "SAMTEC" H 3750 -5070 60  0001 L CNN "Manufacturer"
@@
 F 24 " " H 6050 -4710 60  0001 L CNN "Status Comment"
 F 25 "None" H 6050 -4800 60  0001 L CNN "Status"
-F 26 " " H 6050 -4890 60  0001 L CNN "SCEM"
 F 27 "160 contacts (4 rows cdgh) Surface Mount Female Connector, VITA 57 (CC-LPC-10)" H 6050 -4980 60  0001 L CNN "Part Description"
 F 28 "SAMTEC" H 6050 -5070 60  0001 L CNN "Manufacturer"
@@
 F 24 " " H 8800 -4710 60  0001 L CNN "Status Comment"
 F 25 "None" H 8800 -4800 60  0001 L CNN "Status"
-F 26 " " H 8800 -4890 60  0001 L CNN "SCEM"
 F 27 "160 contacts (4 rows cdgh) Surface Mount Female Connector, VITA 57 (CC-LPC-10)" H 8800 -4980 60  0001 L CNN "Part Description"
 F 28 "SAMTEC" H 8800 -5070 60  0001 L CNN "Manufacturer"
@@
 F 24 " " H 11450 -4710 60  0001 L CNN "Status Comment"
 F 25 "None" H 11450 -4800 60  0001 L CNN "Status"
-F 26 " " H 11450 -4890 60  0001 L CNN "SCEM"
 F 27 "160 contacts (4 rows cdgh) Surface Mount Female Connector, VITA 57 (CC-LPC-10)" H 11450 -4980 60  0001 L CNN "Part Description"
 F 28 "SAMTEC" H 11450 -5070 60  0001 L CNN "Manufacturer"

Commit message: Touch up a few symbols and instances
Add attribute names to MIC2090
Fix spelling error in XRP7724 description
Remove stray AMC_FMC_Carrier-PcbDoc-cache.lib
Parts:
- U45: Case (none) -> SOT-23-5; Field4 MIC2090-1YM5TR -> (none); Field6 SOT-23-5 -> (none); Field7 MICREL SEMICONDUCTOR -> (none); Manufacturer (none) -> MICREL SEMICONDUCTOR; Part Number (none) -> MIC2090-1YM5TR
Changed lines of the file:
@@
 F 2 "ICs And Semiconductors SMD:SOT95P280X145-5N" H 7250 6200 50  0001 L BNN
 F 3 "58T4896" H 7250 5900 50  0001 L BNN
-F 4 "MIC2090-1YM5TR" H 7250 6100 50  0001 L BNN "Field4"
+F 4 "MIC2090-1YM5TR" H 7250 6100 50  0001 L BNN "Part Number"
 F 5 "1924707" H 7250 5800 50  0001 L BNN "Field5"
-F 6 "SOT-23-5" H 7250 6000 50  0001 L BNN "Field6"
-F 7 "MICREL SEMICONDUCTOR" H 7250 6300 50  0001 L BNN "Field7"
+F 6 "SOT-23-5" H 7250 6000 50  0001 L BNN "Case"
+F 7 "MICREL SEMICONDUCTOR" H 7250 6300 50  0001 L BNN "Manufacturer"
 	1    7250 6800
 	-1   0    0    -1
