File: FPGA_13_14.sch (KiCad schematic (older format))
At the start: 15 parts, among them SW1 SW_DIP_x01, U1 XC7A100T-2FGG484C, U11 SN74LVC1G125DCKT, U30 S25FL128SAGMFIR01

Commit message: Rename library AMC_FMC_Carrier-PcbDoc-rescue as marble_misc
Parts:
- SW1: symbol AMC_FMC_Carrier-PcbDoc-rescue:SW_DIP_x01-Switch-AMC_FMC_Carrier-PcbDoc-rescue -> marble_misc:SW_DIP_x01-Switch-AMC_FMC_Carrier-PcbDoc-rescue
- U1: symbol AMC_FMC_Carrier-PcbDoc-rescue:XC7A200T-FBG484-FPGA_Xilinx_Artix7-AMC_FMC_Carrier-PcbDoc-rescue -> marble_misc:XC7A200T-FBG484-FPGA_Xilinx_Artix7-AMC_FMC_Carrier-PcbDoc-rescue
- U11: symbol AMC_FMC_Carrier-PcbDoc-rescue:SN74LVC1G125DCKT-Standard_Logic-AMC_FMC_Carrier-PcbDoc-rescue -> marble_misc:SN74LVC1G125DCKT-Standard_Logic-AMC_FMC_Carrier-PcbDoc-rescue
- U30: symbol AMC_FMC_Carrier-PcbDoc-rescue:S25FL128SAGMFIR01-powerMG-AMC_FMC_Carrier-PcbDoc-rescue -> marble_misc:S25FL128SAGMFIR01-powerMG-AMC_FMC_Carrier-PcbDoc-rescue
Changed lines of the file:
@@
 $EndDescr
 $Comp
-L AMC_FMC_Carrier-PcbDoc-rescue:XC7A200T-FBG484-FPGA_Xilinx_Artix7-AMC_FMC_Carrier-PcbDoc-rescue U?
+L marble_misc:XC7A200T-FBG484-FPGA_Xilinx_Artix7-AMC_FMC_Carrier-PcbDoc-rescue U?
 U 1 1 5CC902F4
 P 8500 5200
@@
 	7200 2300 7100 2300
 $Comp
-L AMC_FMC_Carrier-PcbDoc-rescue:S25FL128SAGMFIR01-powerMG-AMC_FMC_Carrier-PcbDoc-rescue U30
+L marble_misc:S25FL128SAGMFIR01-powerMG-AMC_FMC_Carrier-PcbDoc-rescue U30
 U 1 1 5C40DA57
 P 13400 850
@@
 $EndComp
 $Comp
-L AMC_FMC_Carrier-PcbDoc-rescue:S25FL128SAGMFIR01-powerMG-AMC_FMC_Carrier-PcbDoc-rescue U30
+L marble_misc:S25FL128SAGMFIR01-powerMG-AMC_FMC_Carrier-PcbDoc-rescue U30
 U 2 1 5C40DA9C
 P 14700 850
@@
 	12650 1650 13200 1650
 $Comp
-L AMC_FMC_Carrier-PcbDoc-rescue:SW_DIP_x01-Switch-AMC_FMC_Carrier-PcbDoc-rescue SW1
+L marble_misc:SW_DIP_x01-Switch-AMC_FMC_Carrier-PcbDoc-rescue SW1
 U 1 1 5C881CE2
 P 13300 3000
@@
 $EndComp
 $Comp
-L AMC_FMC_Carrier-PcbDoc-rescue:SN74LVC1G125DCKT-Standard_Logic-AMC_FMC_Carrier-PcbDoc-rescue U11
+L marble_misc:SN74LVC1G125DCKT-Standard_Logic-AMC_FMC_Carrier-PcbDoc-rescue U11
 U 1 1 5C4235B4
 P 14150 2800
