File: WhiteRabbit.sch (KiCad schematic (older format))
At the start: 52 parts, among them U13 LP5951MF-3.0/NOPB, U14 LM336M-2.5, U16 AD5662BRMZ-1, U19 AD5662BRMZ-1, U20 CDCM61004RHBT, Y1 OSC_25MHZ_RAKON_IVT3205CR, Y2 VM53S3-25.000-2.5/-30+75, Y3 OSC_20MHZ_IQD_LFVCXO026156

Commit message: Rename library AMC_FMC_Carrier-PcbDoc-rescue as marble_misc
Parts:
- U13: symbol AMC_FMC_Carrier-PcbDoc-rescue:LP5951-clocks-SchDoc-cache-AMC_FMC_Carrier-PcbDoc-rescue -> marble_misc:LP5951-clocks-SchDoc-cache-AMC_FMC_Carrier-PcbDoc-rescue
- U14: symbol AMC_FMC_Carrier-PcbDoc-rescue:LM336M-2.5-clocks-SchDoc-cache-AMC_FMC_Carrier-PcbDoc-rescue -> marble_misc:LM336M-2.5-clocks-SchDoc-cache-AMC_FMC_Carrier-PcbDoc-rescue
- Y2: symbol AMC_FMC_Carrier-PcbDoc-rescue:Oscillator_1VC_2GND_3OUT_4+Vs-clocks-SchDoc-cache-AMC_FMC_Carrier-PcbDoc-rescue -> marble_misc:Oscillator_1VC_2GND_3OUT_4+Vs-clocks-SchDoc-cache-AMC_FMC_Carrier-PcbDoc-rescue
Changed lines of the file:
@@
 	3750 4450 3750 5450
 $Comp
-L AMC_FMC_Carrier-PcbDoc-rescue:LM336M-2.5-clocks-SchDoc-cache-AMC_FMC_Carrier-PcbDoc-rescue U14
+L marble_misc:LM336M-2.5-clocks-SchDoc-cache-AMC_FMC_Carrier-PcbDoc-rescue U14
 U 1 1 5C21F363
 P 2200 6900
@@
 	8850 5100 8850 5200
 $Comp
-L AMC_FMC_Carrier-PcbDoc-rescue:+3V3_CLEAN-powerMG-AMC_FMC_Carrier-PcbDoc-rescue #PWR0175
+L marble_misc:+3V3_CLEAN-powerMG-AMC_FMC_Carrier-PcbDoc-rescue #PWR0175
 U 1 1 5C2DA97A
 P 2300 6100
@@
 $EndComp
 $Comp
-L AMC_FMC_Carrier-PcbDoc-rescue:+3V3_CLEAN-powerMG-AMC_FMC_Carrier-PcbDoc-rescue #PWR0174
+L marble_misc:+3V3_CLEAN-powerMG-AMC_FMC_Carrier-PcbDoc-rescue #PWR0174
 U 1 1 5C2DA9DF
 P 2250 5650
@@
 $EndComp
 $Comp
-L AMC_FMC_Carrier-PcbDoc-rescue:+3V3_CLEAN-powerMG-AMC_FMC_Carrier-PcbDoc-rescue #PWR0209
+L marble_misc:+3V3_CLEAN-powerMG-AMC_FMC_Carrier-PcbDoc-rescue #PWR0209
 U 1 1 5C2DD28D
 P 7450 5100
@@
 $EndComp
 $Comp
-L AMC_FMC_Carrier-PcbDoc-rescue:+3V3_CLEAN-powerMG-AMC_FMC_Carrier-PcbDoc-rescue #PWR0173
+L marble_misc:+3V3_CLEAN-powerMG-AMC_FMC_Carrier-PcbDoc-rescue #PWR0173
 U 1 1 5C2DDAC4
 P 2250 4650
@@
 CLK20_VCXO
 $Comp
-L AMC_FMC_Carrier-PcbDoc-rescue:LP5951-clocks-SchDoc-cache-AMC_FMC_Carrier-PcbDoc-rescue U13
+L marble_misc:LP5951-clocks-SchDoc-cache-AMC_FMC_Carrier-PcbDoc-rescue U13
 U 1 1 5C2E75E7
 P 1700 2500
@@
 $EndComp
 $Comp
-L AMC_FMC_Carrier-PcbDoc-rescue:+3V3_CLEAN-powerMG-AMC_FMC_Carrier-PcbDoc-rescue #PWR0169
+L marble_misc:+3V3_CLEAN-powerMG-AMC_FMC_Carrier-PcbDoc-rescue #PWR0169
 U 1 1 5C2EF25E
 P 700 2500
@@
 $EndComp
 $Comp
-L AMC_FMC_Carrier-PcbDoc-rescue:Oscillator_1VC_2GND_3OUT_4+Vs-clocks-SchDoc-cache-AMC_FMC_Carrier-PcbDoc-rescue Y2
+L marble_misc:Oscillator_1VC_2GND_3OUT_4+Vs-clocks-SchDoc-cache-AMC_FMC_Carrier-PcbDoc-rescue Y2
 U 1 1 5C2F3070
 P 4050 1950
@@
 $EndComp
 $Comp
-L AMC_FMC_Carrier-PcbDoc-rescue:+3V3_CLEAN-powerMG-AMC_FMC_Carrier-PcbDoc-rescue #PWR0206
+L marble_misc:+3V3_CLEAN-powerMG-AMC_FMC_Carrier-PcbDoc-rescue #PWR0206
 U 1 1 5C33B37A
 P 6550 6900
@@
 	6300 6250 6300 6300
 $Comp
-L AMC_FMC_Carrier-PcbDoc-rescue:+3V3_CLEAN-powerMG-AMC_FMC_Carrier-PcbDoc-rescue #PWR0189
+L marble_misc:+3V3_CLEAN-powerMG-AMC_FMC_Carrier-PcbDoc-rescue #PWR0189
 U 1 1 5C3A12D5
 P 5300 5900
@@
 	5300 5900 5300 5950
 $Comp
-L AMC_FMC_Carrier-PcbDoc-rescue:+3V3_CLEAN-powerMG-AMC_FMC_Carrier-PcbDoc-rescue #PWR0211
+L marble_misc:+3V3_CLEAN-powerMG-AMC_FMC_Carrier-PcbDoc-rescue #PWR0211
 U 1 1 5C8A0C88
 P 6500 1450
@@
 	10050 3750 10050 3800
 $Comp
-L AMC_FMC_Carrier-PcbDoc-rescue:+3V3_CLEAN-powerMG-AMC_FMC_Carrier-PcbDoc-rescue #PWR0399
+L marble_misc:+3V3_CLEAN-powerMG-AMC_FMC_Carrier-PcbDoc-rescue #PWR0399
 U 1 1 5D15AFE0
 P 10050 3400
@@
 NoConn ~ 2500 2800
 $Comp
-L AMC_FMC_Carrier-PcbDoc-rescue:+3V3_CLEAN-powerMG-AMC_FMC_Carrier-PcbDoc-rescue #PWR0401
+L marble_misc:+3V3_CLEAN-powerMG-AMC_FMC_Carrier-PcbDoc-rescue #PWR0401
 U 1 1 5D19EDBE
 P 10850 2700
