File: WhiteRabbit.sch (KiCad schematic (older format))
At the start: 52 parts, among them U13 LP5951MF-3.0/NOPB, U14 LM336M-2.5, U16 AD5662BRMZ-1, U19 AD5662BRMZ-1, U20 CDCM61004RHBT, Y1 OSC_25MHZ_RAKON_IVT3205CR, Y2 VM53S3-25.000-2.5/-30+75, Y3 OSC_20MHZ_IQD_LFVCXO026156

Commit message: Convert 3 caps to CC0402_10NF_35V_10%_X7R
C107 C188 C189
TDK CGA2B3X7R1V103K050B, $0.03250 in 100s at Digi-Key
Reduces BOM count by one
Parts:
- C107: value CC0402_10NF_16V_10%_X7R -> CC0402_10NF_35V_10%_X7R; symbol Capacitors_SMD:CC0402_10NF_16V_10%_X7R -> Capacitors_SMD:CC0402_10NF_35V_10%_X7R; LatestRevisionDate 12/03/07 00:00:00 -> 05/24/20 00:00:00; Manufacturer Part Number CC0402_10NF_16V_10%_X7R -> CC0402_10NF_35V_10%_X7R; Manufacturer1 Example PHYCOMP -> TDK; Manufacturer1 Part Number 223878715636 -> CGA2B3X7R1V103K050B; Part Number CC0402_10NF_16V_10%_X7R -> CC0402_10NF_35V_10%_X7R; Voltage 16V -> 35V
Changed lines of the file:
@@
 Connection ~ 700  2600
 $Comp
-L Capacitors_SMD:CC0402_10NF_16V_10%_X7R C107
+L Capacitors_SMD:CC0402_10NF_35V_10%_X7R C107
 U 1 1 5D4CC6CD
 P 3600 2650
 F 0 "C107" V 3704 2760 50  0000 L CNN
-F 1 "CC0402_10NF_16V_10%_X7R" H 3600 2390 60  0001 L CNN
+F 1 "CC0402_10NF_35V_10%_X7R" H 3600 2390 60  0001 L CNN
 F 2 "Marble:CAPC1005X55N" H 3600 1580 60  0001 L CNN
 F 3 "\\\\cern.ch\\dfs\\Applications\\Altium\\Datasheets\\CC0402_X7R_PHYCOMP.pdf" H 3600 2210 60  0001 L CNN
 F 4 "10nF" V 3795 2760 50  0000 L CNN "Val"
-F 5 "CC0402_10NF_16V_10%_X7R" H 3600 2120 60  0001 L CNN "Part Number"
+F 5 "CC0402_10NF_35V_10%_X7R" H 3600 2120 60  0001 L CNN "Part Number"
 F 6 "Capacitor - non polarized" H 3600 2030 60  0001 L CNN "Library Ref"
 F 7 "SchLib\\Capacitors.SchLib" H 3600 1940 60  0001 L CNN "Library Path"
@@
 F 15 "Not Recommended" H 3600 1040 60  0001 L CNN "Status"
 F 16 " " H 3600 950 60  0001 L CNN "Status Comment"
-F 17 "16V" H 3600 860 60  0001 L CNN "Voltage"
+F 17 "35V" H 3600 860 60  0001 L CNN "Voltage"
 F 18 "X7R" H 3600 770 60  0001 L CNN "TC"
 F 19 "±10%" H 3600 680 60  0001 L CNN "Tolerance"
 F 20 "SMD Multilayer Chip Ceramic Capacitor" H 3600 590 60  0001 L CNN "Part Description"
 F 21 "GENERIC" H 3600 500 60  0001 L CNN "Manufacturer"
-F 22 "CC0402_10NF_16V_10%_X7R" H 3600 410 60  0001 L CNN "Manufacturer Part Number"
+F 22 "CC0402_10NF_35V_10%_X7R" H 3600 410 60  0001 L CNN "Manufacturer Part Number"
 F 23 "0402" H 3600 320 60  0001 L CNN "Case"
 F 24 "Yes" H 3600 230 60  0001 L CNN "Mounted"
@@
 F 29 " " H 3600 -220 60  0001 L CNN "Sense Comment"
 F 30 " " H 3600 -310 60  0001 L CNN "ComponentHeight"
-F 31 "PHYCOMP" H 3600 -400 60  0001 L CNN "Manufacturer1 Example"
-F 32 "223878715636" H 3600 -490 60  0001 L CNN "Manufacturer1 Part Number"
+F 31 "TDK" H 3600 -400 60  0001 L CNN "Manufacturer1 Example"
+F 32 "CGA2B3X7R1V103K050B" H 3600 -490 60  0001 L CNN "Manufacturer1 Part Number"
 F 33 "0.55mm" H 3600 -580 60  0001 L CNN "Manufacturer1 ComponentHeight"
 F 34 "CERN DEM JLC" H 3600 -760 60  0001 L CNN "Author"
 F 35 "12/03/07 00:00:00" H 3600 -850 60  0001 L CNN "CreateDate"
-F 36 "12/03/07 00:00:00" H 3600 -940 60  0001 L CNN "LatestRevisionDate"
+F 36 "05/24/20 00:00:00" H 3600 -940 60  0001 L CNN "LatestRevisionDate"
 F 37 "Capacitors SMD" H 3600 -1030 60  0001 L CNN "Library Name"
 F 38 "This work is licensed under the Creative Commons CC-BY-SA 4.0 License. To the extent that circuit schematics that use Licensed Material can be considered to be ‘Adapted Material’, then the copyright holder waives article 3.b of the license with respect to these schematics." H 3600 -1120 60  0001 L CNN "License"

Commit message: added SI570, U39 3V3 -> 3V3P
Parts:
- added C383: CC0402_1UF_16V_10%_X5R, Marble:CAPC1005X55N, symbol Capacitors_SMD:CC0402_1UF_16V_10%_X5R
- added C384: CC0201_100NF_6.3V_10%_X5R, Marble:CAPC0603X33N, symbol Capacitors_SMD:CC0201_100NF_6.3V_10%_X5R
- added R308: R0402_10K_1%_0.0625W_100PPM, Marble:RESC1005X40N, symbol Resistors_SMD:R0402_10K_1%_0.0625W_100PPM
- added Y6: OSC_10-280MHZ_SILICON-LAB_Si570BBC000121DG, ICs And Semiconductors SMD:OSC_SILICON-LAB_SI570, symbol Crystals_&_Oscillators:OSC_10-280MHZ_SILICON-LAB_Si570BBC000121DG
Connections:
- net labels added: SI570_CLK_N, SI570_CLK_P, SI570_OE, SI570_SCL, SI570_SDA
- wire segments 169 -> 179
- no-connect marks 8 -> 9
Other:
- moved on the sheet: R103, Y3

Commit message: More work on Si570 circuit
Attach SI570_{SCL,SDA} to I2C_APP
Make a part number for Y6 visible on schematic
Mark Y6 Si570 as dnf
Mark C385 C386 as dnf
Layout passes DRC
Parts:
- Y6: Val 10-280MHz -> Si570, 10-280MHz; config (none) -> dnf
Changed lines of the file:
@@
 F 2 "ICs And Semiconductors SMD:OSC_SILICON-LAB_SI570" H 7800 4550 50  0001 L CNN
 F 3 " " H 7800 4475 50  0001 L CNN
-F 4 "10-280MHz" H 8200 5374 50  0000 C CNN "Val"
+F 4 "Si570, 10-280MHz" H 8200 5374 50  0000 C CNN "Val"
 F 5 "OSC_10-280MHZ_SILICON-LAB_Si570BBC000121DG" H 7800 4400 50  0001 L CNN "Part Number"
 F 6 "Oscillator SILICON-LAB_Si570" H 7800 4325 50  0001 L CNN "Library Ref"
@@
 F 37 "ICs And Semiconductors SMD" H 7800 2000 50  0001 L CNN "Footprint Library"
 F 38 "This work is licensed under the Creative Commons CC-BY-SA 4.0 License. To the extent that circuit schematics that use Licensed Material can be considered to be ‘Adapted Material’, then the copyright holder waives article 3.b of the license with respect to these schematics." H 7800 1925 50  0001 L CNN "License"
+F 39 "dnf" H 8350 5450 50  0000 C CNN "config"
 	1    7800 5300
 	1    0    0    -1

Commit message: Better attribute consistency: fewer warnings from KiBoM
Someday maybe we'll just nuke the Comment field entirely
Parts:
- R308: Comment 10k -> =Value
Changed lines of the file:
@@
 F 6 "Resistor - 1%" H 7550 4605 50  0001 L CNN "Library Ref"
 F 7 "SchLib\\Resistors.SchLib" H 7550 4530 50  0001 L CNN "Library Path"
-F 8 "10k" H 7550 4455 50  0001 L CNN "Comment"
+F 8 "=Value" H 7550 4455 50  0001 L CNN "Comment"
 F 9 "Standard" H 7550 4380 50  0001 L CNN "Component Kind"
 F 10 "Standard" H 7550 4305 50  0001 L CNN "Component Type"

Commit message: Start filling in more Manufacturer fields
Parts:
- Y2: symbol marble_misc:Oscillator_1VC_2GND_3OUT_4+Vs-clocks-SchDoc-cache -> marble_misc:Oscillator_1VC_2GND_3OUT_4+Vs; Manufacturer (none) -> Mercury
Changed lines of the file:
@@
 $EndComp
 $Comp
-L marble_misc:Oscillator_1VC_2GND_3OUT_4+Vs-clocks-SchDoc-cache Y2
+L marble_misc:Oscillator_1VC_2GND_3OUT_4+Vs Y2
 U 1 1 5C2F3070
 P 4050 1950
@@
 F 3 "" H 4050 1950 60  0000 C CNN
 F 4 "VM53S3-25.000-2.5/-30+75" H 4050 1950 50  0001 C CNN "Manufacturer Part Number"
+F 5 "Mercury" H 3950 1950 50  0001 C CNN "Manufacturer"
 	1    4050 1950
 	1    0    0    -1

Commit message: List more Manufacturers
Parts:
- U13, U14: Manufacturer (none) -> TEXAS INSTRUMENTS
Changed lines of the file:
@@
 F 3 "" H 2200 6900 60  0000 C CNN
 F 4 "LM336M-2.5" V 2200 6900 50  0001 C CNN "Manufacturer Part Number"
+F 5 "TEXAS INSTRUMENTS" V 2200 6900 50  0001 C CNN "Manufacturer"
 	1    2200 6900
 	0    -1   -1   0
@@
 F 3 "" H 1700 2500 60  0000 C CNN
 F 4 "LP5951MF-3.0/NOPB" H 1700 2500 50  0001 C CNN "Manufacturer Part Number"
+F 5 "TEXAS INSTRUMENTS" H 1700 2500 50  0001 C CNN "Manufacturer"
 	1    1700 2500
 	1    0    0    -1

Commit message: Part substitutions
Mercury VM53S3-25.000-2.5/-30+75 (Y2) => Taiten TXEAADSANF-25.000000 (Y1)
IQD LFVCXO026156 => Kyocera KV7050B20.0000C3GD00
Kingbright KPH-1608CGCK => Wurth 150060VS75000
Should make it easier to source parts in the USA in 2020
Also remove un-helpful (DC-10A) from Cliff FC68148;
Manufacturer part numbers now no longer have spaces; can't say the same about Manufacturer
Parts:
- Y1: Manufacturer RAKON -> TAITEN; Manufacturer Part Number IVT3205CR 25.0 MHz -> TXEAADSANF-25.000000; config dnf -> (none)
- Y2: config (none) -> dnf
- Y3: Manufacturer IQD FREQUENCY PRODUCTS -> KYOCERA; Manufacturer Part Number LFVCXO026156 -> KV7050B20.0000C3GD00
Changed lines of the file:
@@
 F 4 "VM53S3-25.000-2.5/-30+75" H 4050 1950 50  0001 C CNN "Manufacturer Part Number"
 F 5 "Mercury" H 3950 1950 50  0001 C CNN "Manufacturer"
+F 6 "dnf" H 4350 1500 50  0000 C CNN "config"
 	1    4050 1950
 	1    0    0    -1
@@
 F 13 " " H 7800 2740 60  0001 L CNN "Status"
 F 14 "3.3V, ±100ppm, 15pF, 0..70°C, HCMOS Tri-State Surface Mount, VCXO Voltage Controlled Oscillator (CFPV-45 Series)" H 7800 2650 60  0001 L CNN "Part Description"
-F 15 "IQD FREQUENCY PRODUCTS" H 7800 2560 60  0001 L CNN "Manufacturer"
-F 16 "LFVCXO026156" H 7800 2470 60  0001 L CNN "Manufacturer Part Number"
+F 15 "KYOCERA" H 7800 2560 60  0001 L CNN "Manufacturer"
+F 16 "KV7050B20.0000C3GD00" H 7800 2470 60  0001 L CNN "Manufacturer Part Number"
 F 17 "6" H 7800 2380 60  0001 L CNN "Pin Count"
 F 18 " " H 7800 2290 60  0001 L CNN "Case"
@@
 F 13 " " H 4050 -610 60  0001 L CNN "Status"
 F 14 "11pF 3.3V ±1ppm Surface Mount TCXO Voltage Controlled Oscillator (IT3200C Series)" H 4050 -700 60  0001 L CNN "Part Description"
-F 15 "RAKON" H 4050 -790 60  0001 L CNN "Manufacturer"
-F 16 "IVT3205CR 25.0 MHz" H 4050 -880 60  0001 L CNN "Manufacturer Part Number"
+F 15 "TAITEN" H 4000 1500 60  0000 L CNN "Manufacturer"
+F 16 "TXEAADSANF-25.000000" H 4000 1400 60  0000 L CNN "Manufacturer Part Number"
 F 17 "4" H 4050 -970 60  0001 L CNN "Pin Count"
 F 18 " " H 4050 -1060 60  0001 L CNN "Case"
@@
 F 35 "ICs And Semiconductors SMD" H 4050 -2950 60  0001 L CNN "Library Name"
 F 36 "This work is licensed under the Creative Commons CC-BY-SA 4.0 License. To the extent that circuit schematics that use Licensed Material can be considered to be ‘Adapted Material’, then the copyright holder waives article 3.b of the license with respect to these schematics." H 4050 -3040 60  0001 L CNN "License"
-F 37 "dnf" H 4350 700 50  0000 C CNN "config"
+F 37 "" H 4350 700 50  0001 C CNN "config"
 	1    4050 1150
 	1    0    0    -1

Commit message: Fix spelling of Taitien
Manufacturer of VCTCXO
Parts:
- Y1: Manufacturer TAITEN -> TAITIEN
Changed lines of the file:
@@
 F 13 " " H 4050 -610 60  0001 L CNN "Status"
 F 14 "11pF 3.3V ±1ppm Surface Mount TCXO Voltage Controlled Oscillator (IT3200C Series)" H 4050 -700 60  0001 L CNN "Part Description"
-F 15 "TAITEN" H 4000 1500 60  0000 L CNN "Manufacturer"
+F 15 "TAITIEN" H 4000 1500 60  0000 L CNN "Manufacturer"
 F 16 "TXEAADSANF-25.000000" H 4000 1400 60  0000 L CNN "Manufacturer Part Number"
 F 17 "4" H 4050 -970 60  0001 L CNN "Pin Count"
