File: USB.sch (KiCad schematic (older format))
At the start: 74 parts, among them J10 10103594-0001LF, Q14 BSS139, Q18 BSS139, Q24 BSS139, Q6 BSS139, U15 SN74AVC2T245RSWR, U21 M93C46-WMN6TP, U22 TLV62565DBVT, U23 FT4232H-56Q, U24 SN74AVC2T245RSWR, U25 SN74AVC2T245RSWR, U26 SN74AVC2T245RSWR, U33 SN74AVC2T245RSWR, U38 SN74AVC2T245RSWR, Y4 XTAL_12MHZ_TXC_7M-12.000MAAJ-T

Commit message: SW2 placement changed, BOM cleared, FPGA boot, less ERC errors and wornings
Connections:
- wire segments 234 -> 236
Changed lines of the file:
@@
 L power:GND #PWR?
 U 1 1 5C393657
-P 5900 2200
+P 5900 2250
 AR Path="/5BD32060/5C393657" Ref="#PWR?"  Part="1"
 AR Path="/5C16C03C/5C393657" Ref="#PWR0295"  Part="1"
-F 0 "#PWR0295" H 5900 1950 50  0001 C CNN
-F 1 "GND" H 5905 2027 50  0000 C CNN
-F 2 "" H 5900 2200 50  0001 C CNN
-F 3 "" H 5900 2200 50  0001 C CNN
-	1    5900 2200
+F 0 "#PWR0295" H 5900 2000 50  0001 C CNN
+F 1 "GND" H 5905 2077 50  0000 C CNN
+F 2 "" H 5900 2250 50  0001 C CNN
+F 3 "" H 5900 2250 50  0001 C CNN
+	1    5900 2250
 	1    0    0    -1
 $EndComp
@@
 	6100 6500 6400 6500
 Connection ~ 5650 5800
-Wire Wire Line
-	5650 5800 6100 5800
 Connection ~ 6100 5800
 Wire Wire Line
@@
 U 1 1 5CCDD1FD
 P 4450 1900
-F 0 "L23" H 4600 2081 50  0000 C CNN
+F 0 "L23" H 4600 1850 50  0000 C CNN
 F 1 "IND_2.2UH_20%_WURTH_WE-PMCI_74479276222C" H 4450 1710 60  0001 L CNN
 F 2 "IND_WURTH_WE-PMCI_0806LR" H 4450 900 60  0001 L CNN
@@
 	1    0    0    -1
 $EndComp
+$Comp
+L power:PWR_FLAG #FLG?
+U 1 1 5D3A625F
+P 6100 6500
+AR Path="/5BABAC65/5D3A625F" Ref="#FLG?"  Part="1"
+AR Path="/5C16C03C/5D3A625F" Ref="#FLG0123"  Part="1"
+F 0 "#FLG0123" H 6100 6575 50  0001 C CNN
+F 1 "PWR_FLAG" H 6100 6673 50  0000 C CNN
+F 2 "" H 6100 6500 50  0001 C CNN
+F 3 "~" H 6100 6500 50  0001 C CNN
+	1    6100 6500
+	1    0    0    -1
+$EndComp
+$Comp
+L power:PWR_FLAG #FLG?
+U 1 1 5D3B7409
+P 5850 5800
+AR Path="/5BABAC65/5D3B7409" Ref="#FLG?"  Part="1"
+AR Path="/5C16C03C/5D3B7409" Ref="#FLG0124"  Part="1"
+F 0 "#FLG0124" H 5850 5875 50  0001 C CNN
+F 1 "PWR_FLAG" H 5850 5973 50  0000 C CNN
+F 2 "" H 5850 5800 50  0001 C CNN
+F 3 "~" H 5850 5800 50  0001 C CNN
+	1    5850 5800
+	1    0    0    -1
+$EndComp
+Wire Wire Line
+	5650 5800 5850 5800
+Connection ~ 5850 5800
+Wire Wire Line
+	5850 5800 6100 5800
+$Comp
+L power:PWR_FLAG #FLG?
+U 1 1 5D3DB3C4
+P 10050 8850
+AR Path="/5BABAC65/5D3DB3C4" Ref="#FLG?"  Part="1"
+AR Path="/5C16C03C/5D3DB3C4" Ref="#FLG0125"  Part="1"
+F 0 "#FLG0125" H 10050 8925 50  0001 C CNN
+F 1 "PWR_FLAG" H 10050 9023 50  0000 C CNN
+F 2 "" H 10050 8850 50  0001 C CNN
+F 3 "~" H 10050 8850 50  0001 C CNN
+	1    10050 8850
+	1    0    0    -1
+$EndComp
+Connection ~ 10050 8850
+$Comp
+L power:PWR_FLAG #FLG?
+U 1 1 5D3ED707
+P 2500 3700
+AR Path="/5BABAC65/5D3ED707" Ref="#FLG?"  Part="1"
+AR Path="/5C16C03C/5D3ED707" Ref="#FLG0126"  Part="1"
+F 0 "#FLG0126" H 2500 3775 50  0001 C CNN
+F 1 "PWR_FLAG" H 2500 3873 50  0000 C CNN
+F 2 "" H 2500 3700 50  0001 C CNN
+F 3 "~" H 2500 3700 50  0001 C CNN
+	1    2500 3700
+	1    0    0    -1
+$EndComp
+Connection ~ 2500 3700
+$Comp
+L power:PWR_FLAG #FLG?
+U 1 1 5D3FE99C
+P 4350 1900
+AR Path="/5BABAC65/5D3FE99C" Ref="#FLG?"  Part="1"
+AR Path="/5C16C03C/5D3FE99C" Ref="#FLG0127"  Part="1"
+F 0 "#FLG0127" H 4350 1975 50  0001 C CNN
+F 1 "PWR_FLAG" H 4350 2073 50  0000 C CNN
+F 2 "" H 4350 1900 50  0001 C CNN
+F 3 "~" H 4350 1900 50  0001 C CNN
+	1    4350 1900
+	1    0    0    -1
+$EndComp
+Connection ~ 4350 1900
+Wire Wire Line
+	5900 2200 5900 2250
 $EndSCHEMATC

Commit message: BOM updated, 25MHz clock level fixed
Parts:
- J10: symbol AMC_FMC_Carrier-PcbDoc-rescue:HIROSE_ZX62RD-AB-5P8-Miscellaneous -> AMC_FMC_Carrier-PcbDoc-rescue:HIROSE_ZX62RD-AB-5P8-Miscellaneous-AMC_FMC_Carrier-PcbDoc-rescue
Changed lines of the file:
@@
 $EndDescr
 $Comp
-L AMC_FMC_Carrier-PcbDoc-rescue:HIROSE_ZX62RD-AB-5P8-Miscellaneous J10
+L AMC_FMC_Carrier-PcbDoc-rescue:HIROSE_ZX62RD-AB-5P8-Miscellaneous-AMC_FMC_Carrier-PcbDoc-rescue J10
 U 1 1 5BEB92E1
 P 1700 3500
@@
 $EndComp
 $Comp
-L AMC_FMC_Carrier-PcbDoc-rescue:+1V8_USB-powerMG #PWR0296
+L AMC_FMC_Carrier-PcbDoc-rescue:+1V8_USB-powerMG-AMC_FMC_Carrier-PcbDoc-rescue #PWR0296
 U 1 1 5BEBDA76
 P 5900 3250
@@
 $EndComp
 $Comp
-L AMC_FMC_Carrier-PcbDoc-rescue:+3V3_USB #PWR0275
+L AMC_FMC_Carrier-PcbDoc-rescue:+3V3_USB-AMC_FMC_Carrier-PcbDoc-rescue #PWR0275
 U 1 1 5E0639EB
 P 5900 1850
@@
 $EndComp
 $Comp
-L AMC_FMC_Carrier-PcbDoc-rescue:+3V3_USB #PWR0277
+L AMC_FMC_Carrier-PcbDoc-rescue:+3V3_USB-AMC_FMC_Carrier-PcbDoc-rescue #PWR0277
 U 1 1 5E0910B1
 P 6350 3300
@@
 $EndComp
 $Comp
-L AMC_FMC_Carrier-PcbDoc-rescue:+3V3_USB #PWR0279
+L AMC_FMC_Carrier-PcbDoc-rescue:+3V3_USB-AMC_FMC_Carrier-PcbDoc-rescue #PWR0279
 U 1 1 5E0AE015
 P 8300 2950
@@
 $EndComp
 $Comp
-L AMC_FMC_Carrier-PcbDoc-rescue:+3V3_USB #PWR0281
+L AMC_FMC_Carrier-PcbDoc-rescue:+3V3_USB-AMC_FMC_Carrier-PcbDoc-rescue #PWR0281
 U 1 1 5E0CAFF4
 P 11300 1500
@@
 $EndComp
 $Comp
-L AMC_FMC_Carrier-PcbDoc-rescue:+3V3_USB #PWR0282
+L AMC_FMC_Carrier-PcbDoc-rescue:+3V3_USB-AMC_FMC_Carrier-PcbDoc-rescue #PWR0282
 U 1 1 5E0E7F6F
 P 11550 2700
@@
 $EndComp
 $Comp
-L AMC_FMC_Carrier-PcbDoc-rescue:+3V3_USB #PWR0284
+L AMC_FMC_Carrier-PcbDoc-rescue:+3V3_USB-AMC_FMC_Carrier-PcbDoc-rescue #PWR0284
 U 1 1 5E1142BD
 P 11300 3450
@@
 $EndComp
 $Comp
-L AMC_FMC_Carrier-PcbDoc-rescue:+3V3_USB #PWR0285
+L AMC_FMC_Carrier-PcbDoc-rescue:+3V3_USB-AMC_FMC_Carrier-PcbDoc-rescue #PWR0285
 U 1 1 5E131666
 P 11300 2250
@@
 $EndComp
 $Comp
-L AMC_FMC_Carrier-PcbDoc-rescue:+3V3_USB #PWR0294
+L AMC_FMC_Carrier-PcbDoc-rescue:+3V3_USB-AMC_FMC_Carrier-PcbDoc-rescue #PWR0294
 U 1 1 5E14E7E2
 P 11300 4200
@@
 $EndComp
 $Comp
-L AMC_FMC_Carrier-PcbDoc-rescue:+3V3_USB #PWR0304
+L AMC_FMC_Carrier-PcbDoc-rescue:+3V3_USB-AMC_FMC_Carrier-PcbDoc-rescue #PWR0304
 U 1 1 5E16BA3D
 P 11550 4650
@@
 $EndComp
 $Comp
-L AMC_FMC_Carrier-PcbDoc-rescue:+3V3_USB #PWR0306
+L AMC_FMC_Carrier-PcbDoc-rescue:+3V3_USB-AMC_FMC_Carrier-PcbDoc-rescue #PWR0306
 U 1 1 5E1A590C
 P 13600 7250
@@
 $EndComp
 $Comp
-L AMC_FMC_Carrier-PcbDoc-rescue:+3V3_USB #PWR0307
+L AMC_FMC_Carrier-PcbDoc-rescue:+3V3_USB-AMC_FMC_Carrier-PcbDoc-rescue #PWR0307
 U 1 1 5E1B4270
 P 13250 6100
@@
 $EndComp
 $Comp
-L AMC_FMC_Carrier-PcbDoc-rescue:+3V3_USB #PWR0309
+L AMC_FMC_Carrier-PcbDoc-rescue:+3V3_USB-AMC_FMC_Carrier-PcbDoc-rescue #PWR0309
 U 1 1 5E1C2F5B
 P 13350 6800
@@
 	13250 6100 13400 6100
 $Comp
-L AMC_FMC_Carrier-PcbDoc-rescue:+3V3_USB #PWR0311
+L AMC_FMC_Carrier-PcbDoc-rescue:+3V3_USB-AMC_FMC_Carrier-PcbDoc-rescue #PWR0311
 U 1 1 5E1E0E93
 P 11300 7050
@@
 $EndComp
 $Comp
-L AMC_FMC_Carrier-PcbDoc-rescue:+3V3_USB #PWR0316
+L AMC_FMC_Carrier-PcbDoc-rescue:+3V3_USB-AMC_FMC_Carrier-PcbDoc-rescue #PWR0316
 U 1 1 5E20CA7E
 P 11300 7650
@@
 $EndComp
 $Comp
-L AMC_FMC_Carrier-PcbDoc-rescue:+3V3_USB #PWR0319
+L AMC_FMC_Carrier-PcbDoc-rescue:+3V3_USB-AMC_FMC_Carrier-PcbDoc-rescue #PWR0319
 U 1 1 5E24786F
 P 10050 8150
@@
 $EndComp
 $Comp
-L AMC_FMC_Carrier-PcbDoc-rescue:+3V3_USB #PWR0325
+L AMC_FMC_Carrier-PcbDoc-rescue:+3V3_USB-AMC_FMC_Carrier-PcbDoc-rescue #PWR0325
 U 1 1 5E28111D
 P 10000 8850
@@
 $EndComp
 $Comp
-L AMC_FMC_Carrier-PcbDoc-rescue:+3V3_USB #PWR0327
+L AMC_FMC_Carrier-PcbDoc-rescue:+3V3_USB-AMC_FMC_Carrier-PcbDoc-rescue #PWR0327
 U 1 1 5E29D842
 P 7200 8950
@@
 $EndComp
 $Comp
-L AMC_FMC_Carrier-PcbDoc-rescue:+3V3_USB #PWR0328
+L AMC_FMC_Carrier-PcbDoc-rescue:+3V3_USB-AMC_FMC_Carrier-PcbDoc-rescue #PWR0328
 U 1 1 5E2AB899
 P 7200 9050
@@
 $EndComp
 $Comp
-L AMC_FMC_Carrier-PcbDoc-rescue:+3V3_USB #PWR0330
+L AMC_FMC_Carrier-PcbDoc-rescue:+3V3_USB-AMC_FMC_Carrier-PcbDoc-rescue #PWR0330
 U 1 1 5E2C78AB
 P 7250 9650
@@
 $EndComp
 $Comp
-L AMC_FMC_Carrier-PcbDoc-rescue:+3V3_USB #PWR0332
+L AMC_FMC_Carrier-PcbDoc-rescue:+3V3_USB-AMC_FMC_Carrier-PcbDoc-rescue #PWR0332
 U 1 1 5E2E3981
 P 11550 8100
@@
 $EndComp
 $Comp
-L AMC_FMC_Carrier-PcbDoc-rescue:+3V3_USB #PWR0335
+L AMC_FMC_Carrier-PcbDoc-rescue:+3V3_USB-AMC_FMC_Carrier-PcbDoc-rescue #PWR0335
 U 1 1 5E30DBBE
 P 10250 9300
@@
 $EndComp
 $Comp
-L AMC_FMC_Carrier-PcbDoc-rescue:+3V3_USB #PWR0337
+L AMC_FMC_Carrier-PcbDoc-rescue:+3V3_USB-AMC_FMC_Carrier-PcbDoc-rescue #PWR0337
 U 1 1 5E329CA2
 P 7000 10100
@@
 $EndComp
 $Comp
-L AMC_FMC_Carrier-PcbDoc-rescue:+3V3_USB #PWR0339
+L AMC_FMC_Carrier-PcbDoc-rescue:+3V3_USB-AMC_FMC_Carrier-PcbDoc-rescue #PWR0339
 U 1 1 5E345D17
 P 5200 8000
@@
 Connection ~ 5200 8000
 $Comp
-L AMC_FMC_Carrier-PcbDoc-rescue:+3V3_USB #PWR0341
+L AMC_FMC_Carrier-PcbDoc-rescue:+3V3_USB-AMC_FMC_Carrier-PcbDoc-rescue #PWR0341
 U 1 1 5E37DE16
 P 5200 7200
@@
 $EndComp
 $Comp
-L AMC_FMC_Carrier-PcbDoc-rescue:+3V3_USB #PWR0343
+L AMC_FMC_Carrier-PcbDoc-rescue:+3V3_USB-AMC_FMC_Carrier-PcbDoc-rescue #PWR0343
 U 1 1 5E399F01
 P 4900 6500
@@
 $EndComp
 $Comp
-L AMC_FMC_Carrier-PcbDoc-rescue:+3V3_USB #PWR0478
+L AMC_FMC_Carrier-PcbDoc-rescue:+3V3_USB-AMC_FMC_Carrier-PcbDoc-rescue #PWR0478
 U 1 1 5E3B5F64
 P 4900 5800
@@
 $EndComp
 $Comp
-L AMC_FMC_Carrier-PcbDoc-rescue:+3V3_USB #PWR0479
+L AMC_FMC_Carrier-PcbDoc-rescue:+3V3_USB-AMC_FMC_Carrier-PcbDoc-rescue #PWR0479
 U 1 1 5E3DFF47
 P 4050 6550
@@
 $EndComp
 $Comp
-L AMC_FMC_Carrier-PcbDoc-rescue:+3V3_USB #PWR0480
+L AMC_FMC_Carrier-PcbDoc-rescue:+3V3_USB-AMC_FMC_Carrier-PcbDoc-rescue #PWR0480
 U 1 1 5E3EE00F
 P 3450 6200
@@
 $EndComp
 $Comp
-L AMC_FMC_Carrier-PcbDoc-rescue:+3V3_USB #PWR0599
+L AMC_FMC_Carrier-PcbDoc-rescue:+3V3_USB-AMC_FMC_Carrier-PcbDoc-rescue #PWR0599
 U 1 1 5E40A0AB
 P 3650 7250
@@
 $EndComp
 $Comp
-L AMC_FMC_Carrier-PcbDoc-rescue:+3V3_USB #PWR0601
+L AMC_FMC_Carrier-PcbDoc-rescue:+3V3_USB-AMC_FMC_Carrier-PcbDoc-rescue #PWR0601
 U 1 1 5E4346A3
 P 8000 8800
@@
 Connection ~ 6000 9450
 $Comp
-L AMC_FMC_Carrier-PcbDoc-rescue:+3V3_USB #PWR0643
+L AMC_FMC_Carrier-PcbDoc-rescue:+3V3_USB-AMC_FMC_Carrier-PcbDoc-rescue #PWR0643
 U 1 1 5CE79DFD
 P 5150 9500
@@
 Connection ~ 5150 10550
 $Comp
-L AMC_FMC_Carrier-PcbDoc-rescue:+3V3_USB #PWR0645
+L AMC_FMC_Carrier-PcbDoc-rescue:+3V3_USB-AMC_FMC_Carrier-PcbDoc-rescue #PWR0645
 U 1 1 5D07178D
 P 5700 10550

Commit message: BOM configuration file edited, updated Marble picture, some components part number changed
Parts:
- D13: symbol Diodes:PRTR5V0U2X -> AMC_FMC_Carrier-PcbDoc-rescue:PRTR5V0U2X-Diodes
- D16: Manufacturer Part Number BAT165 -> BAT165AX
- Q14, Q18, Q24, Q6: Manufacturer Part Number BSS139 -> BSS139H6327XTSA1
- U21: symbol Logic:M93C46-WMN6TP -> AMC_FMC_Carrier-PcbDoc-rescue:M93C46-WMN6TP-Logic
Changed lines of the file:
@@
 	4050 7150 4350 7150
 $Comp
-L Diodes:PRTR5V0U2X D13
+L AMC_FMC_Carrier-PcbDoc-rescue:PRTR5V0U2X-Diodes D13
 U 1 1 5E04F663
 P 2400 5400
@@
 Connection ~ 4350 4700
 $Comp
-L Logic:M93C46-WMN6TP U21
+L AMC_FMC_Carrier-PcbDoc-rescue:M93C46-WMN6TP-Logic U21
 U 1 1 5C74B2C9
 P 3250 6850
@@
 F 13 "250V 30mA N-Channel  SIPMOS® Small-Signal-Transistor" H 11050 4120 60  0001 L CNN "Part Description"
 F 14 "INFINEON" H 11050 4030 60  0001 L CNN "Manufacturer"
-F 15 "BSS139" H 11050 3940 60  0001 L CNN "Manufacturer Part Number"
+F 15 "BSS139H6327XTSA1" H 11050 3940 60  0001 L CNN "Manufacturer Part Number"
 F 16 "3" H 11050 3850 60  0001 L CNN "Pin Count"
 F 17 "SOT23-3" H 11050 3760 60  0001 L CNN "Case"
@@
 F 15 "Medium Power AF Schottky Diode" H 5150 8960 60  0001 L CNN "Part Description"
 F 16 "INFINEON" H 5150 8870 60  0001 L CNN "Manufacturer"
-F 17 "BAT165" H 5150 8780 60  0001 L CNN "Manufacturer Part Number"
+F 17 "BAT165AX" H 5150 8780 60  0001 L CNN "Manufacturer Part Number"
 F 18 "2" H 5150 8690 60  0001 L CNN "Pin Count"
 F 19 "SOD323" H 5150 8600 60  0001 L CNN "Case"
@@
 F 13 "250V 30mA N-Channel  SIPMOS® Small-Signal-Transistor" H 5850 8420 60  0001 L CNN "Part Description"
 F 14 "INFINEON" H 5850 8330 60  0001 L CNN "Manufacturer"
-F 15 "BSS139" H 5850 8240 60  0001 L CNN "Manufacturer Part Number"
+F 15 "BSS139H6327XTSA1" H 5850 8240 60  0001 L CNN "Manufacturer Part Number"
 F 16 "3" H 5850 8150 60  0001 L CNN "Pin Count"
 F 17 "SOT23-3" H 5850 8060 60  0001 L CNN "Case"
@@
 F 13 "250V 30mA N-Channel  SIPMOS® Small-Signal-Transistor" H 4700 8670 60  0001 L CNN "Part Description"
 F 14 "INFINEON" H 4700 8580 60  0001 L CNN "Manufacturer"
-F 15 "BSS139" H 4700 8490 60  0001 L CNN "Manufacturer Part Number"
+F 15 "BSS139H6327XTSA1" H 4700 8490 60  0001 L CNN "Manufacturer Part Number"
 F 16 "3" H 4700 8400 60  0001 L CNN "Pin Count"
 F 17 "SOT23-3" H 4700 8310 60  0001 L CNN "Case"
@@
 F 13 "250V 30mA N-Channel  SIPMOS® Small-Signal-Transistor" H 4700 9070 60  0001 L CNN "Part Description"
 F 14 "INFINEON" H 4700 8980 60  0001 L CNN "Manufacturer"
-F 15 "BSS139" H 4700 8890 60  0001 L CNN "Manufacturer Part Number"
+F 15 "BSS139H6327XTSA1" H 4700 8890 60  0001 L CNN "Manufacturer Part Number"
 F 16 "3" H 4700 8800 60  0001 L CNN "Pin Count"
 F 17 "SOT23-3" H 4700 8710 60  0001 L CNN "Case"

Commit message: applied all required amendments to the project
Parts:
- Q14, Q18, Q24, Q6: value BSS139 -> BSS138LT1G; footprint SOT95P240X110-3N -> ICs And Semiconductors SMD:SOT95P240X110-3N; symbol Transistors:BSS139 -> Transistors:BSS138LT1G; Comment =Device -> BSS138LT1G; ComponentHeight 1.1mm -> 1.11mm; ComponentLink1Description ~~ -> (none); ComponentLink2Description ~~ -> (none); CreateDate 09/23/14 00:00:00 -> 03/23/09 00:00:00; Database Table Name (none) -> Transistors; Device BSS139 -> BSS138LT1G; Footprint Library (none) -> ICs And Semiconductors SMD; LatestRevisionDate 09/23/14 00:00:00 -> 03/23/09 00:00:00; Library Name ICs And Semiconductors SMD -> ICs And Semiconductors.DbLib; Manufacturer INFINEON -> ON SEMICONDUCTOR; Manufacturer Part Number BSS139H6327XTSA1 -> BSS138LT1G; Part Description 250V 30mA N-Channel SIPMOS® Small-Signal-Transistor -> 50V 200mA N-Channel Enhancement Mode Field-Effect Transistor; Part Number BSS139 -> BSS138LT1G; SCEM (none) -> (none); Sense Comment ~~ -> (none); Status ~~ -> (none); Status Comment ~~ -> (none)
Connections:
- net USB_D_P: no longer R112.1
- net at D13.4 (VCC), J10.1 (VBUS), L10.1: now also R112.1

Commit message: Rename library AMC_FMC_Carrier-PcbDoc-rescue as marble_misc
Parts:
- D13: symbol AMC_FMC_Carrier-PcbDoc-rescue:PRTR5V0U2X-Diodes -> marble_misc:PRTR5V0U2X-Diodes
- J10: symbol AMC_FMC_Carrier-PcbDoc-rescue:HIROSE_ZX62RD-AB-5P8-Miscellaneous-AMC_FMC_Carrier-PcbDoc-rescue -> marble_misc:HIROSE_ZX62RD-AB-5P8-Miscellaneous-AMC_FMC_Carrier-PcbDoc-rescue
- U21: symbol AMC_FMC_Carrier-PcbDoc-rescue:M93C46-WMN6TP-Logic -> marble_misc:M93C46-WMN6TP-Logic
Changed lines of the file:
@@
 $EndDescr
 $Comp
-L AMC_FMC_Carrier-PcbDoc-rescue:HIROSE_ZX62RD-AB-5P8-Miscellaneous-AMC_FMC_Carrier-PcbDoc-rescue J10
+L marble_misc:HIROSE_ZX62RD-AB-5P8-Miscellaneous-AMC_FMC_Carrier-PcbDoc-rescue J10
 U 1 1 5BEB92E1
 P 1700 3500
@@
 $EndComp
 $Comp
-L AMC_FMC_Carrier-PcbDoc-rescue:+1V8_USB-powerMG-AMC_FMC_Carrier-PcbDoc-rescue #PWR0296
+L marble_misc:+1V8_USB-powerMG-AMC_FMC_Carrier-PcbDoc-rescue #PWR0296
 U 1 1 5BEBDA76
 P 5900 3250
@@
 	4050 7150 4350 7150
 $Comp
-L AMC_FMC_Carrier-PcbDoc-rescue:PRTR5V0U2X-Diodes D13
+L marble_misc:PRTR5V0U2X-Diodes D13
 U 1 1 5E04F663
 P 2400 5400
@@
 Connection ~ 4350 4700
 $Comp
-L AMC_FMC_Carrier-PcbDoc-rescue:M93C46-WMN6TP-Logic U21
+L marble_misc:M93C46-WMN6TP-Logic U21
 U 1 1 5C74B2C9
 P 3250 6850
@@
 $EndComp
 $Comp
-L AMC_FMC_Carrier-PcbDoc-rescue:+3V3_USB-AMC_FMC_Carrier-PcbDoc-rescue #PWR0275
+L marble_misc:+3V3_USB-AMC_FMC_Carrier-PcbDoc-rescue #PWR0275
 U 1 1 5E0639EB
 P 5900 1850
@@
 $EndComp
 $Comp
-L AMC_FMC_Carrier-PcbDoc-rescue:+3V3_USB-AMC_FMC_Carrier-PcbDoc-rescue #PWR0277
+L marble_misc:+3V3_USB-AMC_FMC_Carrier-PcbDoc-rescue #PWR0277
 U 1 1 5E0910B1
 P 6350 3300
@@
 $EndComp
 $Comp
-L AMC_FMC_Carrier-PcbDoc-rescue:+3V3_USB-AMC_FMC_Carrier-PcbDoc-rescue #PWR0279
+L marble_misc:+3V3_USB-AMC_FMC_Carrier-PcbDoc-rescue #PWR0279
 U 1 1 5E0AE015
 P 8300 2950
@@
 $EndComp
 $Comp
-L AMC_FMC_Carrier-PcbDoc-rescue:+3V3_USB-AMC_FMC_Carrier-PcbDoc-rescue #PWR0281
+L marble_misc:+3V3_USB-AMC_FMC_Carrier-PcbDoc-rescue #PWR0281
 U 1 1 5E0CAFF4
 P 11300 1500
@@
 $EndComp
 $Comp
-L AMC_FMC_Carrier-PcbDoc-rescue:+3V3_USB-AMC_FMC_Carrier-PcbDoc-rescue #PWR0282
+L marble_misc:+3V3_USB-AMC_FMC_Carrier-PcbDoc-rescue #PWR0282
 U 1 1 5E0E7F6F
 P 11550 2700
@@
 $EndComp
 $Comp
-L AMC_FMC_Carrier-PcbDoc-rescue:+3V3_USB-AMC_FMC_Carrier-PcbDoc-rescue #PWR0284
+L marble_misc:+3V3_USB-AMC_FMC_Carrier-PcbDoc-rescue #PWR0284
 U 1 1 5E1142BD
 P 11300 3450
@@
 $EndComp
 $Comp
-L AMC_FMC_Carrier-PcbDoc-rescue:+3V3_USB-AMC_FMC_Carrier-PcbDoc-rescue #PWR0285
+L marble_misc:+3V3_USB-AMC_FMC_Carrier-PcbDoc-rescue #PWR0285
 U 1 1 5E131666
 P 11300 2250
@@
 $EndComp
 $Comp
-L AMC_FMC_Carrier-PcbDoc-rescue:+3V3_USB-AMC_FMC_Carrier-PcbDoc-rescue #PWR0294
+L marble_misc:+3V3_USB-AMC_FMC_Carrier-PcbDoc-rescue #PWR0294
 U 1 1 5E14E7E2
 P 11300 4200
@@
 $EndComp
 $Comp
-L AMC_FMC_Carrier-PcbDoc-rescue:+3V3_USB-AMC_FMC_Carrier-PcbDoc-rescue #PWR0304
+L marble_misc:+3V3_USB-AMC_FMC_Carrier-PcbDoc-rescue #PWR0304
 U 1 1 5E16BA3D
 P 11550 4650
@@
 $EndComp
 $Comp
-L AMC_FMC_Carrier-PcbDoc-rescue:+3V3_USB-AMC_FMC_Carrier-PcbDoc-rescue #PWR0306
+L marble_misc:+3V3_USB-AMC_FMC_Carrier-PcbDoc-rescue #PWR0306
 U 1 1 5E1A590C
 P 13600 7250
@@
 $EndComp
 $Comp
-L AMC_FMC_Carrier-PcbDoc-rescue:+3V3_USB-AMC_FMC_Carrier-PcbDoc-rescue #PWR0307
+L marble_misc:+3V3_USB-AMC_FMC_Carrier-PcbDoc-rescue #PWR0307
 U 1 1 5E1B4270
 P 13250 6100
@@
 $EndComp
 $Comp
-L AMC_FMC_Carrier-PcbDoc-rescue:+3V3_USB-AMC_FMC_Carrier-PcbDoc-rescue #PWR0309
+L marble_misc:+3V3_USB-AMC_FMC_Carrier-PcbDoc-rescue #PWR0309
 U 1 1 5E1C2F5B
 P 13350 6800
@@
 	13250 6100 13400 6100
 $Comp
-L AMC_FMC_Carrier-PcbDoc-rescue:+3V3_USB-AMC_FMC_Carrier-PcbDoc-rescue #PWR0311
+L marble_misc:+3V3_USB-AMC_FMC_Carrier-PcbDoc-rescue #PWR0311
 U 1 1 5E1E0E93
 P 11300 7050
@@
 $EndComp
 $Comp
-L AMC_FMC_Carrier-PcbDoc-rescue:+3V3_USB-AMC_FMC_Carrier-PcbDoc-rescue #PWR0316
+L marble_misc:+3V3_USB-AMC_FMC_Carrier-PcbDoc-rescue #PWR0316
 U 1 1 5E20CA7E
 P 11300 7650
@@
 $EndComp
 $Comp
-L AMC_FMC_Carrier-PcbDoc-rescue:+3V3_USB-AMC_FMC_Carrier-PcbDoc-rescue #PWR0319
+L marble_misc:+3V3_USB-AMC_FMC_Carrier-PcbDoc-rescue #PWR0319
 U 1 1 5E24786F
 P 10050 8150
@@
 $EndComp
 $Comp
-L AMC_FMC_Carrier-PcbDoc-rescue:+3V3_USB-AMC_FMC_Carrier-PcbDoc-rescue #PWR0325
+L marble_misc:+3V3_USB-AMC_FMC_Carrier-PcbDoc-rescue #PWR0325
 U 1 1 5E28111D
 P 10000 8850
@@
 $EndComp
 $Comp
-L AMC_FMC_Carrier-PcbDoc-rescue:+3V3_USB-AMC_FMC_Carrier-PcbDoc-rescue #PWR0327
+L marble_misc:+3V3_USB-AMC_FMC_Carrier-PcbDoc-rescue #PWR0327
 U 1 1 5E29D842
 P 7200 8950
@@
 $EndComp
 $Comp
-L AMC_FMC_Carrier-PcbDoc-rescue:+3V3_USB-AMC_FMC_Carrier-PcbDoc-rescue #PWR0328
+L marble_misc:+3V3_USB-AMC_FMC_Carrier-PcbDoc-rescue #PWR0328
 U 1 1 5E2AB899
 P 7200 9050
@@
 $EndComp
 $Comp
-L AMC_FMC_Carrier-PcbDoc-rescue:+3V3_USB-AMC_FMC_Carrier-PcbDoc-rescue #PWR0330
+L marble_misc:+3V3_USB-AMC_FMC_Carrier-PcbDoc-rescue #PWR0330
 U 1 1 5E2C78AB
 P 7250 9650
@@
 $EndComp
 $Comp
-L AMC_FMC_Carrier-PcbDoc-rescue:+3V3_USB-AMC_FMC_Carrier-PcbDoc-rescue #PWR0332
+L marble_misc:+3V3_USB-AMC_FMC_Carrier-PcbDoc-rescue #PWR0332
 U 1 1 5E2E3981
 P 11550 8100
@@
 $EndComp
 $Comp
-L AMC_FMC_Carrier-PcbDoc-rescue:+3V3_USB-AMC_FMC_Carrier-PcbDoc-rescue #PWR0335
+L marble_misc:+3V3_USB-AMC_FMC_Carrier-PcbDoc-rescue #PWR0335
 U 1 1 5E30DBBE
 P 10250 9300
@@
 $EndComp
 $Comp
-L AMC_FMC_Carrier-PcbDoc-rescue:+3V3_USB-AMC_FMC_Carrier-PcbDoc-rescue #PWR0337
+L marble_misc:+3V3_USB-AMC_FMC_Carrier-PcbDoc-rescue #PWR0337
 U 1 1 5E329CA2
 P 7000 10100
@@
 $EndComp
 $Comp
-L AMC_FMC_Carrier-PcbDoc-rescue:+3V3_USB-AMC_FMC_Carrier-PcbDoc-rescue #PWR0339
+L marble_misc:+3V3_USB-AMC_FMC_Carrier-PcbDoc-rescue #PWR0339
 U 1 1 5E345D17
 P 5200 8000
@@
 Connection ~ 5200 8000
 $Comp
-L AMC_FMC_Carrier-PcbDoc-rescue:+3V3_USB-AMC_FMC_Carrier-PcbDoc-rescue #PWR0341
+L marble_misc:+3V3_USB-AMC_FMC_Carrier-PcbDoc-rescue #PWR0341
 U 1 1 5E37DE16
 P 5200 7200
@@
 $EndComp
 $Comp
-L AMC_FMC_Carrier-PcbDoc-rescue:+3V3_USB-AMC_FMC_Carrier-PcbDoc-rescue #PWR0343
+L marble_misc:+3V3_USB-AMC_FMC_Carrier-PcbDoc-rescue #PWR0343
 U 1 1 5E399F01
 P 4900 6500
@@
 $EndComp
 $Comp
-L AMC_FMC_Carrier-PcbDoc-rescue:+3V3_USB-AMC_FMC_Carrier-PcbDoc-rescue #PWR0478
+L marble_misc:+3V3_USB-AMC_FMC_Carrier-PcbDoc-rescue #PWR0478
 U 1 1 5E3B5F64
 P 4900 5800
@@
 $EndComp
 $Comp
-L AMC_FMC_Carrier-PcbDoc-rescue:+3V3_USB-AMC_FMC_Carrier-PcbDoc-rescue #PWR0479
+L marble_misc:+3V3_USB-AMC_FMC_Carrier-PcbDoc-rescue #PWR0479
 U 1 1 5E3DFF47
 P 4050 6550
@@
 $EndComp
 $Comp
-L AMC_FMC_Carrier-PcbDoc-rescue:+3V3_USB-AMC_FMC_Carrier-PcbDoc-rescue #PWR0480
+L marble_misc:+3V3_USB-AMC_FMC_Carrier-PcbDoc-rescue #PWR0480
 U 1 1 5E3EE00F
 P 3450 6200
@@
 $EndComp
 $Comp
-L AMC_FMC_Carrier-PcbDoc-rescue:+3V3_USB-AMC_FMC_Carrier-PcbDoc-rescue #PWR0599
+L marble_misc:+3V3_USB-AMC_FMC_Carrier-PcbDoc-rescue #PWR0599
 U 1 1 5E40A0AB
 P 3650 7250
@@
 $EndComp
 $Comp
-L AMC_FMC_Carrier-PcbDoc-rescue:+3V3_USB-AMC_FMC_Carrier-PcbDoc-rescue #PWR0601
+L marble_misc:+3V3_USB-AMC_FMC_Carrier-PcbDoc-rescue #PWR0601
 U 1 1 5E4346A3
 P 8000 8800
@@
 Connection ~ 6000 9450
 $Comp
-L AMC_FMC_Carrier-PcbDoc-rescue:+3V3_USB-AMC_FMC_Carrier-PcbDoc-rescue #PWR0643
+L marble_misc:+3V3_USB-AMC_FMC_Carrier-PcbDoc-rescue #PWR0643
 U 1 1 5CE79DFD
 P 5150 9500
@@
 Connection ~ 5150 10550
 $Comp
-L AMC_FMC_Carrier-PcbDoc-rescue:+3V3_USB-AMC_FMC_Carrier-PcbDoc-rescue #PWR0645
+L marble_misc:+3V3_USB-AMC_FMC_Carrier-PcbDoc-rescue #PWR0645
 U 1 1 5D07178D
 P 5700 10550
