File: USB.sch (KiCad schematic (older format))
At the start: 74 parts, among them J10 10103594-0001LF, Q14 BSS138LT1G, Q18 BSS138LT1G, Q24 BSS138LT1G, Q6 BSS138LT1G, U15 SN74AVC2T245RSWR, U21 M93C46-WMN6TP, U22 TLV62565DBVT, U23 FT4232H-56Q, U24 SN74AVC2T245RSWR, U25 SN74AVC2T245RSWR, U26 SN74AVC2T245RSWR, U33 SN74AVC2T245RSWR, U38 SN74AVC2T245RSWR, Y4 XTAL_12MHZ_TXC_7M-12.000MAAJ-T

Commit message: Strip extraneous AMC_FMC_Carrier-PcbDoc-rescue and powerMG from symbol names
Parts:
- J10: symbol marble_misc:HIROSE_ZX62RD-AB-5P8-Miscellaneous-AMC_FMC_Carrier-PcbDoc-rescue -> marble_misc:HIROSE_ZX62RD-AB-5P8-Miscellaneous
Changed lines of the file:
@@
 $EndDescr
 $Comp
-L marble_misc:HIROSE_ZX62RD-AB-5P8-Miscellaneous-AMC_FMC_Carrier-PcbDoc-rescue J10
+L marble_misc:HIROSE_ZX62RD-AB-5P8-Miscellaneous J10
 U 1 1 5BEB92E1
 P 1700 3500
@@
 $EndComp
 $Comp
-L marble_misc:+1V8_USB-powerMG-AMC_FMC_Carrier-PcbDoc-rescue #PWR0296
+L marble_misc:+1V8_USB #PWR0296
 U 1 1 5BEBDA76
 P 5900 3250
@@
 $EndComp
 $Comp
-L marble_misc:+3V3_USB-AMC_FMC_Carrier-PcbDoc-rescue #PWR0275
+L marble_misc:+3V3_USB #PWR0275
 U 1 1 5E0639EB
 P 5900 1850
@@
 $EndComp
 $Comp
-L marble_misc:+3V3_USB-AMC_FMC_Carrier-PcbDoc-rescue #PWR0277
+L marble_misc:+3V3_USB #PWR0277
 U 1 1 5E0910B1
 P 6350 3300
@@
 $EndComp
 $Comp
-L marble_misc:+3V3_USB-AMC_FMC_Carrier-PcbDoc-rescue #PWR0279
+L marble_misc:+3V3_USB #PWR0279
 U 1 1 5E0AE015
 P 8300 2950
@@
 $EndComp
 $Comp
-L marble_misc:+3V3_USB-AMC_FMC_Carrier-PcbDoc-rescue #PWR0281
+L marble_misc:+3V3_USB #PWR0281
 U 1 1 5E0CAFF4
 P 11300 1500
@@
 $EndComp
 $Comp
-L marble_misc:+3V3_USB-AMC_FMC_Carrier-PcbDoc-rescue #PWR0282
+L marble_misc:+3V3_USB #PWR0282
 U 1 1 5E0E7F6F
 P 11550 2700
@@
 $EndComp
 $Comp
-L marble_misc:+3V3_USB-AMC_FMC_Carrier-PcbDoc-rescue #PWR0284
+L marble_misc:+3V3_USB #PWR0284
 U 1 1 5E1142BD
 P 11300 3450
@@
 $EndComp
 $Comp
-L marble_misc:+3V3_USB-AMC_FMC_Carrier-PcbDoc-rescue #PWR0285
+L marble_misc:+3V3_USB #PWR0285
 U 1 1 5E131666
 P 11300 2250
@@
 $EndComp
 $Comp
-L marble_misc:+3V3_USB-AMC_FMC_Carrier-PcbDoc-rescue #PWR0294
+L marble_misc:+3V3_USB #PWR0294
 U 1 1 5E14E7E2
 P 11300 4200
@@
 $EndComp
 $Comp
-L marble_misc:+3V3_USB-AMC_FMC_Carrier-PcbDoc-rescue #PWR0304
+L marble_misc:+3V3_USB #PWR0304
 U 1 1 5E16BA3D
 P 11550 4650
@@
 $EndComp
 $Comp
-L marble_misc:+3V3_USB-AMC_FMC_Carrier-PcbDoc-rescue #PWR0306
+L marble_misc:+3V3_USB #PWR0306
 U 1 1 5E1A590C
 P 13600 7250
@@
 $EndComp
 $Comp
-L marble_misc:+3V3_USB-AMC_FMC_Carrier-PcbDoc-rescue #PWR0307
+L marble_misc:+3V3_USB #PWR0307
 U 1 1 5E1B4270
 P 13250 6100
@@
 $EndComp
 $Comp
-L marble_misc:+3V3_USB-AMC_FMC_Carrier-PcbDoc-rescue #PWR0309
+L marble_misc:+3V3_USB #PWR0309
 U 1 1 5E1C2F5B
 P 13350 6800
@@
 	13250 6100 13400 6100
 $Comp
-L marble_misc:+3V3_USB-AMC_FMC_Carrier-PcbDoc-rescue #PWR0311
+L marble_misc:+3V3_USB #PWR0311
 U 1 1 5E1E0E93
 P 11300 7050
@@
 $EndComp
 $Comp
-L marble_misc:+3V3_USB-AMC_FMC_Carrier-PcbDoc-rescue #PWR0316
+L marble_misc:+3V3_USB #PWR0316
 U 1 1 5E20CA7E
 P 11300 7650
@@
 $EndComp
 $Comp
-L marble_misc:+3V3_USB-AMC_FMC_Carrier-PcbDoc-rescue #PWR0319
+L marble_misc:+3V3_USB #PWR0319
 U 1 1 5E24786F
 P 10050 8150
@@
 $EndComp
 $Comp
-L marble_misc:+3V3_USB-AMC_FMC_Carrier-PcbDoc-rescue #PWR0325
+L marble_misc:+3V3_USB #PWR0325
 U 1 1 5E28111D
 P 10000 8850
@@
 $EndComp
 $Comp
-L marble_misc:+3V3_USB-AMC_FMC_Carrier-PcbDoc-rescue #PWR0327
+L marble_misc:+3V3_USB #PWR0327
 U 1 1 5E29D842
 P 7200 8950
@@
 $EndComp
 $Comp
-L marble_misc:+3V3_USB-AMC_FMC_Carrier-PcbDoc-rescue #PWR0328
+L marble_misc:+3V3_USB #PWR0328
 U 1 1 5E2AB899
 P 7200 9050
@@
 $EndComp
 $Comp
-L marble_misc:+3V3_USB-AMC_FMC_Carrier-PcbDoc-rescue #PWR0330
+L marble_misc:+3V3_USB #PWR0330
 U 1 1 5E2C78AB
 P 7250 9650
@@
 $EndComp
 $Comp
-L marble_misc:+3V3_USB-AMC_FMC_Carrier-PcbDoc-rescue #PWR0332
+L marble_misc:+3V3_USB #PWR0332
 U 1 1 5E2E3981
 P 11550 8100
@@
 $EndComp
 $Comp
-L marble_misc:+3V3_USB-AMC_FMC_Carrier-PcbDoc-rescue #PWR0335
+L marble_misc:+3V3_USB #PWR0335
 U 1 1 5E30DBBE
 P 10250 9300
@@
 $EndComp
 $Comp
-L marble_misc:+3V3_USB-AMC_FMC_Carrier-PcbDoc-rescue #PWR0337
+L marble_misc:+3V3_USB #PWR0337
 U 1 1 5E329CA2
 P 7000 10100
@@
 $EndComp
 $Comp
-L marble_misc:+3V3_USB-AMC_FMC_Carrier-PcbDoc-rescue #PWR0339
+L marble_misc:+3V3_USB #PWR0339
 U 1 1 5E345D17
 P 5200 8000
@@
 Connection ~ 5200 8000
 $Comp
-L marble_misc:+3V3_USB-AMC_FMC_Carrier-PcbDoc-rescue #PWR0341
+L marble_misc:+3V3_USB #PWR0341
 U 1 1 5E37DE16
 P 5200 7200
@@
 $EndComp
 $Comp
-L marble_misc:+3V3_USB-AMC_FMC_Carrier-PcbDoc-rescue #PWR0343
+L marble_misc:+3V3_USB #PWR0343
 U 1 1 5E399F01
 P 4900 6500
@@
 $EndComp
 $Comp
-L marble_misc:+3V3_USB-AMC_FMC_Carrier-PcbDoc-rescue #PWR0478
+L marble_misc:+3V3_USB #PWR0478
 U 1 1 5E3B5F64
 P 4900 5800
@@
 $EndComp
 $Comp
-L marble_misc:+3V3_USB-AMC_FMC_Carrier-PcbDoc-rescue #PWR0479
+L marble_misc:+3V3_USB #PWR0479
 U 1 1 5E3DFF47
 P 4050 6550
@@
 $EndComp
 $Comp
-L marble_misc:+3V3_USB-AMC_FMC_Carrier-PcbDoc-rescue #PWR0480
+L marble_misc:+3V3_USB #PWR0480
 U 1 1 5E3EE00F
 P 3450 6200
@@
 $EndComp
 $Comp
-L marble_misc:+3V3_USB-AMC_FMC_Carrier-PcbDoc-rescue #PWR0599
+L marble_misc:+3V3_USB #PWR0599
 U 1 1 5E40A0AB
 P 3650 7250
@@
 $EndComp
 $Comp
-L marble_misc:+3V3_USB-AMC_FMC_Carrier-PcbDoc-rescue #PWR0601
+L marble_misc:+3V3_USB #PWR0601
 U 1 1 5E4346A3
 P 8000 8800
@@
 Connection ~ 6000 9450
 $Comp
-L marble_misc:+3V3_USB-AMC_FMC_Carrier-PcbDoc-rescue #PWR0643
+L marble_misc:+3V3_USB #PWR0643
 U 1 1 5CE79DFD
 P 5150 9500
@@
 Connection ~ 5150 10550
 $Comp
-L marble_misc:+3V3_USB-AMC_FMC_Carrier-PcbDoc-rescue #PWR0645
+L marble_misc:+3V3_USB #PWR0645
 U 1 1 5D07178D
 P 5700 10550
