File: USB.sch (KiCad schematic (older format))
At the start: 74 parts, among them J10 10103594-0001LF, Q14 BSS138LT1G, Q18 BSS138LT1G, Q24 BSS138LT1G, Q6 BSS138LT1G, U15 SN74AVC2T245RSWR, U21 M93C46-WMN6TP, U22 TLV62565DBVT, U23 FT4232H-56Q, U24 SN74AVC2T245RSWR, U25 SN74AVC2T245RSWR, U26 SN74AVC2T245RSWR, U33 SN74AVC2T245RSWR, U38 SN74AVC2T245RSWR, Y4 XTAL_12MHZ_TXC_7M-12.000MAAJ-T

Commit message: SCH: shave down ERC to 1 error, 0 warning
  * 1 unavoidable error due to the unpopulated crystal Y2
  * change many pin types in symbol libraries (also for FMC con.)
  * as a result, could remove some power flags
  * fix footrint attribute for SFP module symbols

for most devices (not voltage regulators):
  * vcc = power input
  * gnd = power input
  * gpios (also FMC lanes) = bidirectional
  * configuration pins (tied to vcc / gnd) = inputs
Changed lines of the file:
@@
-$Comp
-L power:PWR_FLAG #FLG?
-U 1 1 5D3ED707
-P 2500 3700
-AR Path="/5BABAC65/5D3ED707" Ref="#FLG?"  Part="1"
-AR Path="/5C16C03C/5D3ED707" Ref="#FLG0126"  Part="1"
-F 0 "#FLG0126" H 2500 3775 50  0001 C CNN
-F 1 "PWR_FLAG" H 2500 3873 50  0000 C CNN
-F 2 "" H 2500 3700 50  0001 C CNN
-F 3 "~" H 2500 3700 50  0001 C CNN
-	1    2500 3700
-	1    0    0    -1
-$EndComp
-Connection ~ 2500 3700
 $Comp
 L power:PWR_FLAG #FLG?

Commit message: SCH: rename +3.3VP, 3V3PM and +3V3MP to +3V3P
  * all of them refer to the same net
  * to make confusion perfect, all 3 power symbols on the schematic
    were an instance of the symbol `+3.3VP` with different
    value attributes
  * renamed the `+3.3VP` symbol to `+3V3P` for naming consistency
  * SCH: replaced all power symbols on the net by the new one
  * PCB: still needs to be synced up, as the net name has changed
Connections:
- net labels added: +3V3P
- net labels removed: +3V3MP
Changed lines of the file:
@@
 	7250 9150 7200 9150
 $Comp
-L power:+3.3VP #PWR0321
+L power:+3V3P #PWR0321
 U 1 1 5C2AA1F5
 P 5650 8850
@@
 AR Path="/5BCEDA39/5C2AA1F5" Ref="#PWR0321"  Part="1"
 F 0 "#PWR0321" H 5650 8700 50  0001 C CNN
-F 1 "+3V3MP" H 5665 9023 50  0000 C CNN
+F 1 "+3V3P" H 5665 9023 50  0000 C CNN
 F 2 "" H 5650 8850 50  0001 C CNN
 F 3 "" H 5650 8850 50  0001 C CNN
@@
 	10000 8950 10050 8950
 $Comp
-L power:+3.3VP #PWR0153
+L power:+3V3P #PWR0153
 U 1 1 5D36D9A1
 P 10800 1400
@@
 AR Path="/5D36D9A1" Ref="#PWR0153"  Part="1"
 F 0 "#PWR0153" H 10800 1250 50  0001 C CNN
-F 1 "+3V3MP" H 10815 1573 50  0000 C CNN
+F 1 "+3V3P" H 10815 1573 50  0000 C CNN
 F 2 "" H 10800 1400 50  0001 C CNN
 F 3 "" H 10800 1400 50  0001 C CNN
@@
 $EndComp
 $Comp
-L power:+3.3VP #PWR0226
+L power:+3V3P #PWR0226
 U 1 1 5D38A959
 P 6550 10100
@@
 AR Path="/5D38A959" Ref="#PWR0226"  Part="1"
 F 0 "#PWR0226" H 6550 9950 50  0001 C CNN
-F 1 "+3V3MP" H 6565 10273 50  0000 C CNN
+F 1 "+3V3P" H 6565 10273 50  0000 C CNN
 F 2 "" H 6550 10100 50  0001 C CNN
 F 3 "" H 6550 10100 50  0001 C CNN
@@
 $EndComp
 $Comp
-L power:+3.3VP #PWR0230
+L power:+3V3P #PWR0230
 U 1 1 5D3A7995
 P 10700 9300
@@
 AR Path="/5D3A7995" Ref="#PWR0230"  Part="1"
 F 0 "#PWR0230" H 10700 9150 50  0001 C CNN
-F 1 "+3V3MP" H 10715 9473 50  0000 C CNN
+F 1 "+3V3P" H 10715 9473 50  0000 C CNN
 F 2 "" H 10700 9300 50  0001 C CNN
 F 3 "" H 10700 9300 50  0001 C CNN
@@
 $EndComp
 $Comp
-L power:+3.3VP #PWR0310
+L power:+3V3P #PWR0310
 U 1 1 5D3C48CF
 P 7250 9750
@@
 AR Path="/5D3C48CF" Ref="#PWR0310"  Part="1"
 F 0 "#PWR0310" H 7250 9600 50  0001 C CNN
-F 1 "+3V3MP" V 7250 10000 50  0000 C CNN
+F 1 "+3V3P" V 7250 10000 50  0000 C CNN
 F 2 "" H 7250 9750 50  0001 C CNN
 F 3 "" H 7250 9750 50  0001 C CNN
@@
 $EndComp
 $Comp
-L power:+3.3VP #PWR0313
+L power:+3V3P #PWR0313
 U 1 1 5D41BA91
 P 10000 8950
@@
 AR Path="/5D41BA91" Ref="#PWR0313"  Part="1"
 F 0 "#PWR0313" H 10000 8800 50  0001 C CNN
-F 1 "+3V3MP" V 10000 9200 50  0000 C CNN
+F 1 "+3V3P" V 10000 9200 50  0000 C CNN
 F 2 "" H 10000 8950 50  0001 C CNN
 F 3 "" H 10000 8950 50  0001 C CNN
@@
 	5650 9200 5650 9350
 $Comp
-L power:+3.3VP #PWR0647
+L power:+3V3P #PWR0647
 U 1 1 5CDA74D2
 P 6000 8850
@@
 AR Path="/5BCEDA39/5CDA74D2" Ref="#PWR?"  Part="1"
 F 0 "#PWR0647" H 6000 8700 50  0001 C CNN
-F 1 "+3V3MP" H 6015 9023 50  0000 C CNN
+F 1 "+3V3P" H 6015 9023 50  0000 C CNN
 F 2 "" H 6000 8850 50  0001 C CNN
 F 3 "" H 6000 8850 50  0001 C CNN

Commit message: Add one more test point, on +3V3_USB
Parts:
- added TP11: TestPoint, Marble:TestPoint_Pad_D1.0mm, symbol Connector_Generic:TestPoint
Connections:
- wire segments 236 -> 238
Changed lines of the file:
@@
 Connection ~ 5000 1900
 Wire Wire Line
-	5000 1900 5450 1900
+	5000 1900 5250 1900
 Connection ~ 5000 2200
 Wire Wire Line
@@
 Wire Wire Line
 	2500 4300 2500 3700
+$Comp
+L Connector_Generic:TestPoint TP11
+U 1 1 5EC72E04
+P 5250 1800
+F 0 "TP11" H 5308 1918 50  0000 L CNN
+F 1 "TestPoint" H 5308 1827 50  0000 L CNN
+F 2 "Marble:TestPoint_Pad_D1.0mm" H 5450 1800 50  0001 C CNN
+F 3 "" H 5450 1800 50  0001 C CNN
+	1    5250 1800
+	1    0    0    -1
+$EndComp
+Wire Wire Line
+	5250 1800 5250 1900
+Connection ~ 5250 1900
+Wire Wire Line
+	5250 1900 5450 1900
 $EndSCHEMATC

Commit message: Convert all footprints to use Marble nickname
Includes both .sch and .lib files
Includes both bare footprint names and those with CERN-like nicknames
Parts:
- C162, C167, C168, C173, C360: footprint CAPC1709X95N -> Marble:CAPC1709X95N
- C163, C164, C166, C169, C170, C174, C175, C176, C177, C178, C179, C180, C181, C182, C183, C184, C185, C186, C187, C355, C356: footprint CAPC0603X33N -> Marble:CAPC0603X33N
- C165, C171: footprint CAPC1005X55N -> Marble:CAPC1005X55N
- C172: footprint CAPC1709X100N -> Marble:CAPC1709X100N
- D13: footprint SOT190P230X110-4N -> Marble:SOT190P230X110-4N
- D16: footprint ICs And Semiconductors SMD:SOD2512X110N -> Marble:SOD2512X110N
- J10: footprint Connector_USB:USB_Micro-B_Amphenol_10103594-0001LF_Horizontal -> Marble:USB_Micro-B_Amphenol_10103594-0001LF_Horizontal
- L10, L24, L25: footprint INDC1608X65N -> Marble:INDC1608X65N
- L23: footprint IND_WURTH_WE-PMCI_0806LR -> Marble:IND_WURTH_WE-PMCI_0806LR
- Q14, Q18, Q24, Q6: footprint ICs And Semiconductors SMD:SOT95P240X110-3N -> Marble:SOT95P240X110-3N
- R112, R113, R114, R115, R116, R117, R118, R119, R120, R121, R122, R123, R124, R125, R126, R127, R128, R200, R204, R269, R270, R271, R272, R273: footprint RESC1005X40N -> Marble:RESC1005X40N
- U15, U24, U25, U26, U33, U38: footprint ICs And Semiconductors SMD:QFN40P140X180X55-10N -> Marble:QFN40P140X180X55-10N
- U21: footprint ICs And Semiconductors SMD:SOIC127P600X175-8N -> Marble:SOIC127P600X175-8N
- U22: footprint ICs And Semiconductors SMD:SOT95P280X145-5N -> Marble:SOT95P280X145-5N
- U23: footprint ICs And Semiconductors SMD:QFN50P800X800X100-57N-S620 -> Marble:QFN50P800X800X100-57N-S620
- Y4: footprint ICs And Semiconductors SMD:XTAL_TXC_7M -> Marble:XTAL_TXC_7M

Commit message: Clean up BSS138 instances in schematic
Q5 Q6 Q8 Q9 Q14 Q17 Q18 Q19 Q20 Q21 Q24
Fewer warnings from KiBoM
Parts:
- Q14, Q18, Q24, Q6: HelpURL \\\\cern.ch\\dfs\\Applications\\Altium\\Datasheets\\BSS139.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 -> \\\\cern.ch\\dfs\\Applications\\Altium\\Datasheets\\BSS138L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
Changed lines of the file:
@@
 F 1 "BSS138LT1G" H 11369 5605 50  0000 L CNN
 F 2 "Marble:SOT95P240X110-3N" H 11050 4390 60  0001 L CNN
-F 3 "\\\\cern.ch\\dfs\\Applications\\Altium\\Datasheets\\BSS139.pdf" H 11050 5110 60  0001 L CNN
+F 3 "\\\\cern.ch\\dfs\\Applications\\Altium\\Datasheets\\BSS138LT1G.pdf" H 11050 5110 60  0001 L CNN
 F 4 "BSS138LT1G" H 11050 5020 60  0001 L CNN "Part Number"
 F 5 "N-MOSFET-D 1G 2S 3D" H 11050 4930 60  0001 L CNN "Library Ref"
@@
 F 27 "PcbLib\\ICs And Semiconductors SMD.PcbLib" H 11050 2860 60  0001 L CNN "Footprint Path"
 F 28 "SOT95P240X110-3N" H 11050 2770 60  0001 L CNN "Footprint Ref"
-F 29 "\\\\cern.ch\\dfs\\Applications\\Altium\\Datasheets\\BSS139.pdf" H 11050 2680 60  0001 L CNN "HelpURL"
+F 29 "\\\\cern.ch\\dfs\\Applications\\Altium\\Datasheets\\BSS138LT1G.pdf" H 11050 2680 60  0001 L CNN "HelpURL"
 F 30 "~~" H 11050 2590 60  0001 L CNN "ComponentLink1URL"
 F 31 " " H 11050 2500 60  0001 L CNN "ComponentLink1Description"
@@
 F 1 "BSS138LT1G" H 6169 9905 50  0000 L CNN
 F 2 "Marble:SOT95P240X110-3N" H 5850 8690 60  0001 L CNN
-F 3 "\\\\cern.ch\\dfs\\Applications\\Altium\\Datasheets\\BSS139.pdf" H 5850 9410 60  0001 L CNN
+F 3 "\\\\cern.ch\\dfs\\Applications\\Altium\\Datasheets\\BSS138LT1G.pdf" H 5850 9410 60  0001 L CNN
 F 4 "BSS138LT1G" H 5850 9320 60  0001 L CNN "Part Number"
 F 5 "N-MOSFET-D 1G 2S 3D" H 5850 9230 60  0001 L CNN "Library Ref"
@@
 F 27 "PcbLib\\ICs And Semiconductors SMD.PcbLib" H 5850 7160 60  0001 L CNN "Footprint Path"
 F 28 "SOT95P240X110-3N" H 5850 7070 60  0001 L CNN "Footprint Ref"
-F 29 "\\\\cern.ch\\dfs\\Applications\\Altium\\Datasheets\\BSS139.pdf" H 5850 6980 60  0001 L CNN "HelpURL"
+F 29 "\\\\cern.ch\\dfs\\Applications\\Altium\\Datasheets\\BSS138LT1G.pdf" H 5850 6980 60  0001 L CNN "HelpURL"
 F 30 "~~" H 5850 6890 60  0001 L CNN "ComponentLink1URL"
 F 31 " " H 5850 6800 60  0001 L CNN "ComponentLink1Description"
@@
 F 1 "BSS138LT1G" H 5019 10155 50  0000 L CNN
 F 2 "Marble:SOT95P240X110-3N" H 4700 8940 60  0001 L CNN
-F 3 "\\\\cern.ch\\dfs\\Applications\\Altium\\Datasheets\\BSS139.pdf" H 4700 9660 60  0001 L CNN
+F 3 "\\\\cern.ch\\dfs\\Applications\\Altium\\Datasheets\\BSS138LT1G.pdf" H 4700 9660 60  0001 L CNN
 F 4 "BSS138LT1G" H 4700 9570 60  0001 L CNN "Part Number"
 F 5 "N-MOSFET-D 1G 2S 3D" H 4700 9480 60  0001 L CNN "Library Ref"
@@
 F 27 "PcbLib\\ICs And Semiconductors SMD.PcbLib" H 4700 7410 60  0001 L CNN "Footprint Path"
 F 28 "SOT95P240X110-3N" H 4700 7320 60  0001 L CNN "Footprint Ref"
-F 29 "\\\\cern.ch\\dfs\\Applications\\Altium\\Datasheets\\BSS139.pdf" H 4700 7230 60  0001 L CNN "HelpURL"
+F 29 "\\\\cern.ch\\dfs\\Applications\\Altium\\Datasheets\\BSS138LT1G.pdf" H 4700 7230 60  0001 L CNN "HelpURL"
 F 30 "~~" H 4700 7140 60  0001 L CNN "ComponentLink1URL"
 F 31 " " H 4700 7050 60  0001 L CNN "ComponentLink1Description"
@@
 F 1 "BSS138LT1G" H 5019 10555 50  0000 L CNN
 F 2 "Marble:SOT95P240X110-3N" H 4700 9340 60  0001 L CNN
-F 3 "\\\\cern.ch\\dfs\\Applications\\Altium\\Datasheets\\BSS139.pdf" H 4700 10060 60  0001 L CNN
+F 3 "\\\\cern.ch\\dfs\\Applications\\Altium\\Datasheets\\BSS138LT1G.pdf" H 4700 10060 60  0001 L CNN
 F 4 "BSS138LT1G" H 4700 9970 60  0001 L CNN "Part Number"
 F 5 "N-MOSFET-D 1G 2S 3D" H 4700 9880 60  0001 L CNN "Library Ref"
@@
 F 27 "PcbLib\\ICs And Semiconductors SMD.PcbLib" H 4700 7810 60  0001 L CNN "Footprint Path"
 F 28 "SOT95P240X110-3N" H 4700 7720 60  0001 L CNN "Footprint Ref"
-F 29 "\\\\cern.ch\\dfs\\Applications\\Altium\\Datasheets\\BSS139.pdf" H 4700 7630 60  0001 L CNN "HelpURL"
+F 29 "\\\\cern.ch\\dfs\\Applications\\Altium\\Datasheets\\BSS138LT1G.pdf" H 4700 7630 60  0001 L CNN "HelpURL"
 F 30 "~~" H 4700 7540 60  0001 L CNN "ComponentLink1URL"
 F 31 " " H 4700 7450 60  0001 L CNN "ComponentLink1Description"

Commit message: Get rid of most .DbLib suffixes in Library Name attributes
Enough that KiBoM no longer complains about them
Parts:
- Q14, Q18, Q24, Q6: Library Name ICs And Semiconductors.DbLib -> ICs And Semiconductors SMD
Changed lines of the file:
@@
 F 35 "03/23/09 00:00:00" H 11050 2140 60  0001 L CNN "CreateDate"
 F 36 "03/23/09 00:00:00" H 11050 2050 60  0001 L CNN "LatestRevisionDate"
-F 37 "ICs And Semiconductors.DbLib" H 11050 1960 60  0001 L CNN "Library Name"
+F 37 "ICs And Semiconductors SMD" H 11050 1960 60  0001 L CNN "Library Name"
 F 38 "This work is licensed under the Creative Commons CC-BY-SA 4.0 License. To the extent that circuit schematics that use Licensed Material can be considered to be ‘Adapted Material’, then the copyright holder waives article 3.b of the license with respect to these schematics." H 11050 1870 60  0001 L CNN "License"
 F 39 "Transistors" H 11050 5600 50  0001 C CNN "Database Table Name"
@@
 F 35 "03/23/09 00:00:00" H 5850 6440 60  0001 L CNN "CreateDate"
 F 36 "03/23/09 00:00:00" H 5850 6350 60  0001 L CNN "LatestRevisionDate"
-F 37 "ICs And Semiconductors.DbLib" H 5850 6260 60  0001 L CNN "Library Name"
+F 37 "ICs And Semiconductors SMD" H 5850 6260 60  0001 L CNN "Library Name"
 F 38 "This work is licensed under the Creative Commons CC-BY-SA 4.0 License. To the extent that circuit schematics that use Licensed Material can be considered to be ‘Adapted Material’, then the copyright holder waives article 3.b of the license with respect to these schematics." H 5850 6170 60  0001 L CNN "License"
 F 39 "Transistors" H 5850 9900 50  0001 C CNN "Database Table Name"
@@
 F 35 "03/23/09 00:00:00" H 4700 6690 60  0001 L CNN "CreateDate"
 F 36 "03/23/09 00:00:00" H 4700 6600 60  0001 L CNN "LatestRevisionDate"
-F 37 "ICs And Semiconductors.DbLib" H 4700 6510 60  0001 L CNN "Library Name"
+F 37 "ICs And Semiconductors SMD" H 4700 6510 60  0001 L CNN "Library Name"
 F 38 "This work is licensed under the Creative Commons CC-BY-SA 4.0 License. To the extent that circuit schematics that use Licensed Material can be considered to be ‘Adapted Material’, then the copyright holder waives article 3.b of the license with respect to these schematics." H 4700 6420 60  0001 L CNN "License"
 F 39 "Transistors" H 4700 10150 50  0001 C CNN "Database Table Name"
@@
 F 35 "03/23/09 00:00:00" H 4700 7090 60  0001 L CNN "CreateDate"
 F 36 "03/23/09 00:00:00" H 4700 7000 60  0001 L CNN "LatestRevisionDate"
-F 37 "ICs And Semiconductors.DbLib" H 4700 6910 60  0001 L CNN "Library Name"
+F 37 "ICs And Semiconductors SMD" H 4700 6910 60  0001 L CNN "Library Name"
 F 38 "This work is licensed under the Creative Commons CC-BY-SA 4.0 License. To the extent that circuit schematics that use Licensed Material can be considered to be ‘Adapted Material’, then the copyright holder waives article 3.b of the license with respect to these schematics." H 4700 6820 60  0001 L CNN "License"
 F 39 "Transistors" H 4700 10550 50  0001 C CNN "Database Table Name"

Commit message: Get rid of "~" attribute in instances
This makes instances line up better with our library
Use a very short python program to rename "~" to "Val" and remove the old "Val".
Required a little pre-patch to correctly handle R297 R298 R299 R300 R162 R274 R197 R198, which had no "~" field.
No net changes to "Val" field contents.
Parts:
- C162, C167, C168, C173, C360: ~ 4.7uF -> (none)
- C163, C164, C166, C169, C170, C174, C175, C176, C177, C178, C179, C180, C181, C182, C183, C184, C185, C186, C187, C355, C356: ~ 100nF -> (none)
- C165, C171: ~ 22pF -> (none)
- C172: ~ 22uF -> (none)
- J10: Val (none) -> Micro-USB AB 2.0; ~ Micro-USB AB 2.0 -> (none)
- L10, L24, L25: ~ 120R@100MHz -> (none)
- L23: ~ 2.2uH -> (none)
- R112, R114, R119: ~ 2k2 -> (none)
- R113, R115, R116, R117, R118, R121, R122, R123, R124, R125, R126, R127, R204, R270, R271, R272: ~ 10k -> (none)
- R120: ~ 12k -> (none)
- R128, R273: ~ 47k -> (none)
- R200: ~ 0 -> (none)
- R269: ~ 82k -> (none)
- Y4: ~ 12MHz -> (none)
