File: Thermometers.sch (KiCad schematic (older format))
At the start: 22 parts, among them M1 Fan_3pin, M2 Fan_3pin, Q7 STS8DN6LF6AG, U27 MAX6639AEE+, U28 LM75AIMM/NOPB, U29 LM75AIMM/NOPB

Commit message: BOM updated, 25MHz clock level fixed
Parts:
- M1, M2: symbol AMC_FMC_Carrier-PcbDoc-rescue:Fan_3pin-Motor -> AMC_FMC_Carrier-PcbDoc-rescue:Fan_3pin-Motor-AMC_FMC_Carrier-PcbDoc-rescue
- Q7: symbol AMC_FMC_Carrier-PcbDoc-rescue:STS2DNE60-Transistor_FET -> AMC_FMC_Carrier-PcbDoc-rescue:STS2DNE60-Transistor_FET-AMC_FMC_Carrier-PcbDoc-rescue
- U28, U29: symbol AMC_FMC_Carrier-PcbDoc-rescue:LM75B-Sensor_Temperature -> AMC_FMC_Carrier-PcbDoc-rescue:LM75B-Sensor_Temperature-AMC_FMC_Carrier-PcbDoc-rescue
Changed lines of the file:
@@
 $EndDescr
 $Comp
-L AMC_FMC_Carrier-PcbDoc-rescue:LM75B-Sensor_Temperature U28
+L AMC_FMC_Carrier-PcbDoc-rescue:LM75B-Sensor_Temperature-AMC_FMC_Carrier-PcbDoc-rescue U28
 U 1 1 5D05AA1A
 P 6900 1850
@@
 	7500 1950 7300 1950
 $Comp
-L AMC_FMC_Carrier-PcbDoc-rescue:LM75B-Sensor_Temperature U29
+L AMC_FMC_Carrier-PcbDoc-rescue:LM75B-Sensor_Temperature-AMC_FMC_Carrier-PcbDoc-rescue U29
 U 1 1 5D05B2F7
 P 6900 3750
@@
 DXN_0
 $Comp
-L AMC_FMC_Carrier-PcbDoc-rescue:Fan_3pin-Motor M1
+L AMC_FMC_Carrier-PcbDoc-rescue:Fan_3pin-Motor-AMC_FMC_Carrier-PcbDoc-rescue M1
 U 1 1 5D543B40
 P 6800 5150
@@
 	2750 5200 2850 5200
 $Comp
-L AMC_FMC_Carrier-PcbDoc-rescue:STS2DNE60-Transistor_FET Q7
+L AMC_FMC_Carrier-PcbDoc-rescue:STS2DNE60-Transistor_FET-AMC_FMC_Carrier-PcbDoc-rescue Q7
 U 1 1 5D559F89
 P 6700 5750
@@
 $EndComp
 $Comp
-L AMC_FMC_Carrier-PcbDoc-rescue:STS2DNE60-Transistor_FET Q7
+L AMC_FMC_Carrier-PcbDoc-rescue:STS2DNE60-Transistor_FET-AMC_FMC_Carrier-PcbDoc-rescue Q7
 U 2 1 5D559FE8
 P 8300 5750
@@
 $EndComp
 $Comp
-L AMC_FMC_Carrier-PcbDoc-rescue:Fan_3pin-Motor M2
+L AMC_FMC_Carrier-PcbDoc-rescue:Fan_3pin-Motor-AMC_FMC_Carrier-PcbDoc-rescue M2
 U 1 1 5D632A5C
 P 8400 5150

Commit message: BOM configuration file edited, updated Marble picture, some components part number changed
Parts:
- M1, M2: Manufacturer Part Number (none) -> SWR25X-NRTC-S03-ST-BA
- Q7: Manufacturer Part Number (none) -> STS8DN6LF6AG; PN STS8DN6LF6AG -> (none)
- U28, U29: Manufacturer Part Number (none) -> LM75AIMM/NOPB; PN LM75AIMM/NOPB -> (none)
Changed lines of the file:
@@
 F 2 "ICs And Semiconductors SMD:SOP65P490X109-8N" H 6900 1850 50  0001 C CNN
 F 3 "http://www.ti.com/lit/ds/symlink/lm75b.pdf" H 6900 1850 50  0001 C CNN
-F 4 "LM75AIMM/NOPB" H 6900 1850 50  0001 C CNN "PN"
+F 4 "LM75AIMM/NOPB" H 6900 1850 50  0001 C CNN "Manufacturer Part Number"
 	1    6900 1850
 	1    0    0    -1
@@
 F 2 "ICs And Semiconductors SMD:SOP65P490X109-8N" H 6900 3750 50  0001 C CNN
 F 3 "http://www.ti.com/lit/ds/symlink/lm75b.pdf" H 6900 3750 50  0001 C CNN
-F 4 "LM75AIMM/NOPB" H 6900 3750 50  0001 C CNN "PN"
+F 4 "LM75AIMM/NOPB" H 6900 3750 50  0001 C CNN "Manufacturer Part Number"
 	1    6900 3750
 	1    0    0    -1
@@
 Text HLabel 1200 5100 0    50   Input ~ 10
 DXN_0
-$Comp
-L AMC_FMC_Carrier-PcbDoc-rescue:Fan_3pin-Motor-AMC_FMC_Carrier-PcbDoc-rescue M1
-U 1 1 5D543B40
-P 6800 5150
-F 0 "M1" H 6958 5146 50  0000 L CNN
-F 1 "Fan_3pin" H 6958 5055 50  0000 L CNN
-F 2 "Connect:Fan_Pin_Header_Straight_1x03" H 6800 5060 50  0001 C CNN
-F 3 "http://www.hardwarecanucks.com/forum/attachments/new-builds/16287d1330775095-help-chassis-power-fan-connectors-motherboard-asus_p8z68.jpg" H 6800 5060 50  0001 C CNN
-	1    6800 5150
-	1    0    0    -1
-$EndComp
 Wire Wire Line
 	2400 6000 2850 6000
@@
 F 2 "ICs And Semiconductors SMD:SOIC127P600X175-8N" H 6900 5675 50  0001 L CIN
 F 3 "www.st.com/resource/en/datasheet/CD00001537.pdf" H 6700 5750 50  0001 L CNN
-F 4 "STS8DN6LF6AG" H 6700 5750 50  0001 C CNN "PN"
+F 4 "STS8DN6LF6AG" H 6700 5750 50  0001 C CNN "Manufacturer Part Number"
 	1    6700 5750
 	1    0    0    -1
@@
 F 2 "ICs And Semiconductors SMD:SOIC127P600X175-8N" H 8500 5675 50  0001 L CIN
 F 3 "www.st.com/resource/en/datasheet/CD00001537.pdf" H 8300 5750 50  0001 L CNN
-F 4 "STS8DN6LF6AG" H 8300 5750 50  0001 C CNN "PN"
+F 4 "STS8DN6LF6AG" H 8300 5750 50  0001 C CNN "Manufacturer Part Number"
 	2    8300 5750
 	1    0    0    -1
@@
 F 2 "Connect:Fan_Pin_Header_Straight_1x03" H 8400 5060 50  0001 C CNN
 F 3 "http://www.hardwarecanucks.com/forum/attachments/new-builds/16287d1330775095-help-chassis-power-fan-connectors-motherboard-asus_p8z68.jpg" H 8400 5060 50  0001 C CNN
+F 4 "SWR25X-NRTC-S03-ST-BA" H 8400 5150 50  0001 C CNN "Manufacturer Part Number"
 	1    8400 5150
 	1    0    0    -1
@@
 Wire Wire Line
 	2750 5300 2850 5300
+$Comp
+L AMC_FMC_Carrier-PcbDoc-rescue:Fan_3pin-Motor-AMC_FMC_Carrier-PcbDoc-rescue M1
+U 1 1 5D543B40
+P 6800 5150
+F 0 "M1" H 6958 5146 50  0000 L CNN
+F 1 "Fan_3pin" H 6958 5055 50  0000 L CNN
+F 2 "Connect:Fan_Pin_Header_Straight_1x03" H 6800 5060 50  0001 C CNN
+F 3 "http://www.hardwarecanucks.com/forum/attachments/new-builds/16287d1330775095-help-chassis-power-fan-connectors-motherboard-asus_p8z68.jpg" H 6800 5060 50  0001 C CNN
+F 4 "SWR25X-NRTC-S03-ST-BA" H 6800 5150 50  0001 C CNN "Manufacturer Part Number"
+	1    6800 5150
+	1    0    0    -1
+$EndComp
 $EndSCHEMATC

Commit message: Rename library AMC_FMC_Carrier-PcbDoc-rescue as marble_misc
Parts:
- M1, M2: symbol AMC_FMC_Carrier-PcbDoc-rescue:Fan_3pin-Motor-AMC_FMC_Carrier-PcbDoc-rescue -> marble_misc:Fan_3pin-Motor-AMC_FMC_Carrier-PcbDoc-rescue
- Q7: symbol AMC_FMC_Carrier-PcbDoc-rescue:STS2DNE60-Transistor_FET-AMC_FMC_Carrier-PcbDoc-rescue -> marble_misc:STS2DNE60-Transistor_FET-AMC_FMC_Carrier-PcbDoc-rescue
- U28, U29: symbol AMC_FMC_Carrier-PcbDoc-rescue:LM75B-Sensor_Temperature-AMC_FMC_Carrier-PcbDoc-rescue -> marble_misc:LM75B-Sensor_Temperature-AMC_FMC_Carrier-PcbDoc-rescue
Changed lines of the file:
@@
 $EndDescr
 $Comp
-L AMC_FMC_Carrier-PcbDoc-rescue:LM75B-Sensor_Temperature-AMC_FMC_Carrier-PcbDoc-rescue U28
+L marble_misc:LM75B-Sensor_Temperature-AMC_FMC_Carrier-PcbDoc-rescue U28
 U 1 1 5D05AA1A
 P 6900 1850
@@
 	7500 1950 7300 1950
 $Comp
-L AMC_FMC_Carrier-PcbDoc-rescue:LM75B-Sensor_Temperature-AMC_FMC_Carrier-PcbDoc-rescue U29
+L marble_misc:LM75B-Sensor_Temperature-AMC_FMC_Carrier-PcbDoc-rescue U29
 U 1 1 5D05B2F7
 P 6900 3750
@@
 	2750 5200 2850 5200
 $Comp
-L AMC_FMC_Carrier-PcbDoc-rescue:STS2DNE60-Transistor_FET-AMC_FMC_Carrier-PcbDoc-rescue Q7
+L marble_misc:STS2DNE60-Transistor_FET-AMC_FMC_Carrier-PcbDoc-rescue Q7
 U 1 1 5D559F89
 P 6700 5750
@@
 $EndComp
 $Comp
-L AMC_FMC_Carrier-PcbDoc-rescue:STS2DNE60-Transistor_FET-AMC_FMC_Carrier-PcbDoc-rescue Q7
+L marble_misc:STS2DNE60-Transistor_FET-AMC_FMC_Carrier-PcbDoc-rescue Q7
 U 2 1 5D559FE8
 P 8300 5750
@@
 $EndComp
 $Comp
-L AMC_FMC_Carrier-PcbDoc-rescue:Fan_3pin-Motor-AMC_FMC_Carrier-PcbDoc-rescue M2
+L marble_misc:Fan_3pin-Motor-AMC_FMC_Carrier-PcbDoc-rescue M2
 U 1 1 5D632A5C
 P 8400 5150
@@
 	2750 5300 2850 5300
 $Comp
-L AMC_FMC_Carrier-PcbDoc-rescue:Fan_3pin-Motor-AMC_FMC_Carrier-PcbDoc-rescue M1
+L marble_misc:Fan_3pin-Motor-AMC_FMC_Carrier-PcbDoc-rescue M1
 U 1 1 5D543B40
 P 6800 5150

Commit message: Strip extraneous AMC_FMC_Carrier-PcbDoc-rescue and powerMG from symbol names
Parts:
- M1, M2: symbol marble_misc:Fan_3pin-Motor-AMC_FMC_Carrier-PcbDoc-rescue -> marble_misc:Fan_3pin-Motor
- Q7: symbol marble_misc:STS2DNE60-Transistor_FET-AMC_FMC_Carrier-PcbDoc-rescue -> marble_misc:STS2DNE60-Transistor_FET
- U28, U29: symbol marble_misc:LM75B-Sensor_Temperature-AMC_FMC_Carrier-PcbDoc-rescue -> marble_misc:LM75B-Sensor_Temperature
Changed lines of the file:
@@
 $EndDescr
 $Comp
-L marble_misc:LM75B-Sensor_Temperature-AMC_FMC_Carrier-PcbDoc-rescue U28
+L marble_misc:LM75B-Sensor_Temperature U28
 U 1 1 5D05AA1A
 P 6900 1850
@@
 	7500 1950 7300 1950
 $Comp
-L marble_misc:LM75B-Sensor_Temperature-AMC_FMC_Carrier-PcbDoc-rescue U29
+L marble_misc:LM75B-Sensor_Temperature U29
 U 1 1 5D05B2F7
 P 6900 3750
@@
 	2750 5200 2850 5200
 $Comp
-L marble_misc:STS2DNE60-Transistor_FET-AMC_FMC_Carrier-PcbDoc-rescue Q7
+L marble_misc:STS2DNE60-Transistor_FET Q7
 U 1 1 5D559F89
 P 6700 5750
@@
 $EndComp
 $Comp
-L marble_misc:STS2DNE60-Transistor_FET-AMC_FMC_Carrier-PcbDoc-rescue Q7
+L marble_misc:STS2DNE60-Transistor_FET Q7
 U 2 1 5D559FE8
 P 8300 5750
@@
 $EndComp
 $Comp
-L marble_misc:Fan_3pin-Motor-AMC_FMC_Carrier-PcbDoc-rescue M2
+L marble_misc:Fan_3pin-Motor M2
 U 1 1 5D632A5C
 P 8400 5150
@@
 	2750 5300 2850 5300
 $Comp
-L marble_misc:Fan_3pin-Motor-AMC_FMC_Carrier-PcbDoc-rescue M1
+L marble_misc:Fan_3pin-Motor M1
 U 1 1 5D543B40
 P 6800 5150
