File: Thermometers.sch (KiCad schematic (older format))
At the start: 22 parts, among them M1 Fan_3pin, M2 Fan_3pin, Q7 STS8DN6LF6AG, U27 MAX6639AEE+, U28 LM75AIMM/NOPB, U29 LM75AIMM/NOPB

Commit message: SCH: rename +3.3VP, 3V3PM and +3V3MP to +3V3P
  * all of them refer to the same net
  * to make confusion perfect, all 3 power symbols on the schematic
    were an instance of the symbol `+3.3VP` with different
    value attributes
  * renamed the `+3.3VP` symbol to `+3V3P` for naming consistency
  * SCH: replaced all power symbols on the net by the new one
  * PCB: still needs to be synced up, as the net name has changed
Connections:
- net labels added: +3V3P
- net labels removed: +3V3MP
Changed lines of the file:
@@
 $EndComp
 $Comp
-L power:+3.3VP #PWR?
+L power:+3V3P #PWR?
 U 1 1 5D05AEC2
 P 6900 1100
@@
 AR Path="/5D05AEC2" Ref="#PWR0358"  Part="1"
 F 0 "#PWR0358" H 6900 950 50  0001 C CNN
-F 1 "+3V3MP" H 6915 1273 50  0000 C CNN
+F 1 "+3V3P" H 6915 1273 50  0000 C CNN
 F 2 "" H 6900 1100 50  0001 C CNN
 F 3 "" H 6900 1100 50  0001 C CNN
@@
 $EndComp
 $Comp
-L power:+3.3VP #PWR?
+L power:+3V3P #PWR?
 U 1 1 5D05B18E
 P 7500 1750
@@
 AR Path="/5D05B18E" Ref="#PWR0364"  Part="1"
 F 0 "#PWR0364" H 7500 1600 50  0001 C CNN
-F 1 "+3V3MP" V 7500 2000 50  0000 C CNN
+F 1 "+3V3P" V 7500 2000 50  0000 C CNN
 F 2 "" H 7500 1750 50  0001 C CNN
 F 3 "" H 7500 1750 50  0001 C CNN
@@
 $EndComp
 $Comp
-L power:+3.3VP #PWR?
+L power:+3V3P #PWR?
 U 1 1 5D05B203
 P 7500 1850
@@
 AR Path="/5D05B203" Ref="#PWR0365"  Part="1"
 F 0 "#PWR0365" H 7500 1700 50  0001 C CNN
-F 1 "+3V3MP" V 7500 2100 50  0000 C CNN
+F 1 "+3V3P" V 7500 2100 50  0000 C CNN
 F 2 "" H 7500 1850 50  0001 C CNN
 F 3 "" H 7500 1850 50  0001 C CNN
@@
 $EndComp
 $Comp
-L power:+3.3VP #PWR?
+L power:+3V3P #PWR?
 U 1 1 5D05B306
 P 6900 3000
@@
 AR Path="/5D05B306" Ref="#PWR0360"  Part="1"
 F 0 "#PWR0360" H 6900 2850 50  0001 C CNN
-F 1 "+3V3MP" H 6915 3173 50  0000 C CNN
+F 1 "+3V3P" H 6915 3173 50  0000 C CNN
 F 2 "" H 6900 3000 50  0001 C CNN
 F 3 "" H 6900 3000 50  0001 C CNN
@@
 $EndComp
 $Comp
-L power:+3.3VP #PWR?
+L power:+3V3P #PWR?
 U 1 1 5D05B324
 P 7500 3650
@@
 AR Path="/5D05B324" Ref="#PWR0367"  Part="1"
 F 0 "#PWR0367" H 7500 3500 50  0001 C CNN
-F 1 "+3V3MP" V 7500 3900 50  0000 C CNN
+F 1 "+3V3P" V 7500 3900 50  0000 C CNN
 F 2 "" H 7500 3650 50  0001 C CNN
 F 3 "" H 7500 3650 50  0001 C CNN
@@
 Connection ~ 6300 1950
 $Comp
-L power:+3.3VP #PWR?
+L power:+3V3P #PWR?
 U 1 1 5D05D39D
 P 6300 1100
@@
 AR Path="/5D05D39D" Ref="#PWR0357"  Part="1"
 F 0 "#PWR0357" H 6300 950 50  0001 C CNN
-F 1 "+3V3MP" H 6315 1273 50  0000 C CNN
+F 1 "+3V3P" H 6315 1273 50  0000 C CNN
 F 2 "" H 6300 1100 50  0001 C CNN
 F 3 "" H 6300 1100 50  0001 C CNN
@@
 	6300 1100 6300 1200
 $Comp
-L power:+3.3VP #PWR?
+L power:+3V3P #PWR?
 U 1 1 5D0665E3
 P 2300 6000
@@
 AR Path="/5D0665E3" Ref="#PWR0356"  Part="1"
 F 0 "#PWR0356" H 2300 5850 50  0001 C CNN
-F 1 "+3V3MP" V 2300 6250 50  0000 C CNN
+F 1 "+3V3P" V 2300 6250 50  0000 C CNN
 F 2 "" H 2300 6000 50  0001 C CNN
 F 3 "" H 2300 6000 50  0001 C CNN
@@
 	4800 5100 4800 5200
 $Comp
-L power:+3.3VP #PWR?
+L power:+3V3P #PWR?
 U 1 1 5D57B1C9
 P 4800 4750
@@
 AR Path="/5D57B1C9" Ref="#PWR0507"  Part="1"
 F 0 "#PWR0507" H 4800 4600 50  0001 C CNN
-F 1 "+3V3MP" H 4800 4900 50  0000 C CNN
+F 1 "+3V3P" H 4800 4900 50  0000 C CNN
 F 2 "" H 4800 4750 50  0001 C CNN
 F 3 "" H 4800 4750 50  0001 C CNN
@@
 $EndComp
 $Comp
-L power:+3.3VP #PWR?
+L power:+3V3P #PWR?
 U 1 1 5D581F39
 P 5350 4750
@@
 AR Path="/5D581F39" Ref="#PWR0508"  Part="1"
 F 0 "#PWR0508" H 5350 4600 50  0001 C CNN
-F 1 "+3V3MP" H 5350 4900 50  0000 C CNN
+F 1 "+3V3P" H 5350 4900 50  0000 C CNN
 F 2 "" H 5350 4750 50  0001 C CNN
 F 3 "" H 5350 4750 50  0001 C CNN
@@
 Connection ~ 4600 6000
 $Comp
-L power:+3.3VP #PWR?
+L power:+3V3P #PWR?
 U 1 1 5D5D3DE2
 P 4200 4750
@@
 AR Path="/5D5D3DE2" Ref="#PWR0506"  Part="1"
 F 0 "#PWR0506" H 4200 4600 50  0001 C CNN
-F 1 "+3V3MP" H 4200 4900 50  0000 C CNN
+F 1 "+3V3P" H 4200 4900 50  0000 C CNN
 F 2 "" H 4200 4750 50  0001 C CNN
 F 3 "" H 4200 4750 50  0001 C CNN

Commit message: Convert all footprints to use Marble nickname
Includes both .sch and .lib files
Includes both bare footprint names and those with CERN-like nicknames
Parts:
- C188, C189: footprint CAPC1005X55N -> Marble:CAPC1005X55N
- C190, C191, C192: footprint CAPC0603X33N -> Marble:CAPC0603X33N
- C343, C344: footprint CAPC1709X95N -> Marble:CAPC1709X95N
- M1, M2: footprint Connect:Fan_Pin_Header_Straight_1x03 -> Marble:Fan_Pin_Header_Straight_1x03
- Q7: footprint ICs And Semiconductors SMD:SOIC127P600X175-8N -> Marble:SOIC127P600X175-8N
- R129, R130, R172, R173, R174, R175, R176, R177, R178: footprint RESC1005X40N -> Marble:RESC1005X40N
- U27: footprint ICs And Semiconductors SMD:SOP63P600X175-16N -> Marble:SOP63P600X175-16N
- U28, U29: footprint ICs And Semiconductors SMD:SOP65P490X109-8N -> Marble:SOP65P490X109-8N
Changed lines of the file:
@@
 F 0 "U28" H 6650 2300 50  0000 C CNN
 F 1 "LM75AIMM/NOPB" H 7250 1400 50  0000 C CNN
-F 2 "ICs And Semiconductors SMD:SOP65P490X109-8N" H 6900 1850 50  0001 C CNN
+F 2 "Marble:SOP65P490X109-8N" H 6900 1850 50  0001 C CNN
 F 3 "http://www.ti.com/lit/ds/symlink/lm75b.pdf" H 6900 1850 50  0001 C CNN
 F 4 "LM75AIMM/NOPB" H 6900 1850 50  0001 C CNN "Manufacturer Part Number"
@@
 F 0 "U29" H 6650 4200 50  0000 C CNN
 F 1 "LM75AIMM/NOPB" H 7250 3300 50  0000 C CNN
-F 2 "ICs And Semiconductors SMD:SOP65P490X109-8N" H 6900 3750 50  0001 C CNN
+F 2 "Marble:SOP65P490X109-8N" H 6900 3750 50  0001 C CNN
 F 3 "http://www.ti.com/lit/ds/symlink/lm75b.pdf" H 6900 3750 50  0001 C CNN
 F 4 "LM75AIMM/NOPB" H 6900 3750 50  0001 C CNN "Manufacturer Part Number"
@@
 F 0 "Q7" H 6906 5796 50  0000 L CNN
 F 1 "STS8DN6LF6AG" H 6906 5705 50  0000 L CNN
-F 2 "ICs And Semiconductors SMD:SOIC127P600X175-8N" H 6900 5675 50  0001 L CIN
+F 2 "Marble:SOIC127P600X175-8N" H 6900 5675 50  0001 L CIN
 F 3 "www.st.com/resource/en/datasheet/CD00001537.pdf" H 6700 5750 50  0001 L CNN
 F 4 "STS8DN6LF6AG" H 6700 5750 50  0001 C CNN "Manufacturer Part Number"
@@
 F 0 "Q7" H 8506 5796 50  0000 L CNN
 F 1 "STS8DN6LF6AG" H 8506 5705 50  0000 L CNN
-F 2 "ICs And Semiconductors SMD:SOIC127P600X175-8N" H 8500 5675 50  0001 L CIN
+F 2 "Marble:SOIC127P600X175-8N" H 8500 5675 50  0001 L CIN
 F 3 "www.st.com/resource/en/datasheet/CD00001537.pdf" H 8300 5750 50  0001 L CNN
 F 4 "STS8DN6LF6AG" H 8300 5750 50  0001 C CNN "Manufacturer Part Number"
@@
 F 0 "M2" H 8558 5146 50  0000 L CNN
 F 1 "Fan_3pin" H 8558 5055 50  0000 L CNN
-F 2 "Connect:Fan_Pin_Header_Straight_1x03" H 8400 5060 50  0001 C CNN
+F 2 "Marble:Fan_Pin_Header_Straight_1x03" H 8400 5060 50  0001 C CNN
 F 3 "http://www.hardwarecanucks.com/forum/attachments/new-builds/16287d1330775095-help-chassis-power-fan-connectors-motherboard-asus_p8z68.jpg" H 8400 5060 50  0001 C CNN
 F 4 "SWR25X-NRTC-S03-ST-BA" H 8400 5150 50  0001 C CNN "Manufacturer Part Number"
@@
 F 0 "U27" H 3450 5265 50  0000 C CNN
 F 1 "MAX6639AEE+" H 3450 5174 50  0000 C CNN
-F 2 "ICs And Semiconductors SMD:SOP63P600X175-16N" H 3050 2910 60  0001 L CNN
+F 2 "Marble:SOP63P600X175-16N" H 3050 2910 60  0001 L CNN
 F 3 "" H 3050 3630 60  0001 L CNN
 F 4 "MAX6639AEE+" H 3050 3540 60  0001 L CNN "Part Number"
@@
 F 0 "C343" V 9600 4900 50  0000 L CNN
 F 1 "CC0603_4.7UF_16V_10%_X5R" H 9550 4640 60  0001 L CNN
-F 2 "CAPC1709X95N" H 9550 3830 60  0001 L CNN
+F 2 "Marble:CAPC1709X95N" H 9550 3830 60  0001 L CNN
 F 3 "\\\\cern.ch\\dfs\\Applications\\Altium\\Datasheets\\CC0603_X7R_TAIYO-YUDEN_HIGH-VALUE.pdf" H 9550 4460 60  0001 L CNN
 F 4 "4.7uF" V 9800 4900 50  0000 L CNN "~"
@@
 F 0 "C344" V 10050 4900 50  0000 L CNN
 F 1 "CC0603_4.7UF_16V_10%_X5R" H 10000 4640 60  0001 L CNN
-F 2 "CAPC1709X95N" H 10000 3830 60  0001 L CNN
+F 2 "Marble:CAPC1709X95N" H 10000 3830 60  0001 L CNN
 F 3 "\\\\cern.ch\\dfs\\Applications\\Altium\\Datasheets\\CC0603_X7R_TAIYO-YUDEN_HIGH-VALUE.pdf" H 10000 4460 60  0001 L CNN
 F 4 "4.7uF" V 10250 4900 50  0000 L CNN "~"
@@
 F 0 "C188" V 2054 5110 50  0000 L CNN
 F 1 "CC0402_1NF_50V_10%_X7R" H 1950 4740 60  0001 L CNN
-F 2 "CAPC1005X55N" H 1950 3930 60  0001 L CNN
+F 2 "Marble:CAPC1005X55N" H 1950 3930 60  0001 L CNN
 F 3 "\\\\cern.ch\\dfs\\Applications\\Altium\\Datasheets\\CC0402_X7R_PHYCOMP.pdf" H 1950 4560 60  0001 L CNN
 F 4 "1nF" V 2145 5110 50  0000 L CNN "~"
@@
 F 0 "C189" V 2504 5110 50  0000 L CNN
 F 1 "CC0402_1NF_50V_10%_X7R" H 2400 4740 60  0001 L CNN
-F 2 "CAPC1005X55N" H 2400 3930 60  0001 L CNN
+F 2 "Marble:CAPC1005X55N" H 2400 3930 60  0001 L CNN
 F 3 "\\\\cern.ch\\dfs\\Applications\\Altium\\Datasheets\\CC0402_X7R_PHYCOMP.pdf" H 2400 4560 60  0001 L CNN
 F 4 "1nF" V 2595 5110 50  0000 L CNN "~"
@@
 F 0 "C190" V 2504 6160 50  0000 L CNN
 F 1 "CC0201_100NF_6.3V_10%_X5R" H 2400 5790 60  0001 L CNN
-F 2 "CAPC0603X33N" H 2400 4980 60  0001 L CNN
+F 2 "Marble:CAPC0603X33N" H 2400 4980 60  0001 L CNN
 F 3 "\\\\cern.ch\\dfs\\Applications\\Altium\\Datasheets\\CC0201_X5R_AVX.pdf" H 2400 5610 60  0001 L CNN
 F 4 "100nF" V 2595 6160 50  0000 L CNN "~"
@@
 F 0 "C192" H 7550 3100 50  0000 L CNN
 F 1 "CC0201_100NF_6.3V_10%_X5R" H 7300 2890 60  0001 L CNN
-F 2 "CAPC0603X33N" H 7300 2080 60  0001 L CNN
+F 2 "Marble:CAPC0603X33N" H 7300 2080 60  0001 L CNN
 F 3 "\\\\cern.ch\\dfs\\Applications\\Altium\\Datasheets\\CC0201_X5R_AVX.pdf" H 7300 2710 60  0001 L CNN
 F 4 "100nF" H 7150 3100 50  0000 L CNN "~"
@@
 F 0 "C191" H 7550 1200 50  0000 L CNN
 F 1 "CC0201_100NF_6.3V_10%_X5R" H 7300 990 60  0001 L CNN
-F 2 "CAPC0603X33N" H 7300 180 60  0001 L CNN
+F 2 "Marble:CAPC0603X33N" H 7300 180 60  0001 L CNN
 F 3 "\\\\cern.ch\\dfs\\Applications\\Altium\\Datasheets\\CC0201_X5R_AVX.pdf" H 7300 810 60  0001 L CNN
 F 4 "100nF" H 7150 1200 50  0000 L CNN "~"
@@
 F 0 "R130" H 4250 4900 50  0000 L CNN
 F 1 "R0402_10K_1%_0.0625W_100PPM" H 4200 4590 60  0001 L CNN
-F 2 "RESC1005X40N" H 4200 3780 60  0001 L CNN
+F 2 "Marble:RESC1005X40N" H 4200 3780 60  0001 L CNN
 F 3 "\\\\cern.ch\\dfs\\Applications\\Altium\\Datasheets\\R0402_Phycomp_RC0402.pdf" H 4200 4410 60  0001 L CNN
 F 4 "10k" V 4500 4800 50  0000 L CNN "~"
@@
 F 0 "R172" H 4450 4900 50  0000 L CNN
 F 1 "R0402_10K_1%_0.0625W_100PPM" H 4400 4590 60  0001 L CNN
-F 2 "RESC1005X40N" H 4400 3780 60  0001 L CNN
+F 2 "Marble:RESC1005X40N" H 4400 3780 60  0001 L CNN
 F 3 "\\\\cern.ch\\dfs\\Applications\\Altium\\Datasheets\\R0402_Phycomp_RC0402.pdf" H 4400 4410 60  0001 L CNN
 F 4 "10k" V 4700 4800 50  0000 L CNN "~"
@@
 F 0 "R173" H 4650 4900 50  0000 L CNN
 F 1 "R0402_10K_1%_0.0625W_100PPM" H 4600 4590 60  0001 L CNN
-F 2 "RESC1005X40N" H 4600 3780 60  0001 L CNN
+F 2 "Marble:RESC1005X40N" H 4600 3780 60  0001 L CNN
 F 3 "\\\\cern.ch\\dfs\\Applications\\Altium\\Datasheets\\R0402_Phycomp_RC0402.pdf" H 4600 4410 60  0001 L CNN
 F 4 "10k" V 4900 4800 50  0000 L CNN "~"
@@
 F 0 "R174" H 4850 4900 50  0000 L CNN
 F 1 "R0402_10K_1%_0.0625W_100PPM" H 4800 4590 60  0001 L CNN
-F 2 "RESC1005X40N" H 4800 3780 60  0001 L CNN
+F 2 "Marble:RESC1005X40N" H 4800 3780 60  0001 L CNN
 F 3 "\\\\cern.ch\\dfs\\Applications\\Altium\\Datasheets\\R0402_Phycomp_RC0402.pdf" H 4800 4410 60  0001 L CNN
 F 4 "10k" V 5100 4800 50  0000 L CNN "~"
@@
 F 0 "R175" H 5050 4900 50  0000 L CNN
 F 1 "R0402_10K_1%_0.0625W_100PPM" H 5000 4590 60  0001 L CNN
-F 2 "RESC1005X40N" H 5000 3780 60  0001 L CNN
+F 2 "Marble:RESC1005X40N" H 5000 3780 60  0001 L CNN
 F 3 "\\\\cern.ch\\dfs\\Applications\\Altium\\Datasheets\\R0402_Phycomp_RC0402.pdf" H 5000 4410 60  0001 L CNN
 F 4 "10k" V 5300 4800 50  0000 L CNN "~"
@@
 F 0 "R176" H 5400 4900 50  0000 L CNN
 F 1 "R0402_10K_1%_0.0625W_100PPM" H 5350 4590 60  0001 L CNN
-F 2 "RESC1005X40N" H 5350 3780 60  0001 L CNN
+F 2 "Marble:RESC1005X40N" H 5350 3780 60  0001 L CNN
 F 3 "\\\\cern.ch\\dfs\\Applications\\Altium\\Datasheets\\R0402_Phycomp_RC0402.pdf" H 5350 4410 60  0001 L CNN
 F 4 "10k" V 5650 4800 50  0000 L CNN "~"
@@
 F 0 "R177" H 5700 4900 50  0000 L CNN
 F 1 "R0402_10K_1%_0.0625W_100PPM" H 5650 4590 60  0001 L CNN
-F 2 "RESC1005X40N" H 5650 3780 60  0001 L CNN
+F 2 "Marble:RESC1005X40N" H 5650 3780 60  0001 L CNN
 F 3 "\\\\cern.ch\\dfs\\Applications\\Altium\\Datasheets\\R0402_Phycomp_RC0402.pdf" H 5650 4410 60  0001 L CNN
 F 4 "10k" V 5950 4800 50  0000 L CNN "~"
@@
 F 0 "R178" H 6350 1300 50  0000 L CNN
 F 1 "R0402_10K_1%_0.0625W_100PPM" H 6300 990 60  0001 L CNN
-F 2 "RESC1005X40N" H 6300 180 60  0001 L CNN
+F 2 "Marble:RESC1005X40N" H 6300 180 60  0001 L CNN
 F 3 "\\\\cern.ch\\dfs\\Applications\\Altium\\Datasheets\\R0402_Phycomp_RC0402.pdf" H 6300 810 60  0001 L CNN
 F 4 "10k" V 6600 1200 50  0000 L CNN "~"
@@
 F 0 "R129" H 1550 5497 50  0000 C CNN
 F 1 "R0402_0R_JUMPER" H 1400 5090 60  0001 L CNN
-F 2 "RESC1005X40N" H 1400 4280 60  0001 L CNN
+F 2 "Marble:RESC1005X40N" H 1400 4280 60  0001 L CNN
 F 3 "\\\\cern.ch\\dfs\\Applications\\Altium\\Datasheets\\R0402_Phycomp_RC0402.pdf" H 1400 4910 60  0001 L CNN
 F 4 "0" H 1550 5406 50  0000 C CNN "~"
@@
 F 0 "M1" H 6958 5146 50  0000 L CNN
 F 1 "Fan_3pin" H 6958 5055 50  0000 L CNN
-F 2 "Connect:Fan_Pin_Header_Straight_1x03" H 6800 5060 50  0001 C CNN
+F 2 "Marble:Fan_Pin_Header_Straight_1x03" H 6800 5060 50  0001 C CNN
 F 3 "http://www.hardwarecanucks.com/forum/attachments/new-builds/16287d1330775095-help-chassis-power-fan-connectors-motherboard-asus_p8z68.jpg" H 6800 5060 50  0001 C CNN
 F 4 "SWR25X-NRTC-S03-ST-BA" H 6800 5150 50  0001 C CNN "Manufacturer Part Number"

Commit message: Document location of LM75 thermometer chips
Other:
- note added: "Near front panel under FMC1"
- note added: "Nestled in with XRP7724 and\nits power transistors"
Changed lines of the file:
@@
 	1    0    0    -1
 $EndComp
+Text Notes 7600 3450 0    50   ~ 0
+Nestled in with XRP7724 and\nits power transistors
+Text Notes 7600 1550 0    50   ~ 0
+Near front panel under FMC1
 $EndSCHEMATC

Commit message: Get rid of "~" attribute in instances
This makes instances line up better with our library
Use a very short python program to rename "~" to "Val" and remove the old "Val".
Required a little pre-patch to correctly handle R297 R298 R299 R300 R162 R274 R197 R198, which had no "~" field.
No net changes to "Val" field contents.
Parts:
- C188, C189: ~ 1nF -> (none)
- C190, C191, C192: ~ 100nF -> (none)
- C343, C344: ~ 4.7uF -> (none)
- R129: ~ 0 -> (none)
- R130, R172, R173, R174, R175, R176, R177, R178: ~ 10k -> (none)
