File: SFP.sch (KiCad schematic (older format))
At the start: 27 parts, among them J4 TYCO_1367073-1, U4 74LVC2T45DC, U5 74LVC2T45DC

Commit message: Convert all footprints to use Marble nickname
Includes both .sch and .lib files
Includes both bare footprint names and those with CERN-like nicknames
Parts:
- C19, C23, C25, C26, C27, C28, C29, C30: footprint Capacitors SMD:CAPC0603X33N -> Marble:CAPC0603X33N
- C20, C22: footprint Capacitors SMD:CAPC1005X55N -> Marble:CAPC1005X55N
- C21, C24: footprint Capacitors SMD:CAPC1608X87N -> Marble:CAPC1608X87N
- CageBot1: footprint TYCO_6367034-1 -> Marble:TYCO_6367034-1
- CageTop1: footprint TYCO_6367035-1 -> Marble:TYCO_6367035-1
- J4: footprint TYCO_1367073-1 -> Marble:TYCO_1367073-1
- L1, L2: footprint Inductors SMD:INDC1608X65N -> Marble:INDC1608X65N
- R32, R33, R34, R35, R36, R37, R38, R39: footprint Resistors SMD:RESC1005X40N -> Marble:RESC1005X40N
- U4, U5: footprint kicad-libraries-master:VSSOP8 -> Marble:VSSOP8
Changed lines of the file:
@@
 F 0 "CageBot?" H 5000 4215 50  0000 C CNN
 F 1 "TYCO_6367034-1" H 4500 3060 60  0001 L CNN
-F 2 "TYCO_6367034-1" H 4500 2250 60  0001 L CNN
+F 2 "Marble:TYCO_6367034-1" H 4500 2250 60  0001 L CNN
 F 3 "\\\\cern.ch\\dfs\\Applications\\Altium\\Datasheets\\TYCO_6367034-1.pdf" H 4500 2880 60  0001 L CNN
 F 4 "SFP" H 5000 4124 50  0000 C CNN "~"
@@
 F 0 "J?" H 5000 2015 50  0000 C CNN
 F 1 "TYCO_1367073-1" H 4500 -140 60  0001 L CNN
-F 2 "TYCO_1367073-1" H 4500 -950 60  0001 L CNN
+F 2 "Marble:TYCO_1367073-1" H 4500 -950 60  0001 L CNN
 F 3 "\\\\cern.ch\\dfs\\Applications\\Altium\\Datasheets\\TYCO_1367073-1.pdf" H 4500 -320 60  0001 L CNN
 F 4 "SFP" H 5000 1924 50  0000 C CNN "~"
@@
 F 0 "CageTop?" H 5528 746 50  0000 L CNN
 F 1 "TYCO_6367035-1" H 4500 310 60  0001 L CNN
-F 2 "TYCO_6367035-1" H 4500 -500 60  0001 L CNN
+F 2 "Marble:TYCO_6367035-1" H 4500 -500 60  0001 L CNN
 F 3 "\\\\cern.ch\\dfs\\Applications\\Altium\\Datasheets\\TYCO_6367035-1.pdf" H 4500 130 60  0001 L CNN
 F 4 "SFP" H 5528 655 50  0000 L CNN "~"
@@
 F 0 "C?" H 1715 2146 50  0000 L CNN
 F 1 "1uF" H 1715 2055 50  0000 L CNN
-F 2 "Capacitors SMD:CAPC1005X55N" H 1638 1950 50  0001 C CNN
+F 2 "Marble:CAPC1005X55N" H 1638 1950 50  0001 C CNN
 F 3 "~" H 1600 2100 50  0001 C CNN
 F 4 "CC0402_1UF_16V_10%_X5R" H 1600 2100 50  0001 C CNN "PN"
@@
 F 0 "C?" H 1265 2146 50  0000 L CNN
 F 1 "100nF" H 1265 2055 50  0000 L CNN
-F 2 "Capacitors SMD:CAPC0603X33N" H 1188 1950 50  0001 C CNN
+F 2 "Marble:CAPC0603X33N" H 1188 1950 50  0001 C CNN
 F 3 "~" H 1150 2100 50  0001 C CNN
 F 4 "CC0201_100NF_6.3V_10%_X5R" H 1265 2009 50  0001 L CNN "PN"
@@
 F 0 "C?" H 2415 2146 50  0000 L CNN
 F 1 "10uF" H 2415 2055 50  0000 L CNN
-F 2 "Capacitors SMD:CAPC1608X87N" H 2338 1950 50  0001 C CNN
+F 2 "Marble:CAPC1608X87N" H 2338 1950 50  0001 C CNN
 F 3 "~" H 2300 2100 50  0001 C CNN
 F 4 "CC0603_10uF_6.3V_20%_X5R" H 2415 2009 50  0001 L CNN "PN"
@@
 F 0 "L?" V 2190 1950 50  0000 C CNN
 F 1 "120R@100MHz" V 2099 1950 50  0000 C CNN
-F 2 "Inductors SMD:INDC1608X65N" H 2000 1950 50  0001 C CNN
+F 2 "Marble:INDC1608X65N" H 2000 1950 50  0001 C CNN
 F 3 "~" H 2000 1950 50  0001 C CNN
 F 4 "IND0603_MURATA_BLM18SG121TN1D" V 2000 1950 50  0001 C CNN "PN"
@@
 F 0 "C?" H 2815 2146 50  0000 L CNN
 F 1 "1uF" H 2815 2055 50  0000 L CNN
-F 2 "Capacitors SMD:CAPC1005X55N" H 2738 1950 50  0001 C CNN
+F 2 "Marble:CAPC1005X55N" H 2738 1950 50  0001 C CNN
 F 3 "~" H 2700 2100 50  0001 C CNN
 F 4 "CC0402_1UF_16V_10%_X5R" H 2700 2100 50  0001 C CNN "PN"
@@
 F 0 "C?" H 3165 2146 50  0000 L CNN
 F 1 "100nF" H 3165 2055 50  0000 L CNN
-F 2 "Capacitors SMD:CAPC0603X33N" H 3088 1950 50  0001 C CNN
+F 2 "Marble:CAPC0603X33N" H 3088 1950 50  0001 C CNN
 F 3 "~" H 3050 2100 50  0001 C CNN
 F 4 "CC0201_100NF_6.3V_10%_X5R" H 3165 2009 50  0001 L CNN "PN"
@@
 F 0 "C?" H 3615 2146 50  0000 L CNN
 F 1 "100nF" H 3615 2055 50  0000 L CNN
-F 2 "Capacitors SMD:CAPC0603X33N" H 3538 1950 50  0001 C CNN
+F 2 "Marble:CAPC0603X33N" H 3538 1950 50  0001 C CNN
 F 3 "~" H 3500 2100 50  0001 C CNN
 F 4 "CC0201_100NF_6.3V_10%_X5R" H 3615 2009 50  0001 L CNN "PN"
@@
 F 0 "R?" V 3493 2500 50  0000 C CNN
 F 1 "10k" V 3584 2500 50  0000 C CNN
-F 2 "Resistors SMD:RESC1005X40N" V 3630 2500 50  0001 C CNN
+F 2 "Marble:RESC1005X40N" V 3630 2500 50  0001 C CNN
 F 3 "~" H 3700 2500 50  0001 C CNN
 F 4 "R0402_10K_1%_0.0625W_100PPM" V 3700 2500 50  0001 C CNN "PN"
@@
 F 0 "L?" V 3440 2950 50  0000 C CNN
 F 1 "120R@100MHz" V 3349 2950 50  0000 C CNN
-F 2 "Inductors SMD:INDC1608X65N" H 3250 2950 50  0001 C CNN
+F 2 "Marble:INDC1608X65N" H 3250 2950 50  0001 C CNN
 F 3 "~" H 3250 2950 50  0001 C CNN
 F 4 "IND0603_MURATA_BLM18SG121TN1D" V 3250 2950 50  0001 C CNN "PN"
@@
 F 0 "C?" H 3565 3146 50  0000 L CNN
 F 1 "10uF" H 3565 3055 50  0000 L CNN
-F 2 "Capacitors SMD:CAPC1608X87N" H 3488 2950 50  0001 C CNN
+F 2 "Marble:CAPC1608X87N" H 3488 2950 50  0001 C CNN
 F 3 "~" H 3450 3100 50  0001 C CNN
 F 4 "CC0603_10uF_6.3V_20%_X5R" H 3565 3009 50  0001 L CNN "PN"
@@
 F 0 "C?" H 3965 3146 50  0000 L CNN
 F 1 "100nF" H 3965 3055 50  0000 L CNN
-F 2 "Capacitors SMD:CAPC0603X33N" H 3888 2950 50  0001 C CNN
+F 2 "Marble:CAPC0603X33N" H 3888 2950 50  0001 C CNN
 F 3 "~" H 3850 3100 50  0001 C CNN
 F 4 "CC0201_100NF_6.3V_10%_X5R" H 3965 3009 50  0001 L CNN "PN"
@@
 F 0 "R?" H 6770 2846 50  0000 L CNN
 F 1 "10k" H 6770 2755 50  0000 L CNN
-F 2 "Resistors SMD:RESC1005X40N" V 6630 2800 50  0001 C CNN
+F 2 "Marble:RESC1005X40N" V 6630 2800 50  0001 C CNN
 F 3 "~" H 6700 2800 50  0001 C CNN
 F 4 "R0402_10K_1%_0.0625W_100PPM" H 6700 2800 50  0001 C CNN "PN"
@@
 F 0 "R?" H 7020 2846 50  0000 L CNN
 F 1 "10k" H 7020 2755 50  0000 L CNN
-F 2 "Resistors SMD:RESC1005X40N" V 6880 2800 50  0001 C CNN
+F 2 "Marble:RESC1005X40N" V 6880 2800 50  0001 C CNN
 F 3 "~" H 6950 2800 50  0001 C CNN
 F 4 "R0402_10K_1%_0.0625W_100PPM" H 6950 2800 50  0001 C CNN "PN"
@@
 F 0 "R?" H 7270 2846 50  0000 L CNN
 F 1 "10k" H 7270 2755 50  0000 L CNN
-F 2 "Resistors SMD:RESC1005X40N" V 7130 2800 50  0001 C CNN
+F 2 "Marble:RESC1005X40N" V 7130 2800 50  0001 C CNN
 F 3 "~" H 7200 2800 50  0001 C CNN
 F 4 "R0402_10K_1%_0.0625W_100PPM" H 7200 2800 50  0001 C CNN "PN"
@@
 F 0 "R?" H 7520 2846 50  0000 L CNN
 F 1 "10k" H 7520 2755 50  0000 L CNN
-F 2 "Resistors SMD:RESC1005X40N" V 7380 2800 50  0001 C CNN
+F 2 "Marble:RESC1005X40N" V 7380 2800 50  0001 C CNN
 F 3 "~" H 7450 2800 50  0001 C CNN
 F 4 "R0402_10K_1%_0.0625W_100PPM" H 7450 2800 50  0001 C CNN "PN"
@@
 F 0 "R?" H 7770 2846 50  0000 L CNN
 F 1 "10k" H 7770 2755 50  0000 L CNN
-F 2 "Resistors SMD:RESC1005X40N" V 7630 2800 50  0001 C CNN
+F 2 "Marble:RESC1005X40N" V 7630 2800 50  0001 C CNN
 F 3 "~" H 7700 2800 50  0001 C CNN
 F 4 "R0402_10K_1%_0.0625W_100PPM" H 7700 2800 50  0001 C CNN "PN"
@@
 F 0 "U?" H 8550 3764 50  0000 R CNN
 F 1 "74LVC2T45DC" H 8550 3673 50  0000 R CNN
-F 2 "kicad-libraries-master:VSSOP8" H 8550 3500 50  0001 C CNN
+F 2 "Marble:VSSOP8" H 8550 3500 50  0001 C CNN
 F 3 "https://assets.nexperia.com/documents/data-sheet/74LVC_LVCH2T45.pdf" H 8800 4100 50  0001 C CNN
 	1    8550 4350
@@
 F 0 "C?" H 8315 3796 50  0000 L CNN
 F 1 "100nF" H 8315 3705 50  0000 L CNN
-F 2 "Capacitors SMD:CAPC0603X33N" H 8238 3600 50  0001 C CNN
+F 2 "Marble:CAPC0603X33N" H 8238 3600 50  0001 C CNN
 F 3 "~" H 8200 3750 50  0001 C CNN
 F 4 "CC0201_100NF_6.3V_10%_X5R" H 8315 3659 50  0001 L CNN "PN"
@@
 F 0 "C?" H 9015 3796 50  0000 L CNN
 F 1 "100nF" H 9015 3705 50  0000 L CNN
-F 2 "Capacitors SMD:CAPC0603X33N" H 8938 3600 50  0001 C CNN
+F 2 "Marble:CAPC0603X33N" H 8938 3600 50  0001 C CNN
 F 3 "~" H 8900 3750 50  0001 C CNN
 F 4 "CC0201_100NF_6.3V_10%_X5R" H 9015 3659 50  0001 L CNN "PN"
@@
 F 0 "U?" H 9600 5014 50  0000 R CNN
 F 1 "74LVC2T45DC" H 9600 4923 50  0000 R CNN
-F 2 "kicad-libraries-master:VSSOP8" H 9600 4750 50  0001 C CNN
+F 2 "Marble:VSSOP8" H 9600 4750 50  0001 C CNN
 F 3 "https://assets.nexperia.com/documents/data-sheet/74LVC_LVCH2T45.pdf" H 9850 5350 50  0001 C CNN
 	1    9600 5600
@@
 F 0 "C?" H 9365 5046 50  0000 L CNN
 F 1 "100nF" H 9365 4955 50  0000 L CNN
-F 2 "Capacitors SMD:CAPC0603X33N" H 9288 4850 50  0001 C CNN
+F 2 "Marble:CAPC0603X33N" H 9288 4850 50  0001 C CNN
 F 3 "~" H 9250 5000 50  0001 C CNN
 F 4 "CC0201_100NF_6.3V_10%_X5R" H 9365 4909 50  0001 L CNN "PN"
@@
 F 0 "C?" H 10065 5046 50  0000 L CNN
 F 1 "100nF" H 10065 4955 50  0000 L CNN
-F 2 "Capacitors SMD:CAPC0603X33N" H 9988 4850 50  0001 C CNN
+F 2 "Marble:CAPC0603X33N" H 9988 4850 50  0001 C CNN
 F 3 "~" H 9950 5000 50  0001 C CNN
 F 4 "CC0201_100NF_6.3V_10%_X5R" H 10065 4909 50  0001 L CNN "PN"
@@
 F 0 "R?" H 9370 4046 50  0000 L CNN
 F 1 "10k" H 9370 3955 50  0000 L CNN
-F 2 "Resistors SMD:RESC1005X40N" V 9230 4000 50  0001 C CNN
+F 2 "Marble:RESC1005X40N" V 9230 4000 50  0001 C CNN
 F 3 "~" H 9300 4000 50  0001 C CNN
 F 4 "R0402_10K_1%_0.0625W_100PPM" H 9300 4000 50  0001 C CNN "PN"
@@
 F 0 "R?" H 7820 4046 50  0000 L CNN
 F 1 "10k" H 7820 3955 50  0000 L CNN
-F 2 "Resistors SMD:RESC1005X40N" V 7680 4000 50  0001 C CNN
+F 2 "Marble:RESC1005X40N" V 7680 4000 50  0001 C CNN
 F 3 "~" H 7750 4000 50  0001 C CNN
 F 4 "R0402_10K_1%_0.0625W_100PPM" H 7750 4000 50  0001 C CNN "PN"
