File: FPGA_15_16.sch (KiCad schematic (older format))
At the start: 24 parts, among them J15 10029449-111RLF, Q20 BSS138LT1G, Q21 BSS138LT1G, U1 XC7A100T-2FGG484C, U12 MC78L05ACDR2G, U42 SN65MLVD2DRBT

Commit message: Convert all footprints to use Marble nickname
Includes both .sch and .lib files
Includes both bare footprint names and those with CERN-like nicknames
Parts:
- C103, C104: footprint CAPC2012X135N -> Marble:CAPC2012X135N
- C37, C376, C377: footprint CAPC0603X33N -> Marble:CAPC0603X33N
- D10, D11: footprint SOT95P280X145-6N -> Marble:SOT95P280X145-6N
- Q20, Q21: footprint ICs And Semiconductors SMD:SOT95P240X110-3N -> Marble:SOT95P240X110-3N
- R141, R164, R206, R207, R208, R211, R217, R218, R219, R220, R226: footprint RESC1005X40N -> Marble:RESC1005X40N
- U1: footprint ICs And Semiconductors SMD_BGA:BGA484C100P22X22_2300X2300X240 -> Marble:BGA484C100P22X22_2300X2300X240
- U12: footprint SOIC127P600X175-8N -> Marble:SOIC127P600X175-8N
- U42: footprint ICs And Semiconductors SMD:SON50P300X300X80-9N-R175X248 -> Marble:SON50P300X300X80-9N-R175X248
Changed lines of the file:
@@
 F 0 "D10" H 5750 7750 50  0000 C CNN
 F 1 "HDMIULC6-4SC6" H 5750 7850 50  0000 C CNN
-F 2 "SOT95P280X145-6N" H 5550 6910 60  0001 L CNN
+F 2 "Marble:SOT95P280X145-6N" H 5550 6910 60  0001 L CNN
 F 3 "\\\\cern.ch\\dfs\\Applications\\Altium\\Datasheets\\HDMIULC6-4SC6.pdf" H 5550 7630 60  0001 L CNN
 F 4 "HDMIULC6-4SC6" H 5550 7540 60  0001 L CNN "Part Number"
@@
 F 0 "D11" H 5350 8915 50  0000 C CNN
 F 1 "HDMIULC6-4SC6" H 5350 8824 50  0000 C CNN
-F 2 "SOT95P280X145-6N" H 5150 7260 60  0001 L CNN
+F 2 "Marble:SOT95P280X145-6N" H 5150 7260 60  0001 L CNN
 F 3 "\\\\cern.ch\\dfs\\Applications\\Altium\\Datasheets\\HDMIULC6-4SC6.pdf" H 5150 7980 60  0001 L CNN
 F 4 "HDMIULC6-4SC6" H 5150 7890 60  0001 L CNN "Part Number"
@@
 F 0 "U12" H 11650 9265 50  0000 C CNN
 F 1 "MC78L05ACDR2G" H 11650 9174 50  0000 C CNN
-F 2 "SOIC127P600X175-8N" H 11350 7510 60  0001 L CNN
+F 2 "Marble:SOIC127P600X175-8N" H 11350 7510 60  0001 L CNN
 F 3 "\\\\cern.ch\\dfs\\Applications\\Altium\\Datasheets\\MC78L05ACDG.pdf" H 11350 8230 60  0001 L CNN
 F 4 "MC78L05ACDG" H 11350 8140 60  0001 L CNN "Part Number"
@@
 F 0 "Q20" V 7614 9300 50  0000 C CNN
 F 1 "BSS138LT1G" V 7705 9300 50  0000 C CNN
-F 2 "ICs And Semiconductors SMD:SOT95P240X110-3N" H 7250 8040 60  0001 L CNN
+F 2 "Marble:SOT95P240X110-3N" H 7250 8040 60  0001 L CNN
 F 3 "\\\\cern.ch\\dfs\\Applications\\Altium\\Datasheets\\BSS139.pdf" H 7250 8760 60  0001 L CNN
 F 4 "BSS138LT1G" H 7250 8670 60  0001 L CNN "Part Number"
@@
 F 0 "Q21" V 7614 10100 50  0000 C CNN
 F 1 "BSS138LT1G" V 7705 10100 50  0000 C CNN
-F 2 "ICs And Semiconductors SMD:SOT95P240X110-3N" H 7250 8840 60  0001 L CNN
+F 2 "Marble:SOT95P240X110-3N" H 7250 8840 60  0001 L CNN
 F 3 "\\\\cern.ch\\dfs\\Applications\\Altium\\Datasheets\\BSS139.pdf" H 7250 9560 60  0001 L CNN
 F 4 "BSS138LT1G" H 7250 9470 60  0001 L CNN "Part Number"
@@
 F 0 "C103" V 10900 9200 50  0000 L CNN
 F 1 "CC0805_4.7UF_10V_10%_X5R" H 10850 8940 60  0001 L CNN
-F 2 "CAPC2012X135N" H 10850 8130 60  0001 L CNN
+F 2 "Marble:CAPC2012X135N" H 10850 8130 60  0001 L CNN
 F 3 "\\\\cern.ch\\dfs\\Applications\\Altium\\Datasheets\\CC0805_X5R_PHYCOMP_HC.pdf" H 10850 8760 60  0001 L CNN
 F 4 "4.7uF" V 11100 9200 50  0000 L CNN "~"
@@
 F 0 "C104" V 12600 9200 50  0000 L CNN
 F 1 "CC0805_4.7UF_10V_10%_X5R" H 12550 8940 60  0001 L CNN
-F 2 "CAPC2012X135N" H 12550 8130 60  0001 L CNN
+F 2 "Marble:CAPC2012X135N" H 12550 8130 60  0001 L CNN
 F 3 "\\\\cern.ch\\dfs\\Applications\\Altium\\Datasheets\\CC0805_X5R_PHYCOMP_HC.pdf" H 12550 8760 60  0001 L CNN
 F 4 "4.7uF" V 12800 9200 50  0000 L CNN "~"
@@
 F 0 "R226" H 8250 7400 50  0000 L CNN
 F 1 "R0402_49R9_1%_0.0625W_100PPM" H 8200 7290 60  0001 L CNN
-F 2 "RESC1005X40N" H 8200 6480 60  0001 L CNN
+F 2 "Marble:RESC1005X40N" H 8200 6480 60  0001 L CNN
 F 3 "\\\\cern.ch\\dfs\\Applications\\Altium\\Datasheets\\R0402_Phycomp_RC0402.pdf" H 8200 7110 60  0001 L CNN
 F 4 "49R9" H 8250 7600 50  0000 L CNN "~"
@@
 F 0 "R219" H 7950 7400 50  0000 L CNN
 F 1 "R0402_49R9_1%_0.0625W_100PPM" H 7900 7290 60  0001 L CNN
-F 2 "RESC1005X40N" H 7900 6480 60  0001 L CNN
+F 2 "Marble:RESC1005X40N" H 7900 6480 60  0001 L CNN
 F 3 "\\\\cern.ch\\dfs\\Applications\\Altium\\Datasheets\\R0402_Phycomp_RC0402.pdf" H 7900 7110 60  0001 L CNN
 F 4 "49R9" H 7950 7600 50  0000 L CNN "~"
@@
 F 0 "R211" H 7650 7400 50  0000 L CNN
 F 1 "R0402_49R9_1%_0.0625W_100PPM" H 7600 7290 60  0001 L CNN
-F 2 "RESC1005X40N" H 7600 6480 60  0001 L CNN
+F 2 "Marble:RESC1005X40N" H 7600 6480 60  0001 L CNN
 F 3 "\\\\cern.ch\\dfs\\Applications\\Altium\\Datasheets\\R0402_Phycomp_RC0402.pdf" H 7600 7110 60  0001 L CNN
 F 4 "49R9" H 7650 7600 50  0000 L CNN "~"
@@
 F 0 "R208" H 7350 7400 50  0000 L CNN
 F 1 "R0402_49R9_1%_0.0625W_100PPM" H 7300 7290 60  0001 L CNN
-F 2 "RESC1005X40N" H 7300 6480 60  0001 L CNN
+F 2 "Marble:RESC1005X40N" H 7300 6480 60  0001 L CNN
 F 3 "\\\\cern.ch\\dfs\\Applications\\Altium\\Datasheets\\R0402_Phycomp_RC0402.pdf" H 7300 7110 60  0001 L CNN
 F 4 "49R9" H 7350 7600 50  0000 L CNN "~"
@@
 F 0 "R207" H 7050 7400 50  0000 L CNN
 F 1 "R0402_49R9_1%_0.0625W_100PPM" H 7000 7290 60  0001 L CNN
-F 2 "RESC1005X40N" H 7000 6480 60  0001 L CNN
+F 2 "Marble:RESC1005X40N" H 7000 6480 60  0001 L CNN
 F 3 "\\\\cern.ch\\dfs\\Applications\\Altium\\Datasheets\\R0402_Phycomp_RC0402.pdf" H 7000 7110 60  0001 L CNN
 F 4 "49R9" H 7050 7600 50  0000 L CNN "~"
@@
 F 0 "R206" H 6750 7400 50  0000 L CNN
 F 1 "R0402_49R9_1%_0.0625W_100PPM" H 6700 7290 60  0001 L CNN
-F 2 "RESC1005X40N" H 6700 6480 60  0001 L CNN
+F 2 "Marble:RESC1005X40N" H 6700 6480 60  0001 L CNN
 F 3 "\\\\cern.ch\\dfs\\Applications\\Altium\\Datasheets\\R0402_Phycomp_RC0402.pdf" H 6700 7110 60  0001 L CNN
 F 4 "49R9" H 6750 7600 50  0000 L CNN "~"
@@
 F 0 "R164" H 6450 7400 50  0000 L CNN
 F 1 "R0402_49R9_1%_0.0625W_100PPM" H 6400 7290 60  0001 L CNN
-F 2 "RESC1005X40N" H 6400 6480 60  0001 L CNN
+F 2 "Marble:RESC1005X40N" H 6400 6480 60  0001 L CNN
 F 3 "\\\\cern.ch\\dfs\\Applications\\Altium\\Datasheets\\R0402_Phycomp_RC0402.pdf" H 6400 7110 60  0001 L CNN
 F 4 "49R9" H 6450 7600 50  0000 L CNN "~"
@@
 F 0 "R141" H 6150 7400 50  0000 L CNN
 F 1 "R0402_49R9_1%_0.0625W_100PPM" H 6100 7290 60  0001 L CNN
-F 2 "RESC1005X40N" H 6100 6480 60  0001 L CNN
+F 2 "Marble:RESC1005X40N" H 6100 6480 60  0001 L CNN
 F 3 "\\\\cern.ch\\dfs\\Applications\\Altium\\Datasheets\\R0402_Phycomp_RC0402.pdf" H 6100 7110 60  0001 L CNN
 F 4 "49R9" H 6150 7600 50  0000 L CNN "~"
@@
 F 0 "R217" V 7954 9260 50  0000 L CNN
 F 1 "R0402_2K2_1%_0.0625W_100PPM" H 7850 8990 60  0001 L CNN
-F 2 "RESC1005X40N" H 7850 8180 60  0001 L CNN
+F 2 "Marble:RESC1005X40N" H 7850 8180 60  0001 L CNN
 F 3 "\\\\cern.ch\\dfs\\Applications\\Altium\\Datasheets\\R0402_Phycomp_RC0402.pdf" H 7850 8810 60  0001 L CNN
 F 4 "2k2" V 8045 9260 50  0000 L CNN "~"
@@
 F 0 "R218" V 7954 10060 50  0000 L CNN
 F 1 "R0402_2K2_1%_0.0625W_100PPM" H 7850 9790 60  0001 L CNN
-F 2 "RESC1005X40N" H 7850 8980 60  0001 L CNN
+F 2 "Marble:RESC1005X40N" H 7850 8980 60  0001 L CNN
 F 3 "\\\\cern.ch\\dfs\\Applications\\Altium\\Datasheets\\R0402_Phycomp_RC0402.pdf" H 7850 9610 60  0001 L CNN
 F 4 "2k2" V 8045 10060 50  0000 L CNN "~"
@@
 F 0 "R220" V 8904 9910 50  0000 L CNN
 F 1 "R0402_2K2_1%_0.0625W_100PPM" H 8800 9640 60  0001 L CNN
-F 2 "RESC1005X40N" H 8800 8830 60  0001 L CNN
+F 2 "Marble:RESC1005X40N" H 8800 8830 60  0001 L CNN
 F 3 "\\\\cern.ch\\dfs\\Applications\\Altium\\Datasheets\\R0402_Phycomp_RC0402.pdf" H 8800 9460 60  0001 L CNN
 F 4 "2k2" V 8995 9910 50  0000 L CNN "~"
@@
 F 0 "C37" V 9200 9550 50  0000 L CNN
 F 1 "CC0201_100NF_6.3V_10%_X5R" H 9150 9290 60  0001 L CNN
-F 2 "CAPC0603X33N" H 9150 8480 60  0001 L CNN
+F 2 "Marble:CAPC0603X33N" H 9150 8480 60  0001 L CNN
 F 3 "\\\\cern.ch\\dfs\\Applications\\Altium\\Datasheets\\CC0201_X5R_AVX.pdf" H 9150 9110 60  0001 L CNN
 F 4 "100nF" V 9400 9550 50  0000 L CNN "~"
@@
 F 0 "U42" H 11050 5850 50  0000 C CNN
 F 1 "SN65MLVD2DRBT" H 11050 5774 50  0000 C CNN
-F 2 "ICs And Semiconductors SMD:SON50P300X300X80-9N-R175X248" H 10800 5600 50  0001 C CNN
+F 2 "Marble:SON50P300X300X80-9N-R175X248" H 10800 5600 50  0001 C CNN
 F 3 "" H 10800 5600 50  0001 C CNN
 F 4 "SN65MLVD2DRBT" H 11050 5773 50  0001 C CNN "Manufacturer Part Number"
@@
 F 0 "U1" H 7250 926 50  0000 C CNN
 F 1 "XC7A100T-2FGG484C" H 7250 835 50  0000 C CNN
-F 2 "ICs And Semiconductors SMD_BGA:BGA484C100P22X22_2300X2300X240" H 7250 3900 50  0001 C CNN
+F 2 "Marble:BGA484C100P22X22_2300X2300X240" H 7250 3900 50  0001 C CNN
 F 3 "" H 7250 3900 50  0000 C CNN
 F 4 "XC7A100T-2FGG484C" H 7250 3900 50  0001 C CNN "Manufacturer Part Number"
@@
 F 0 "C376" V 11704 6260 50  0000 L CNN
 F 1 "CC0201_100NF_6.3V_10%_X5R" H 11600 5890 60  0001 L CNN
-F 2 "CAPC0603X33N" H 11600 5080 60  0001 L CNN
+F 2 "Marble:CAPC0603X33N" H 11600 5080 60  0001 L CNN
 F 3 "\\\\cern.ch\\dfs\\Applications\\Altium\\Datasheets\\CC0201_X5R_AVX.pdf" H 11600 5710 60  0001 L CNN
 F 4 "100nF" V 11795 6260 50  0000 L CNN "~"
@@
 F 0 "C377" V 12154 6260 50  0000 L CNN
 F 1 "CC0201_100NF_6.3V_10%_X5R" H 12050 5890 60  0001 L CNN
-F 2 "CAPC0603X33N" H 12050 5080 60  0001 L CNN
+F 2 "Marble:CAPC0603X33N" H 12050 5080 60  0001 L CNN
 F 3 "\\\\cern.ch\\dfs\\Applications\\Altium\\Datasheets\\CC0201_X5R_AVX.pdf" H 12050 5710 60  0001 L CNN
 F 4 "100nF" V 12245 6260 50  0000 L CNN "~"

Commit message: Clean up BSS138 instances in schematic
Q5 Q6 Q8 Q9 Q14 Q17 Q18 Q19 Q20 Q21 Q24
Fewer warnings from KiBoM
Parts:
- Q20, Q21: HelpURL \\\\cern.ch\\dfs\\Applications\\Altium\\Datasheets\\BSS139.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 -> \\\\cern.ch\\dfs\\Applications\\Altium\\Datasheets\\BSS138L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
Changed lines of the file:
@@
 F 1 "BSS138LT1G" V 7705 9300 50  0000 C CNN
 F 2 "Marble:SOT95P240X110-3N" H 7250 8040 60  0001 L CNN
-F 3 "\\\\cern.ch\\dfs\\Applications\\Altium\\Datasheets\\BSS139.pdf" H 7250 8760 60  0001 L CNN
+F 3 "\\\\cern.ch\\dfs\\Applications\\Altium\\Datasheets\\BSS138LT1G.pdf" H 7250 8760 60  0001 L CNN
 F 4 "BSS138LT1G" H 7250 8670 60  0001 L CNN "Part Number"
 F 5 "N-MOSFET-D 1G 2S 3D" H 7250 8580 60  0001 L CNN "Library Ref"
@@
 F 27 "PcbLib\\ICs And Semiconductors SMD.PcbLib" H 7250 6510 60  0001 L CNN "Footprint Path"
 F 28 "SOT95P240X110-3N" H 7250 6420 60  0001 L CNN "Footprint Ref"
-F 29 "\\\\cern.ch\\dfs\\Applications\\Altium\\Datasheets\\BSS139.pdf" H 7250 6330 60  0001 L CNN "HelpURL"
+F 29 "\\\\cern.ch\\dfs\\Applications\\Altium\\Datasheets\\BSS138LT1G.pdf" H 7250 6330 60  0001 L CNN "HelpURL"
 F 30 "~~" H 7250 6240 60  0001 L CNN "ComponentLink1URL"
 F 31 " " H 7250 6150 60  0001 L CNN "ComponentLink1Description"
@@
 F 1 "BSS138LT1G" V 7705 10100 50  0000 C CNN
 F 2 "Marble:SOT95P240X110-3N" H 7250 8840 60  0001 L CNN
-F 3 "\\\\cern.ch\\dfs\\Applications\\Altium\\Datasheets\\BSS139.pdf" H 7250 9560 60  0001 L CNN
+F 3 "\\\\cern.ch\\dfs\\Applications\\Altium\\Datasheets\\BSS138LT1G.pdf" H 7250 9560 60  0001 L CNN
 F 4 "BSS138LT1G" H 7250 9470 60  0001 L CNN "Part Number"
 F 5 "N-MOSFET-D 1G 2S 3D" H 7250 9380 60  0001 L CNN "Library Ref"
@@
 F 27 "PcbLib\\ICs And Semiconductors SMD.PcbLib" H 7250 7310 60  0001 L CNN "Footprint Path"
 F 28 "SOT95P240X110-3N" H 7250 7220 60  0001 L CNN "Footprint Ref"
-F 29 "\\\\cern.ch\\dfs\\Applications\\Altium\\Datasheets\\BSS139.pdf" H 7250 7130 60  0001 L CNN "HelpURL"
+F 29 "\\\\cern.ch\\dfs\\Applications\\Altium\\Datasheets\\BSS138LT1G.pdf" H 7250 7130 60  0001 L CNN "HelpURL"
 F 30 "~~" H 7250 7040 60  0001 L CNN "ComponentLink1URL"
 F 31 " " H 7250 6950 60  0001 L CNN "ComponentLink1Description"
