File: FPGA_15_16.sch (KiCad schematic (older format))
At the start: 29 parts, among them J15 10029449-111RLF, Q20 BSS138LT1G, Q21 BSS138LT1G, U1 XC7A100T-2FGG484C, U12 MC78L05ACDR2G, U42 SN65MLVD2DRBT, U46 TCA9517DGKR

Commit message: Improve listing for SN65MLVD2DRBT
In both U42 instance, and the library
Parts:
- U42: Manufacturer (none) -> TEXAS INSTRUMENTS
Changed lines of the file:
@@
 F 4 "SN65MLVD2DRBT" H 11050 5773 50  0001 C CNN "Manufacturer Part Number"
 F 5 "-standalone" H 11050 5150 50  0001 C CNN "config"
+F 6 "TEXAS INSTRUMENTS" H 10600 5700 50  0001 C CNN "Manufacturer"
 	1    10600 5700
 	1    0    0    -1

Commit message: Trigger one less warning from KiBoM
Parts:
- C103: Comment 4.7uF -> =Value
Changed lines of the file:
@@
 F 6 "Capacitor - non polarized" H 10850 8580 60  0001 L CNN "Library Ref"
 F 7 "SchLib\\Capacitors.SchLib" H 10850 8490 60  0001 L CNN "Library Path"
-F 8 "4.7uF" H 10850 8400 60  0001 L CNN "Comment"
+F 8 "=Value" H 10850 8400 60  0001 L CNN "Comment"
 F 9 "Standard" H 10850 8310 60  0001 L CNN "Component Kind"
 F 10 "Standard" H 10850 8220 60  0001 L CNN "Component Type"

Commit message: Fix footprint field in sch. and symbol lib.
... concerns U44 - U46, which didn't have the Marble: prefix
Parts:
- U46: footprint ICs And Semiconductors SMD:SOP65P490X110-8N -> Marble:SOP65P490X110-8N
Changed lines of the file:
@@
 F 0 "U46" H 11350 3765 50  0000 C CNN
 F 1 "TCA9517DGKR" H 11350 3674 50  0000 C CNN
-F 2 "ICs And Semiconductors SMD:SOP65P490X110-8N" H 10950 2650 50  0001 L CNN
+F 2 "Marble:SOP65P490X110-8N" H 10950 2650 50  0001 L CNN
 F 3 " " H 10950 2575 50  0001 L CNN
 F 4 "TCA9517DGKR" H 10950 2500 50  0001 L CNN "Part Number"
@@
 Wire Wire Line
 	12150 4100 11950 4100
+Connection ~ 12150 4100
 Wire Bus Line
 	14050 7300 14050 7600
@@
 Wire Bus Line
 	13600 4850 13600 5750
-Connection ~ 12150 4100
 $EndSCHEMATC

Commit message: Upgrade voltage rating on 0603 4.7uF
Convert 26 caps from CC0603_4.7UF_16V_10%_X5R to CC0603_4.7UF_25V_10%_X5R
C57 C103 C105 C127 C129 C139 C142 C143 C144 C159 C161 C162 C167 C168 C173 C195 C331 C343 C344 C347 C348 C349 C360 C361 C364 C373
Samsung CL10A475KA8NQN, $0.11456 in 500s at Digi-Key
Parts:
- C103: value CC0603_4.7UF_16V_10%_X5R -> CC0603_4.7UF_25V_10%_X5R; symbol Capacitors_SMD:CC0603_4.7UF_16V_10%_X5R -> Capacitors_SMD:CC0603_4.7UF_25V_10%_X5R; Manufacturer Part Number CC0603_4.7UF_16V_10%_X5R -> CC0603_4.7UF_25V_10%_X5R; Manufacturer1 Example TAIYO YUDEN -> Samsung; Manufacturer1 Part Number EMK107ABJ475KA-T -> CL10A475KA8NQN; Part Number CC0603_4.7UF_16V_10%_X5R -> CC0603_4.7UF_25V_10%_X5R; Voltage 16V -> 25V
Changed lines of the file:
@@
 $EndComp
 $Comp
-L Capacitors_SMD:CC0603_4.7UF_16V_10%_X5R C?
+L Capacitors_SMD:CC0603_4.7UF_25V_10%_X5R C?
 U 1 1 5F501BA6
 P 10850 9200
@@
 AR Path="/5C907554/5CAAC367/5F501BA6" Ref="C103"  Part="1"
 F 0 "C103" V 10900 9200 50  0000 L CNN
-F 1 "CC0603_4.7UF_16V_10%_X5R" H 10850 8940 60  0001 L CNN
+F 1 "CC0603_4.7UF_25V_10%_X5R" H 10850 8940 60  0001 L CNN
 F 2 "Marble:CAPC1709X95N" H 10850 8130 60  0001 L CNN
 F 3 "\\\\cern.ch\\dfs\\Applications\\Altium\\Datasheets\\CC0805_X5R_PHYCOMP_HC.pdf" H 10850 8760 60  0001 L CNN
 F 4 "4.7uF" V 11100 9200 50  0000 L CNN "Val"
-F 5 "CC0603_4.7UF_16V_10%_X5R" H 10850 8670 60  0001 L CNN "Part Number"
+F 5 "CC0603_4.7UF_25V_10%_X5R" H 10850 8670 60  0001 L CNN "Part Number"
 F 6 "Capacitor - non polarized" H 10850 8580 60  0001 L CNN "Library Ref"
 F 7 "SchLib\\Capacitors.SchLib" H 10850 8490 60  0001 L CNN "Library Path"
@@
 F 15 "None" H 10850 7590 60  0001 L CNN "Status"
 F 16 " " H 10850 7500 60  0001 L CNN "Status Comment"
-F 17 "16V" H 10850 7410 60  0001 L CNN "Voltage"
+F 17 "25V" H 10850 7410 60  0001 L CNN "Voltage"
 F 18 "X5R" H 10850 7320 60  0001 L CNN "TC"
 F 19 "±10%" H 10850 7230 60  0001 L CNN "Tolerance"
 F 20 "SMD Multilayer Chip Ceramic Capacitor" H 10850 7140 60  0001 L CNN "Part Description"
 F 21 "GENERIC" H 10850 7050 60  0001 L CNN "Manufacturer"
-F 22 "CC0603_4.7UF_16V_10%_X5R" H 10850 6960 60  0001 L CNN "Manufacturer Part Number"
+F 22 "CC0603_4.7UF_25V_10%_X5R" H 10850 6960 60  0001 L CNN "Manufacturer Part Number"
 F 23 "0603" H 10850 6870 60  0001 L CNN "Case"
 F 24 "Yes" H 10850 6780 60  0001 L CNN "Mounted"
@@
 F 29 " " H 10850 6330 60  0001 L CNN "Sense Comment"
 F 30 " " H 10850 6240 60  0001 L CNN "ComponentHeight"
-F 31 "TAIYO YUDEN" H 10850 6150 60  0001 L CNN "Manufacturer1 Example"
-F 32 "EMK107ABJ475KA-T" H 10850 6060 60  0001 L CNN "Manufacturer1 Part Number"
+F 31 "Samsung" H 10850 6150 60  0001 L CNN "Manufacturer1 Example"
+F 32 "CL10A475KA8NQN" H 10850 6060 60  0001 L CNN "Manufacturer1 Part Number"
 F 33 "0.95mm" H 10850 5970 60  0001 L CNN "Manufacturer1 ComponentHeight"
 F 34 "CERN DEM JLC" H 10850 5790 60  0001 L CNN "Author"

Commit message: Add two user LEDs to FPGA pins
LD16 LD17
Parts:
- added LD16, LD17: LED_KINGBRIGHT_KPH-1608CGCK, Marble:LED_KINGBRIGHT_KPH-1608CGCK, symbol LEDs_&_Displays:LED_KINGBRIGHT_KPH-1608CGCK
- added R306, R307: R0402_1K_1%_0.0625W_100PPM, Marble:RESC1005X40N, symbol Resistors_SMD:R0402_1K_1%_0.0625W_100PPM
Connections:
- wire segments 267 -> 277
- no-connect marks 13 -> 11

Commit message: Better attribute consistency: fewer warnings from KiBoM
Someday maybe we'll just nuke the Comment field entirely
Parts:
- R306, R307: Comment 1k -> =Value
Changed lines of the file:
@@
 F 6 "Resistor - 1%" H 11100 805 50  0001 L CNN "Library Ref"
 F 7 "SchLib\\Resistors.SchLib" H 11100 730 50  0001 L CNN "Library Path"
-F 8 "1k" H 11100 655 50  0001 L CNN "Comment"
+F 8 "=Value" H 11100 655 50  0001 L CNN "Comment"
 F 9 "Standard" H 11100 580 50  0001 L CNN "Component Kind"
 F 10 "Standard" H 11100 505 50  0001 L CNN "Component Type"
@@
 F 6 "Resistor - 1%" H 11700 805 50  0001 L CNN "Library Ref"
 F 7 "SchLib\\Resistors.SchLib" H 11700 730 50  0001 L CNN "Library Path"
-F 8 "1k" H 11700 655 50  0001 L CNN "Comment"
+F 8 "=Value" H 11700 655 50  0001 L CNN "Comment"
 F 9 "Standard" H 11700 580 50  0001 L CNN "Component Kind"
 F 10 "Standard" H 11700 505 50  0001 L CNN "Component Type"

Commit message: Change 8 x TMDS termination resistors from 49R9 to 51R
Reduces BoM line count by one
R226 R219 R211 R208 R207 R206 R164 R141
Parts:
- R141, R164, R206, R207, R208, R211, R219, R226: value R0402_49R9_1%_0.0625W_100PPM -> R0402_51R_1%_0.0625W_100PPM; symbol Resistors_SMD:R0402_49R9_1%_0.0625W_100PPM -> Resistors_SMD:R0402_51R_1%_0.0625W_100PPM; CreateDate 10/24/12 00:00:00 -> 12/03/07 00:00:00; LatestRevisionDate 10/24/12 00:00:00 -> 10/17/12 00:00:00; Manufacturer Part Number R0402_49R9_1%_0.0625W_100PPM -> R0402_51R_1%_0.0625W_100PPM; Manufacturer1 Part Number 232270674999L or RC0402FR-0749R9L -> 232270675109L; Part Number R0402_49R9_1%_0.0625W_100PPM -> R0402_51R_1%_0.0625W_100PPM; Val 49R9 -> 51

Commit message: Start adding isolation for I2C_FPGA_SW_RST and EXP_INT
Adds U47, another TCA9517
Parts:
- added C387, C388: CC0201_100NF_6.3V_10%_X5R, Marble:CAPC0603X33N, symbol Capacitors_SMD:CC0201_100NF_6.3V_10%_X5R
- added R311, R312: R0402_2K2_1%_0.0625W_100PPM, Marble:RESC1005X40N, symbol Resistors_SMD:R0402_2K2_1%_0.0625W_100PPM
- added R313: R0402_0R_JUMPER, Marble:RESC1005X40N, symbol Resistors_SMD:R0402_0R_JUMPER
- added U47: TCA9517DGKR, Marble:SOP65P490X110-8N, symbol Analog_&_Interface:TCA9517DGKR
Connections:
- wire segments 277 -> 301
- no-connect marks 11 -> 10
Other:
- note added: "To FPGA_DONE"
- moved on the sheet: C376, C377
