File: Power.sch (KiCad schematic (older format))
At the start: 75 parts, among them J1 CLIFF_FC68148(DC-10A), Q1 BC857BV, Q15 BC857BV, Q16 SI4425DDY-T1-GE3, Q2 SI4425DDY-T1-GE3, Q22 BC857BV, Q23 SI4425DDY-T1-GE3, Q25 Si2315BDS-T1-E3, Q3 SI4425DDY-T1-GE3, Q4 SI4425DDY-T1-GE3, Q8 BSS138LT1G, Q9 BSS138LT1G, U17 INA219BIDCNT, U18 TPS62175DQC, U32 INA219BIDCNT, U40 AG5300, U41 FOD817DSD, U43 INA219BIDCNT

Commit message: Sync PCB
Parts:
- U43: footprint ICs And Semiconductors SMD:SOT65P280X145-8N -> Marble:SOT65P280X145-8N; Comment =Device -> INA219BIDCNT; ComponentLink1Description ~~ -> (none); ComponentLink2Description ~~ -> (none); Database Table Name (none) -> Analog & Interface; Footprint Library (none) -> ICs And Semiconductors SMD; Library Name ICs And Semiconductors SMD -> ICs And Semiconductors.DbLib; SCEM (none) -> (none); Sense Comment ~~ -> (none); Status ~~ -> (none); Status Comment ~~ -> (none)
Changed lines of the file:
@@
 F 0 "U43" H 7950 1715 50  0000 C CNN
 F 1 "INA219BIDCNT" H 7950 1624 50  0000 C CNN
-F 2 "ICs And Semiconductors SMD:SOT65P280X145-8N" H 7600 -340 60  0001 L CNN
-F 3 "" H 7600 380 60  0001 L CNN
+F 2 "Marble:SOT65P280X145-8N" H 7600 -340 60  0001 L CNN
+F 3 " " H 7600 380 60  0001 L CNN
 F 4 "INA219BIDCNT" H 7600 290 60  0001 L CNN "Part Number"
 F 5 "INA219BIDCNT" H 7600 200 60  0001 L CNN "Library Ref"
 F 6 "SchLib\\Analog & Interface.SchLib" H 7600 110 60  0001 L CNN "Library Path"
-F 7 "=Device" H 7600 20  60  0001 L CNN "Comment"
+F 7 "INA219BIDCNT" H 7600 20  60  0001 L CNN "Comment"
 F 8 "Standard" H 7600 -70 60  0001 L CNN "Component Kind"
 F 9 "Standard" H 7600 -160 60  0001 L CNN "Component Type"
 F 10 "INA219BIDCNT" H 7600 -250 60  0001 L CNN "Device"
 F 11 "SOT, 0.65mm pitch; 8 pin, 1.625mm W X 2.90mm L X 1.45mm H body, IPC Medium Density" H 7600 -430 60  0001 L CNN "PackageDescription"
-F 12 "~~" H 7600 -520 60  0001 L CNN "Status"
+F 12 " " H 7600 -520 60  0001 L CNN "Status"
 F 13 "Zero-Drift, Bi-Directional CURRENT/POWER MONITOR with I2C™ Interface" H 7600 -610 60  0001 L CNN "Part Description"
 F 14 "TEXAS INSTRUMENTS" H 7600 -700 60  0001 L CNN "Manufacturer"
@@
 F 21 "No" H 7600 -1330 60  0001 L CNN "PressFit"
 F 22 "No" H 7600 -1420 60  0001 L CNN "Sense"
-F 23 "~~" H 7600 -1510 60  0001 L CNN "Sense Comment"
+F 23 " " H 7600 -1510 60  0001 L CNN "Sense Comment"
 F 24 "No" H 7600 -1600 60  0001 L CNN "Bonding"
-F 25 "~~" H 7600 -1690 60  0001 L CNN "Status Comment"
+F 25 " " H 7600 -1690 60  0001 L CNN "Status Comment"
 F 26 "1.45mm" H 7600 -1780 60  0001 L CNN "ComponentHeight"
 F 27 "PcbLib\\ICs And Semiconductors SMD.PcbLib" H 7600 -1870 60  0001 L CNN "Footprint Path"
@@
 F 31 "~~" H 7600 -2230 60  0001 L CNN "ComponentLink1URL"
 F 32 "~~" H 7600 -2320 60  0001 L CNN "ComponentLink2URL"
-F 33 "~~" H 7600 -2410 60  0001 L CNN "ComponentLink2Description"
-F 34 "~~" H 7600 -2500 60  0001 L CNN "ComponentLink1Description"
+F 33 " " H 7600 -2410 60  0001 L CNN "ComponentLink2Description"
+F 34 " " H 7600 -2500 60  0001 L CNN "ComponentLink1Description"
 F 35 "09/24/13 00:00:00" H 7600 -2590 60  0001 L CNN "CreateDate"
 F 36 "09/24/13 00:00:00" H 7600 -2680 60  0001 L CNN "LatestRevisionDate"
-F 37 "ICs And Semiconductors SMD" H 7600 -2770 60  0001 L CNN "Library Name"
+F 37 "ICs And Semiconductors.DbLib" H 7600 -2770 60  0001 L CNN "Library Name"
 F 38 "This work is licensed under the Creative Commons CC-BY-SA 4.0 License. To the extent that circuit schematics that use Licensed Material can be considered to be ‘Adapted Material’, then the copyright holder waives article 3.b of the license with respect to these schematics." H 7600 -2860 60  0001 L CNN "License"
+F 39 "Analog & Interface" H 7600 1550 50  0001 C CNN "Database Table Name"
+F 40 "ICs And Semiconductors SMD" H 7600 1550 50  0001 C CNN "Footprint Library"
+F 41 " " H 7600 1550 50  0001 C CNN "SCEM"
 	1    7600 1550
 	1    0    0    -1

Commit message: Change R182 R183 R301 from 0.02 Ohm to 0.082 Ohm
More work than it sounds.
Ohmite KDV12DR082ET.
Sets up INA219 for FMC to register 82 mV at FMC spec max 12P0V current of 1.0 Amp.
Whole-board current monitor isn't right yet.  Soon.
Parts:
- R182, R183, R301: value R1206_0R02_1%_0.5W_100PPM -> R1206_0R082_1%_0.5W_100PPM; symbol Resistors_SMD:R1206_0R02_1%_0.5W_100PPM -> Resistors_SMD:R1206_0R082_1%_0.5W_100PPM; LatestRevisionDate 09/03/12 00:00:00 -> 05/12/20 00:00:00; Manufacturer TT Electronics -> Ohmite; Manufacturer Part Number CSR1206FK20L0 -> KDV12DR082ET; Part Number R1206_0R02_1%_0.5W_100PPM -> R1206_0R082_1%_0.5W_100PPM; Val 0R02 -> 0R082; ~ 0R02 -> 0R082
Changed lines of the file:
@@
 Connection ~ 7450 8750
 $Comp
-L Resistors_SMD:R1206_0R02_1%_0.5W_100PPM R182
+L Resistors_SMD:R1206_0R082_1%_0.5W_100PPM R182
 U 1 1 5E1246EE
 P 14100 1900
 F 0 "R182" H 14250 2000 50  0000 C CNN
-F 1 "R1206_0R02_1%_0.5W_100PPM" H 14100 1690 60  0001 L CNN
+F 1 "R1206_0R082_1%_0.5W_100PPM" H 14100 1690 60  0001 L CNN
 F 2 "RESC3216X80N" H 14100 880 60  0001 L CNN
 F 3 "\\\\cern.ch\\dfs\\Applications\\Altium\\Datasheets\\R1206_WELWYN_LRF.pdf" H 14100 1510 60  0001 L CNN
-F 4 "0R02" H 14250 1800 50  0000 C CNN "~"
-F 5 "R1206_0R02_1%_0.5W_100PPM" H 14100 1420 60  0001 L CNN "Part Number"
+F 4 "0R082" H 14250 1800 50  0000 C CNN "~"
+F 5 "R1206_0R082_1%_0.5W_100PPM" H 14100 1420 60  0001 L CNN "Part Number"
 F 6 "Resistor - 1%" H 14100 1330 60  0001 L CNN "Library Ref"
 F 7 "SchLib\\Resistors.SchLib" H 14100 1240 60  0001 L CNN "Library Path"
@@
 F 13 "PcbLib\\Resistors SMD.PcbLib" H 14100 610 60  0001 L CNN "Footprint Path"
 F 14 "RESC3216X80N" H 14100 520 60  0001 L CNN "Footprint Ref"
-F 15 "0R02" H 14100 430 60  0001 L CNN "Val"
+F 15 "0R082" H 14100 430 60  0001 L CNN "Val"
 F 16 "None" H 14100 340 60  0001 L CNN "Status"
 F 17 "0.5W" H 14100 250 60  0001 L CNN "Power"
@@
 F 20 "±1%" H 14100 -20 60  0001 L CNN "Tolerance"
 F 21 "Low Value Flat Chip Resistor" H 14100 -110 60  0001 L CNN "Part Description"
-F 22 "TT Electronics" H 14100 -200 60  0001 L CNN "Manufacturer"
-F 23 "CSR1206FK20L0" H 14100 -290 60  0001 L CNN "Manufacturer Part Number"
+F 22 "Ohmite" H 14100 -200 60  0001 L CNN "Manufacturer"
+F 23 "KDV12DR082ET" H 14100 -290 60  0001 L CNN "Manufacturer Part Number"
 F 24 "1206" H 14100 -380 60  0001 L CNN "Case"
 F 25 "No" H 14100 -470 60  0001 L CNN "PressFit"
@@
 F 37 "CERN DEM JLC" H 14100 -1550 60  0001 L CNN "Author"
 F 38 "05/11/10 00:00:00" H 14100 -1640 60  0001 L CNN "CreateDate"
-F 39 "09/03/12 00:00:00" H 14100 -1730 60  0001 L CNN "LatestRevisionDate"
+F 39 "05/12/20 00:00:00" H 14100 -1730 60  0001 L CNN "LatestRevisionDate"
 F 40 "Resistors SMD" H 14100 -1820 60  0001 L CNN "Library Name"
 F 41 "This work is licensed under the Creative Commons CC-BY-SA 4.0 License. To the extent that circuit schematics that use Licensed Material can be considered to be ‘Adapted Material’, then the copyright holder waives article 3.b of the license with respect to these schematics." H 14100 -1910 60  0001 L CNN "License"
@@
 $EndComp
 $Comp
-L Resistors_SMD:R1206_0R02_1%_0.5W_100PPM R183
+L Resistors_SMD:R1206_0R082_1%_0.5W_100PPM R183
 U 1 1 5E156EFB
 P 14100 5300
 F 0 "R183" H 14250 5400 50  0000 C CNN
-F 1 "R1206_0R02_1%_0.5W_100PPM" H 14100 5090 60  0001 L CNN
+F 1 "R1206_0R082_1%_0.5W_100PPM" H 14100 5090 60  0001 L CNN
 F 2 "RESC3216X80N" H 14100 4280 60  0001 L CNN
 F 3 "\\\\cern.ch\\dfs\\Applications\\Altium\\Datasheets\\R1206_WELWYN_LRF.pdf" H 14100 4910 60  0001 L CNN
-F 4 "0R02" H 14250 5200 50  0000 C CNN "~"
-F 5 "R1206_0R02_1%_0.5W_100PPM" H 14100 4820 60  0001 L CNN "Part Number"
+F 4 "0R082" H 14250 5200 50  0000 C CNN "~"
+F 5 "R1206_0R082_1%_0.5W_100PPM" H 14100 4820 60  0001 L CNN "Part Number"
 F 6 "Resistor - 1%" H 14100 4730 60  0001 L CNN "Library Ref"
 F 7 "SchLib\\Resistors.SchLib" H 14100 4640 60  0001 L CNN "Library Path"
@@
 F 13 "PcbLib\\Resistors SMD.PcbLib" H 14100 4010 60  0001 L CNN "Footprint Path"
 F 14 "RESC3216X80N" H 14100 3920 60  0001 L CNN "Footprint Ref"
-F 15 "0R02" H 14100 3830 60  0001 L CNN "Val"
+F 15 "0R082" H 14100 3830 60  0001 L CNN "Val"
 F 16 "None" H 14100 3740 60  0001 L CNN "Status"
 F 17 "0.5W" H 14100 3650 60  0001 L CNN "Power"
@@
 F 20 "±1%" H 14100 3380 60  0001 L CNN "Tolerance"
 F 21 "Low Value Flat Chip Resistor" H 14100 3290 60  0001 L CNN "Part Description"
-F 22 "TT Electronics" H 14100 3200 60  0001 L CNN "Manufacturer"
-F 23 "CSR1206FK20L0" H 14100 3110 60  0001 L CNN "Manufacturer Part Number"
+F 22 "Ohmite" H 14100 3200 60  0001 L CNN "Manufacturer"
+F 23 "KDV12DR082ET" H 14100 3110 60  0001 L CNN "Manufacturer Part Number"
 F 24 "1206" H 14100 3020 60  0001 L CNN "Case"
 F 25 "No" H 14100 2930 60  0001 L CNN "PressFit"
@@
 F 37 "CERN DEM JLC" H 14100 1850 60  0001 L CNN "Author"
 F 38 "05/11/10 00:00:00" H 14100 1760 60  0001 L CNN "CreateDate"
-F 39 "09/03/12 00:00:00" H 14100 1670 60  0001 L CNN "LatestRevisionDate"
+F 39 "05/12/20 00:00:00" H 14100 1670 60  0001 L CNN "LatestRevisionDate"
 F 40 "Resistors SMD" H 14100 1580 60  0001 L CNN "Library Name"
 F 41 "This work is licensed under the Creative Commons CC-BY-SA 4.0 License. To the extent that circuit schematics that use Licensed Material can be considered to be ‘Adapted Material’, then the copyright holder waives article 3.b of the license with respect to these schematics." H 14100 1490 60  0001 L CNN "License"
@@
 $EndComp
 $Comp
-L Resistors_SMD:R1206_0R02_1%_0.5W_100PPM R301
+L Resistors_SMD:R1206_0R082_1%_0.5W_100PPM R301
 U 1 1 5EC1B35B
 P 6950 1150
 F 0 "R301" H 7100 1250 50  0000 C CNN
-F 1 "R1206_0R02_1%_0.5W_100PPM" H 6950 940 60  0001 L CNN
+F 1 "R1206_0R082_1%_0.5W_100PPM" H 6950 940 60  0001 L CNN
 F 2 "RESC3216X80N" H 6950 130 60  0001 L CNN
 F 3 "\\\\cern.ch\\dfs\\Applications\\Altium\\Datasheets\\R1206_WELWYN_LRF.pdf" H 6950 760 60  0001 L CNN
-F 4 "0R02" H 7100 1050 50  0000 C CNN "~"
-F 5 "R1206_0R02_1%_0.5W_100PPM" H 6950 670 60  0001 L CNN "Part Number"
+F 4 "0R082" H 7100 1050 50  0000 C CNN "~"
+F 5 "R1206_0R082_1%_0.5W_100PPM" H 6950 670 60  0001 L CNN "Part Number"
 F 6 "Resistor - 1%" H 6950 580 60  0001 L CNN "Library Ref"
 F 7 "SchLib\\Resistors.SchLib" H 6950 490 60  0001 L CNN "Library Path"
@@
 F 13 "PcbLib\\Resistors SMD.PcbLib" H 6950 -140 60  0001 L CNN "Footprint Path"
 F 14 "RESC3216X80N" H 6950 -230 60  0001 L CNN "Footprint Ref"
-F 15 "0R02" H 6950 -320 60  0001 L CNN "Val"
+F 15 "0R082" H 6950 -320 60  0001 L CNN "Val"
 F 16 "None" H 6950 -410 60  0001 L CNN "Status"
 F 17 "0.5W" H 6950 -500 60  0001 L CNN "Power"
@@
 F 20 "±1%" H 6950 -770 60  0001 L CNN "Tolerance"
 F 21 "Low Value Flat Chip Resistor" H 6950 -860 60  0001 L CNN "Part Description"
-F 22 "TT Electronics" H 6950 -950 60  0001 L CNN "Manufacturer"
-F 23 "CSR1206FK20L0" H 6950 -1040 60  0001 L CNN "Manufacturer Part Number"
+F 22 "Ohmite" H 6950 -950 60  0001 L CNN "Manufacturer"
+F 23 "KDV12DR082ET" H 6950 -1040 60  0001 L CNN "Manufacturer Part Number"
 F 24 "1206" H 6950 -1130 60  0001 L CNN "Case"
 F 25 "No" H 6950 -1220 60  0001 L CNN "PressFit"
@@
 F 37 "CERN DEM JLC" H 6950 -2300 60  0001 L CNN "Author"
 F 38 "05/11/10 00:00:00" H 6950 -2390 60  0001 L CNN "CreateDate"
-F 39 "09/03/12 00:00:00" H 6950 -2480 60  0001 L CNN "LatestRevisionDate"
+F 39 "05/12/20 00:00:00" H 6950 -2480 60  0001 L CNN "LatestRevisionDate"
 F 40 "Resistors SMD" H 6950 -2570 60  0001 L CNN "Library Name"
 F 41 "This work is licensed under the Creative Commons CC-BY-SA 4.0 License. To the extent that circuit schematics that use Licensed Material can be considered to be ‘Adapted Material’, then the copyright holder waives article 3.b of the license with respect to these schematics." H 6950 -2660 60  0001 L CNN "License"

Commit message: Turn R301 into a triple
with R302 and R303, net sense resistor value 0.0273 Ohms.
With the INA219 set to a full-scale of 80 mV, that will yield 2.93 Amps full-scale.
Have the option to go up from there by a factor of two and still be safe.
Parts:
- added R302, R303: R1206_0R082_1%_0.5W_100PPM, RESC3216X80N, symbol Resistors_SMD:R1206_0R082_1%_0.5W_100PPM
Connections:
- wire segments 253 -> 262
Other:
- moved on the sheet: C380, U43

Commit message: Add six test points
Parts:
- added TP1, TP2: TestPoint, Marble:TestPoint_Pad_D1.0mm, symbol Connector_Generic:TestPoint
Connections:
- wire segments 262 -> 266
Other:
- note added: "+12V can be supplied by any one of:\n * barrel jack\n * AMC connector\n * POE module\n"
- note removed: "+12V can be supplied by:\n * barrel jack\n * AMC connector\n * POE module\n"
Changed lines of the file:
@@
 	9500 9400 9700 9400
 Wire Wire Line
-	7900 8450 8650 8450
+	7900 8450 8350 8450
 Connection ~ 7900 8450
 Text HLabel 11500 8350 0    50   Input ~ 10
@@
 	7800 1450 7800 1350
 Text Notes 3000 1100 0    50   ~ 0
-+12V can be supplied by:\n  * barrel jack\n  * AMC connector\n  * POE module\n
++12V can be supplied by any one of:\n  * barrel jack\n  * AMC connector\n  * POE module\n
 Wire Wire Line
 	3600 1850 4000 1850
@@
 --->
 Wire Wire Line
-	4000 1150 6400 1150
+	4000 1150 6000 1150
 Wire Wire Line
 	6400 1150 6400 1450
@@
 Wire Wire Line
 	6400 1450 6400 1750
+Connection ~ 6400 1450
+$Comp
+L Connector_Generic:TestPoint TP1
+U 1 1 5ECE8EDE
+P 8350 7850
+F 0 "TP1" H 8408 7968 50  0000 L CNN
+F 1 "TestPoint" H 8408 7877 50  0000 L CNN
+F 2 "Marble:TestPoint_Pad_D1.0mm" H 8550 7850 50  0001 C CNN
+F 3 "" H 8550 7850 50  0001 C CNN
+	1    8350 7850
+	1    0    0    -1
+$EndComp
+Wire Wire Line
+	8350 7850 8350 8450
+Connection ~ 8350 8450
+Wire Wire Line
+	8350 8450 8650 8450
+$Comp
+L Connector_Generic:TestPoint TP2
+U 1 1 5ED180B0
+P 6000 950
+F 0 "TP2" H 6058 1068 50  0000 L CNN
+F 1 "TestPoint" H 6058 977 50  0000 L CNN
+F 2 "Marble:TestPoint_Pad_D1.0mm" H 6200 950 50  0001 C CNN
+F 3 "" H 6200 950 50  0001 C CNN
+	1    6000 950
+	1    0    0    -1
+$EndComp
+Wire Wire Line
+	6000 950  6000 1150
 Wire Bus Line
 	2100 8250 2100 9850
-Connection ~ 6400 1450
+Connection ~ 6000 1150
+Wire Wire Line
+	6000 1150 6400 1150
 $EndSCHEMATC

Commit message: Add four more testpoints to power nets
Parts:
- added TP10: TestPoint, Marble:TestPoint_Pad_D1.0mm, symbol Connector_Generic:TestPoint
Connections:
- wire segments 266 -> 268
Changed lines of the file:
@@
 	7000 4050 7350 4050
 Wire Wire Line
-	7350 4600 7350 4050
+	7350 4600 7350 4250
 Wire Wire Line
 	6600 4050 6300 4050
@@
 Wire Wire Line
 	6000 950  6000 1150
-Wire Bus Line
-	2100 8250 2100 9850
 Connection ~ 6000 1150
 Wire Wire Line
 	6000 1150 6400 1150
+$Comp
+L Connector_Generic:TestPoint TP10
+U 1 1 5ED1928E
+P 7600 4250
+F 0 "TP10" H 7658 4368 50  0000 L CNN
+F 1 "TestPoint" H 7658 4277 50  0000 L CNN
+F 2 "Marble:TestPoint_Pad_D1.0mm" H 7800 4250 50  0001 C CNN
+F 3 "" H 7800 4250 50  0001 C CNN
+	1    7600 4250
+	1    0    0    -1
+$EndComp
+Wire Wire Line
+	7600 4250 7350 4250
+Wire Bus Line
+	2100 8250 2100 9850
+Connection ~ 7350 4250
+Wire Wire Line
+	7350 4250 7350 4050
 $EndSCHEMATC

Commit message: Convert all footprints to use Marble nickname
Includes both .sch and .lib files
Includes both bare footprint names and those with CERN-like nicknames
Parts:
- C128, C130, C131, C134, C135, C357: footprint CAPC1005X55N -> Marble:CAPC1005X55N
- C129: footprint CAPC1709X95N -> Marble:CAPC1709X95N
- C132: footprint CAPC1709X100N -> Marble:CAPC1709X100N
- C133, C136, C351, C380: footprint CAPC0603X33N -> Marble:CAPC0603X33N
- C350: footprint CAPAE830X1020N -> Marble:CAPAE830X1020N
- C353, C354: footprint CAPR500-250X720X650 -> Marble:CAPR500-250X720X650
- D12, D4: footprint DIOM5127X229N -> Marble:DIOM5127X229N
- D6, D7: footprint ICs And Semiconductors SMD:SOIC254P665X290-4N -> Marble:SOIC254P665X290-4N
- D8: footprint ICs And Semiconductors SMD:DIOM5226X262N -> Marble:DIOM5226X262N
- D9: footprint ICs And Semiconductors SMD:SOD2512X110N -> Marble:SOD2512X110N
- J1: footprint Miscellaneous THD:CLIFF_FC68148(DC-10A) -> Marble:CLIFF_FC68148(DC-10A)
- L13: footprint IND_TDK_VLCF5020-1 -> Marble:IND_TDK_VLCF5020-1
- L35, L36, L37, L38, L39, L40: footprint Inductors SMD:INDC2012X145N -> Marble:INDC2012X145N
- LD1, LD2: footprint ICs And Semiconductors SMD:LED_KINGBRIGHT_KPH-1608CGCK -> Marble:LED_KINGBRIGHT_KPH-1608CGCK
- Q1, Q15, Q22: footprint SOTFL50P160X60-6N -> Marble:SOTFL50P160X60-6N
- Q16, Q2, Q23, Q3, Q4: footprint ICs And Semiconductors SMD:SOIC127P600X175-8N -> Marble:SOIC127P600X175-8N
- Q25: footprint ICs And Semiconductors SMD:SOT95P237X112-3N -> Marble:SOT95P237X112-3N
- Q8, Q9: footprint ICs And Semiconductors SMD:SOT95P240X110-3N -> Marble:SOT95P240X110-3N
- R104, R107, R108, R109, R110, R170, R171, R179, R180, R181, R184, R188, R197, R198, R201, R202, R203, R212, R213, R214, R235, R236, R281: footprint RESC1005X40N -> Marble:RESC1005X40N
- R111: footprint RESC3216X65N -> Marble:RESC3216X65N
- R182, R183, R301, R302, R303: footprint RESC3216X80N -> Marble:RESC3216X80N
- U17, U32: footprint ICs And Semiconductors SMD:SOT65P280X145-8N -> Marble:SOT65P280X145-8N
- U18: footprint SON50P200X300X80-11N-R94X250 -> Marble:SON50P200X300X80-11N-R94X250
- U41: footprint FAIRCHILD_FOD817DSD -> Marble:FAIRCHILD_FOD817DSD

Commit message: Clean up BSS138 instances in schematic
Q5 Q6 Q8 Q9 Q14 Q17 Q18 Q19 Q20 Q21 Q24
Fewer warnings from KiBoM
Parts:
- Q8, Q9: Comment =Device -> BSS138LT1G; ComponentLink1Description ~~ -> (none); ComponentLink2Description ~~ -> (none); Database Table Name (none) -> Transistors; Footprint Library (none) -> ICs And Semiconductors SMD; Library Name ICs And Semiconductors SMD -> ICs And Semiconductors.DbLib; SCEM (none) -> (none); Sense Comment ~~ -> (none); Status ~~ -> (none); Status Comment ~~ -> (none)
Changed lines of the file:
@@
 F 5 "N-MOSFET-D 1G 2S 3D" H 12150 4380 60  0001 L CNN "Library Ref"
 F 6 "SchLib\\Transistors.SchLib" H 12150 4290 60  0001 L CNN "Library Path"
-F 7 "=Device" H 12150 4200 60  0001 L CNN "Comment"
+F 7 "BSS138LT1G" H 12150 4200 60  0001 L CNN "Comment"
 F 8 "Standard" H 12150 4110 60  0001 L CNN "Component Kind"
 F 9 "Standard" H 12150 4020 60  0001 L CNN "Component Type"
 F 10 "BSS138LT1G" H 12150 3930 60  0001 L CNN "Device"
 F 11 "SOT23 3-Leads, Pitch 0.95mm - Body 1.4x3mm, IPC Medium Density" H 12150 3750 60  0001 L CNN "PackageDescription"
-F 12 "~~" H 12150 3660 60  0001 L CNN "Status"
+F 12 " " H 12150 3660 60  0001 L CNN "Status"
 F 13 "50V 200mA N-Channel Enhancement Mode Field-Effect Transistor" H 12150 3570 60  0001 L CNN "Part Description"
 F 14 "ON SEMICONDUCTOR" H 12150 3480 60  0001 L CNN "Manufacturer"
@@
 F 21 "Yes" H 12150 2850 60  0001 L CNN "SMD"
 F 22 "No" H 12150 2760 60  0001 L CNN "Sense"
-F 23 "~~" H 12150 2670 60  0001 L CNN "Sense Comment"
+F 23 " " H 12150 2670 60  0001 L CNN "Sense Comment"
 F 24 "No" H 12150 2580 60  0001 L CNN "Bonding"
-F 25 "~~" H 12150 2490 60  0001 L CNN "Status Comment"
+F 25 " " H 12150 2490 60  0001 L CNN "Status Comment"
 F 26 "1.11mm" H 12150 2400 60  0001 L CNN "ComponentHeight"
 F 27 "PcbLib\\ICs And Semiconductors SMD.PcbLib" H 12150 2310 60  0001 L CNN "Footprint Path"
@@
 F 29 "\\\\cern.ch\\dfs\\Applications\\Altium\\Datasheets\\BSS138LT1G.pdf" H 12150 2130 60  0001 L CNN "HelpURL"
 F 30 "~~" H 12150 2040 60  0001 L CNN "ComponentLink1URL"
-F 31 "~~" H 12150 1950 60  0001 L CNN "ComponentLink1Description"
+F 31 " " H 12150 1950 60  0001 L CNN "ComponentLink1Description"
 F 32 "~~" H 12150 1860 60  0001 L CNN "ComponentLink2URL"
-F 33 "~~" H 12150 1770 60  0001 L CNN "ComponentLink2Description"
+F 33 " " H 12150 1770 60  0001 L CNN "ComponentLink2Description"
 F 34 "CERN DEM JLC" H 12150 1680 60  0001 L CNN "Author"
 F 35 "03/23/09 00:00:00" H 12150 1590 60  0001 L CNN "CreateDate"
 F 36 "03/23/09 00:00:00" H 12150 1500 60  0001 L CNN "LatestRevisionDate"
-F 37 "ICs And Semiconductors SMD" H 12150 1410 60  0001 L CNN "Library Name"
+F 37 "ICs And Semiconductors.DbLib" H 12150 1410 60  0001 L CNN "Library Name"
 F 38 "This work is licensed under the Creative Commons CC-BY-SA 4.0 License. To the extent that circuit schematics that use Licensed Material can be considered to be ‘Adapted Material’, then the copyright holder waives article 3.b of the license with respect to these schematics." H 12150 1320 60  0001 L CNN "License"
+F 39 "Transistors" H 12150 5050 50  0001 C CNN "Database Table Name"
+F 40 "ICs And Semiconductors SMD" H 12150 5050 50  0001 C CNN "Footprint Library"
+F 41 " " H 12150 5050 50  0001 C CNN "SCEM"
 	1    12150 5050
 	1    0    0    -1
@@
 F 5 "N-MOSFET-D 1G 2S 3D" H 12150 980 60  0001 L CNN "Library Ref"
 F 6 "SchLib\\Transistors.SchLib" H 12150 890 60  0001 L CNN "Library Path"
-F 7 "=Device" H 12150 800 60  0001 L CNN "Comment"
+F 7 "BSS138LT1G" H 12150 800 60  0001 L CNN "Comment"
 F 8 "Standard" H 12150 710 60  0001 L CNN "Component Kind"
 F 9 "Standard" H 12150 620 60  0001 L CNN "Component Type"
 F 10 "BSS138LT1G" H 12150 530 60  0001 L CNN "Device"
 F 11 "SOT23 3-Leads, Pitch 0.95mm - Body 1.4x3mm, IPC Medium Density" H 12150 350 60  0001 L CNN "PackageDescription"
-F 12 "~~" H 12150 260 60  0001 L CNN "Status"
+F 12 " " H 12150 260 60  0001 L CNN "Status"
 F 13 "50V 200mA N-Channel Enhancement Mode Field-Effect Transistor" H 12150 170 60  0001 L CNN "Part Description"
 F 14 "ON SEMICONDUCTOR" H 12150 80  60  0001 L CNN "Manufacturer"
@@
 F 21 "Yes" H 12150 -550 60  0001 L CNN "SMD"
 F 22 "No" H 12150 -640 60  0001 L CNN "Sense"
-F 23 "~~" H 12150 -730 60  0001 L CNN "Sense Comment"
+F 23 " " H 12150 -730 60  0001 L CNN "Sense Comment"
 F 24 "No" H 12150 -820 60  0001 L CNN "Bonding"
-F 25 "~~" H 12150 -910 60  0001 L CNN "Status Comment"
+F 25 " " H 12150 -910 60  0001 L CNN "Status Comment"
 F 26 "1.11mm" H 12150 -1000 60  0001 L CNN "ComponentHeight"
 F 27 "PcbLib\\ICs And Semiconductors SMD.PcbLib" H 12150 -1090 60  0001 L CNN "Footprint Path"
@@
 F 29 "\\\\cern.ch\\dfs\\Applications\\Altium\\Datasheets\\BSS138LT1G.pdf" H 12150 -1270 60  0001 L CNN "HelpURL"
 F 30 "~~" H 12150 -1360 60  0001 L CNN "ComponentLink1URL"
-F 31 "~~" H 12150 -1450 60  0001 L CNN "ComponentLink1Description"
+F 31 " " H 12150 -1450 60  0001 L CNN "ComponentLink1Description"
 F 32 "~~" H 12150 -1540 60  0001 L CNN "ComponentLink2URL"
-F 33 "~~" H 12150 -1630 60  0001 L CNN "ComponentLink2Description"
+F 33 " " H 12150 -1630 60  0001 L CNN "ComponentLink2Description"
 F 34 "CERN DEM JLC" H 12150 -1720 60  0001 L CNN "Author"
 F 35 "03/23/09 00:00:00" H 12150 -1810 60  0001 L CNN "CreateDate"
 F 36 "03/23/09 00:00:00" H 12150 -1900 60  0001 L CNN "LatestRevisionDate"
-F 37 "ICs And Semiconductors SMD" H 12150 -1990 60  0001 L CNN "Library Name"
+F 37 "ICs And Semiconductors.DbLib" H 12150 -1990 60  0001 L CNN "Library Name"
 F 38 "This work is licensed under the Creative Commons CC-BY-SA 4.0 License. To the extent that circuit schematics that use Licensed Material can be considered to be ‘Adapted Material’, then the copyright holder waives article 3.b of the license with respect to these schematics." H 12150 -2080 60  0001 L CNN "License"
+F 39 "Transistors" H 12150 1650 50  0001 C CNN "Database Table Name"
+F 40 "ICs And Semiconductors SMD" H 12150 1650 50  0001 C CNN "Footprint Library"
+F 41 " " H 12150 1650 50  0001 C CNN "SCEM"
 	1    12150 1650
 	1    0    0    -1
@@
 Wire Wire Line
 	7600 4250 7350 4250
+Connection ~ 7350 4250
+Wire Wire Line
+	7350 4250 7350 4050
 Wire Bus Line
 	2100 8250 2100 9850
-Connection ~ 7350 4250
-Wire Wire Line
-	7350 4250 7350 4050
 $EndSCHEMATC
