File: Power.sch (KiCad schematic (older format))
At the start: 80 parts, among them J1 CLIFF_FC68148(DC-10A), Q1 BC857BV, Q15 BC857BV, Q16 SI4425DDY-T1-GE3, Q2 SI4425DDY-T1-GE3, Q22 BC857BV, Q23 SI4425DDY-T1-GE3, Q25 Si2315BDS-T1-E3, Q3 SI4425DDY-T1-GE3, Q4 SI4425DDY-T1-GE3, Q8 BSS138LT1G, Q9 BSS138LT1G, U17 INA219BIDCNT, U18 TPS62175DQC, U32 INA219BIDCNT, U40 AG5300, U41 FOD817DSD, U43 INA219BIDCNT

Commit message: Get rid of most .DbLib suffixes in Library Name attributes
Enough that KiBoM no longer complains about them
Parts:
- Q8, Q9, U43: Library Name ICs And Semiconductors.DbLib -> ICs And Semiconductors SMD
Changed lines of the file:
@@
 F 35 "03/23/09 00:00:00" H 12150 1590 60  0001 L CNN "CreateDate"
 F 36 "03/23/09 00:00:00" H 12150 1500 60  0001 L CNN "LatestRevisionDate"
-F 37 "ICs And Semiconductors.DbLib" H 12150 1410 60  0001 L CNN "Library Name"
+F 37 "ICs And Semiconductors SMD" H 12150 1410 60  0001 L CNN "Library Name"
 F 38 "This work is licensed under the Creative Commons CC-BY-SA 4.0 License. To the extent that circuit schematics that use Licensed Material can be considered to be ‘Adapted Material’, then the copyright holder waives article 3.b of the license with respect to these schematics." H 12150 1320 60  0001 L CNN "License"
 F 39 "Transistors" H 12150 5050 50  0001 C CNN "Database Table Name"
@@
 F 35 "03/23/09 00:00:00" H 12150 -1810 60  0001 L CNN "CreateDate"
 F 36 "03/23/09 00:00:00" H 12150 -1900 60  0001 L CNN "LatestRevisionDate"
-F 37 "ICs And Semiconductors.DbLib" H 12150 -1990 60  0001 L CNN "Library Name"
+F 37 "ICs And Semiconductors SMD" H 12150 -1990 60  0001 L CNN "Library Name"
 F 38 "This work is licensed under the Creative Commons CC-BY-SA 4.0 License. To the extent that circuit schematics that use Licensed Material can be considered to be ‘Adapted Material’, then the copyright holder waives article 3.b of the license with respect to these schematics." H 12150 -2080 60  0001 L CNN "License"
 F 39 "Transistors" H 12150 1650 50  0001 C CNN "Database Table Name"
@@
 F 35 "09/24/13 00:00:00" H 7600 -2290 60  0001 L CNN "CreateDate"
 F 36 "09/24/13 00:00:00" H 7600 -2380 60  0001 L CNN "LatestRevisionDate"
-F 37 "ICs And Semiconductors.DbLib" H 7600 -2470 60  0001 L CNN "Library Name"
+F 37 "ICs And Semiconductors SMD" H 7600 -2470 60  0001 L CNN "Library Name"
 F 38 "This work is licensed under the Creative Commons CC-BY-SA 4.0 License. To the extent that circuit schematics that use Licensed Material can be considered to be ‘Adapted Material’, then the copyright holder waives article 3.b of the license with respect to these schematics." H 7600 -2560 60  0001 L CNN "License"
 F 39 "Analog & Interface" H 7600 1850 50  0001 C CNN "Database Table Name"
