File: Power.sch (KiCad schematic (older format))
At the start: 80 parts, among them J1 CLIFF_FC68148(DC-10A), Q1 BC857BV, Q15 BC857BV, Q16 SI4425DDY-T1-GE3, Q2 SI4425DDY-T1-GE3, Q22 BC857BV, Q23 SI4425DDY-T1-GE3, Q25 Si2315BDS-T1-E3, Q3 SI4425DDY-T1-GE3, Q4 SI4425DDY-T1-GE3, Q8 BSS138LT1G, Q9 BSS138LT1G, U17 INA219BIDCNT, U18 TPS62175DQC, U32 INA219BIDCNT, U40 AG5300, U41 FOD817DSD, U43 INA219BIDCNT

Commit message: Manufacturer Part Number clean-up
Convert Manufacturer Part Number BAT165AX to BAT165
The AX suffix refers to Nexperia, and the Manufacturer we list is Infineon.
Digi-Key has both Nexperia BAT165AX and Infineon BAT165E6327HTSA1 in stock, and the two are fungible to us

Get rid of stray ,115 after BC857BV in a couple of places
Parts:
- D9: Manufacturer Part Number BAT165AX -> BAT165
- Q1, Q15: Manufacturer Part Number BC857BV,115 -> BC857BV
Changed lines of the file:
@@
 F 13 "-45V -100mA PNP General Purpose Double Transistor" H 6550 3270 60  0001 L CNN "Part Description"
 F 14 "NXP SEMICONDUCTORS" H 6550 3180 60  0001 L CNN "Manufacturer"
-F 15 "BC857BV,115" H 6550 3090 60  0001 L CNN "Manufacturer Part Number"
+F 15 "BC857BV" H 6550 3090 60  0001 L CNN "Manufacturer Part Number"
 F 16 "6" H 6550 3000 60  0001 L CNN "Pin Count"
 F 17 "SOT666" H 6550 2910 60  0001 L CNN "Case"
@@
 F 13 "-45V -100mA PNP General Purpose Double Transistor" H 7100 3270 60  0001 L CNN "Part Description"
 F 14 "NXP SEMICONDUCTORS" H 7100 3180 60  0001 L CNN "Manufacturer"
-F 15 "BC857BV,115" H 7100 3090 60  0001 L CNN "Manufacturer Part Number"
+F 15 "BC857BV" H 7100 3090 60  0001 L CNN "Manufacturer Part Number"
 F 16 "6" H 7100 3000 60  0001 L CNN "Pin Count"
 F 17 "SOT666" H 7100 2910 60  0001 L CNN "Case"
@@
 F 13 "-45V -100mA PNP General Purpose Double Transistor" H 2800 1070 60  0001 L CNN "Part Description"
 F 14 "NXP SEMICONDUCTORS" H 2800 980 60  0001 L CNN "Manufacturer"
-F 15 "BC857BV,115" H 2800 890 60  0001 L CNN "Manufacturer Part Number"
+F 15 "BC857BV" H 2800 890 60  0001 L CNN "Manufacturer Part Number"
 F 16 "6" H 2800 800 60  0001 L CNN "Pin Count"
 F 17 "SOT666" H 2800 710 60  0001 L CNN "Case"
@@
 F 13 "-45V -100mA PNP General Purpose Double Transistor" H 3350 1070 60  0001 L CNN "Part Description"
 F 14 "NXP SEMICONDUCTORS" H 3350 980 60  0001 L CNN "Manufacturer"
-F 15 "BC857BV,115" H 3350 890 60  0001 L CNN "Manufacturer Part Number"
+F 15 "BC857BV" H 3350 890 60  0001 L CNN "Manufacturer Part Number"
 F 16 "6" H 3350 800 60  0001 L CNN "Pin Count"
 F 17 "SOT666" H 3350 710 60  0001 L CNN "Case"
@@
 F 15 "Medium Power AF Schottky Diode" H 5300 1410 60  0001 L CNN "Part Description"
 F 16 "INFINEON" H 5300 1320 60  0001 L CNN "Manufacturer"
-F 17 "BAT165AX" H 5300 1230 60  0001 L CNN "Manufacturer Part Number"
+F 17 "BAT165" H 5300 1230 60  0001 L CNN "Manufacturer Part Number"
 F 18 "2" H 5300 1140 60  0001 L CNN "Pin Count"
 F 19 "SOD323" H 5300 1050 60  0001 L CNN "Case"

Commit message: More attribute fixes
Fix up Attribute names in HDT0001 and AG5300
Remove stray attribute for SN65MLVD2DRBT (added in last commit)
Parts:
- U40: Manufacturer (none) -> Silvertel; Manufacturer_Name Silvertel -> (none); Manufacturer_Part_Number AG5300 -> (none)
Changed lines of the file:
@@
 F 4 "Power-over-Ethernet Plus Module" H 6700 8200 50  0001 L CNN "Description"
 F 5 "14" H 6700 8100 50  0001 L CNN "Height"
-F 6 "Silvertel" H 6700 7900 50  0001 L CNN "Manufacturer_Name"
+F 6 "Silvertel" H 6700 7900 50  0001 L CNN "Manufacturer"
 F 7 "AG5300" H 6700 7800 50  0001 L CNN "Manufacturer Part Number"
-F 8 "AG5300" H 5550 8300 50  0001 C CNN "Manufacturer_Part_Number"
 	1    5550 8300
 	1    0    0    -1

Commit message: Upgrade voltage rating on 0402 100nF
Convert 16 caps from CC0402_100NF_16V_10%_X5R to CC0402_100NF_25V_10%_X5R
C5 C61 C128 C130 C131 C134 C135 C137 C140 C147 C148 C149 C150 C357 C362 C363
Samsung CL05A104KA5NNNC, $0.00658 in 500s at Digi-Key
Parts:
- C128, C130, C131, C134, C135, C357: value CC0402_100NF_16V_10%_X5R -> CC0402_100NF_25V_10%_X5R; symbol Capacitors_SMD:CC0402_100NF_16V_10%_X5R -> Capacitors_SMD:CC0402_100NF_25V_10%_X5R; Manufacturer Part Number CC0402_100NF_16V_10%_X5R -> CC0402_100NF_25V_10%_X5R; Manufacturer1 Example MURATA -> Samsung; Manufacturer1 Part Number GRM155R61C104KA88D -> CL05A104KA5NNNC; Part Number CC0402_100NF_16V_10%_X5R -> CC0402_100NF_25V_10%_X5R; Voltage 16V -> 25V

Commit message: Upgrade voltage rating on 0603 4.7uF
Convert 26 caps from CC0603_4.7UF_16V_10%_X5R to CC0603_4.7UF_25V_10%_X5R
C57 C103 C105 C127 C129 C139 C142 C143 C144 C159 C161 C162 C167 C168 C173 C195 C331 C343 C344 C347 C348 C349 C360 C361 C364 C373
Samsung CL10A475KA8NQN, $0.11456 in 500s at Digi-Key
Parts:
- C129: value CC0603_4.7UF_16V_10%_X5R -> CC0603_4.7UF_25V_10%_X5R; symbol Capacitors_SMD:CC0603_4.7UF_16V_10%_X5R -> Capacitors_SMD:CC0603_4.7UF_25V_10%_X5R; Manufacturer Part Number CC0603_4.7UF_16V_10%_X5R -> CC0603_4.7UF_25V_10%_X5R; Manufacturer1 Example TAIYO YUDEN -> Samsung; Manufacturer1 Part Number EMK107ABJ475KA-T -> CL10A475KA8NQN; Part Number CC0603_4.7UF_16V_10%_X5R -> CC0603_4.7UF_25V_10%_X5R; Voltage 16V -> 25V
Changed lines of the file:
@@
 $EndComp
 $Comp
-L Capacitors_SMD:CC0603_4.7UF_16V_10%_X5R C?
+L Capacitors_SMD:CC0603_4.7UF_25V_10%_X5R C?
 U 1 1 5C7A3EEE
 P 2250 4050
@@
 AR Path="/5C16BF8E/5C7A3EEE" Ref="C129"  Part="1"
 F 0 "C129" V 2300 4050 50  0000 L CNN
-F 1 "CC0603_4.7UF_16V_10%_X5R" H 2250 3790 60  0001 L CNN
+F 1 "CC0603_4.7UF_25V_10%_X5R" H 2250 3790 60  0001 L CNN
 F 2 "Marble:CAPC1709X95N" H 2250 2980 60  0001 L CNN
 F 3 "\\\\cern.ch\\dfs\\Applications\\Altium\\Datasheets\\CC0603_X7R_TAIYO-YUDEN_HIGH-VALUE.pdf" H 2250 3610 60  0001 L CNN
 F 4 "4.7uF" V 2500 4050 50  0000 L CNN "Val"
-F 5 "CC0603_4.7UF_16V_10%_X5R" H 2250 3520 60  0001 L CNN "Part Number"
+F 5 "CC0603_4.7UF_25V_10%_X5R" H 2250 3520 60  0001 L CNN "Part Number"
 F 6 "Capacitor - non polarized" H 2250 3430 60  0001 L CNN "Library Ref"
 F 7 "SchLib\\Capacitors.SchLib" H 2250 3340 60  0001 L CNN "Library Path"
@@
 F 15 "None" H 2250 2440 60  0001 L CNN "Status"
 F 16 " " H 2250 2350 60  0001 L CNN "Status Comment"
-F 17 "16V" H 2250 2260 60  0001 L CNN "Voltage"
+F 17 "25V" H 2250 2260 60  0001 L CNN "Voltage"
 F 18 "X5R" H 2250 2170 60  0001 L CNN "TC"
 F 19 "±10%" H 2250 2080 60  0001 L CNN "Tolerance"
 F 20 "SMD Multilayer Chip Ceramic Capacitor" H 2250 1990 60  0001 L CNN "Part Description"
 F 21 "GENERIC" H 2250 1900 60  0001 L CNN "Manufacturer"
-F 22 "CC0603_4.7UF_16V_10%_X5R" H 2250 1810 60  0001 L CNN "Manufacturer Part Number"
+F 22 "CC0603_4.7UF_25V_10%_X5R" H 2250 1810 60  0001 L CNN "Manufacturer Part Number"
 F 23 "0603" H 2250 1720 60  0001 L CNN "Case"
 F 24 "Yes" H 2250 1630 60  0001 L CNN "Mounted"
@@
 F 29 " " H 2250 1180 60  0001 L CNN "Sense Comment"
 F 30 " " H 2250 1090 60  0001 L CNN "ComponentHeight"
-F 31 "TAIYO YUDEN" H 2250 1000 60  0001 L CNN "Manufacturer1 Example"
-F 32 "EMK107ABJ475KA-T" H 2250 910 60  0001 L CNN "Manufacturer1 Part Number"
+F 31 "Samsung" H 2250 1000 60  0001 L CNN "Manufacturer1 Example"
+F 32 "CL10A475KA8NQN" H 2250 910 60  0001 L CNN "Manufacturer1 Part Number"
 F 33 "0.95mm" H 2250 820 60  0001 L CNN "Manufacturer1 ComponentHeight"
 F 34 "CERN DEM JLC" H 2250 640 60  0001 L CNN "Author"

Commit message: List more Manufacturers
Parts:
- L35, L37, L39: Manufacturer (none) -> TDK
Changed lines of the file:
@@
 F 3 " " H 4250 8650 50  0001 C CNN
 F 4 "MPZ2012S102A" V 4250 8650 50  0001 C CNN "Manufacturer Part Number"
+F 5 "TDK" V 4250 8650 50  0001 C CNN "Manufacturer"
 	1    4250 8650
 	0    -1   -1   0
@@
 F 3 " " H 4750 8650 50  0001 C CNN
 F 4 "MPZ2012S102A" V 4750 8650 50  0001 C CNN "Manufacturer Part Number"
+F 5 "TDK" V 4750 8650 50  0001 C CNN "Manufacturer"
 	1    4750 8650
 	0    -1   -1   0
@@
 F 3 " " H 5250 8650 50  0001 C CNN
 F 4 "MPZ2012S102A" V 5250 8650 50  0001 C CNN "Manufacturer Part Number"
+F 5 "TDK" V 5250 8650 50  0001 C CNN "Manufacturer"
 	1    5250 8650
 	0    -1   -1   0

Commit message: More part number progress
Parts:
- D6, D7: Manufacturer (none) -> SMC; Manufacturer Part Number MB210S-TP -> KMB210STR
- D8: Manufacturer (none) -> DIODES INC; Manufacturer Part Number SMAJ58A -> SMAJ58A-13-F
Changed lines of the file:
@@
 F 2 "Marble:SOIC254P665X290-4N" H 3400 8775 50  0001 L CNN
 F 3 "http://www.vishay.com/docs/88573/dfs.pdf" H 3250 8650 50  0001 C CNN
-F 4 "MB210S-TP" H 3250 8650 50  0001 C CNN "Manufacturer Part Number"
+F 4 "KMB210STR" H 3250 8650 50  0001 C CNN "Manufacturer Part Number"
+F 5 "SMC" H 3250 8650 50  0001 C CNN "Manufacturer"
 	1    3250 8650
 	1    0    0    -1
@@
 F 2 "Marble:SOIC254P665X290-4N" H 3400 9775 50  0001 L CNN
 F 3 "http://www.vishay.com/docs/88573/dfs.pdf" H 3250 9650 50  0001 C CNN
-F 4 "MB210S-TP" H 3250 9650 50  0001 C CNN "Manufacturer Part Number"
+F 4 "KMB210STR" H 3250 9650 50  0001 C CNN "Manufacturer Part Number"
+F 5 "SMC" H 3250 9650 50  0001 C CNN "Manufacturer"
 	1    3250 9650
 	1    0    0    -1
@@
 F 2 "Marble:DIOM5226X262N" H 3600 8650 50  0001 C CNN
 F 3 "https://www.vishay.com/docs/88301/15ke.pdf" H 3550 8850 50  0001 C CNN
-F 4 "SMAJ58A" H 3600 8850 50  0001 C CNN "Manufacturer Part Number"
+F 4 "SMAJ58A-13-F" H 3600 8850 50  0001 C CNN "Manufacturer Part Number"
+F 5 "DIODES INC" H 3600 8850 50  0001 C CNN "Manufacturer"
 	1    3600 8850
 	0    1    1    0

Commit message: A little more clarity on Manufacturer and Part Number
Adjustments to DDR3 memory, a resistor, and a push-button
Parts:
- R111: Manufacturer YAGEO PHYCOMP -> YAGEO; Manufacturer Part Number RL1206FR-7W0R47 (35051914707) -> RL1206FR-7W0R47L
Changed lines of the file:
@@
 F 19 "±1%" H 5200 -270 60  0001 L CNN "Tolerance"
 F 20 "Low Ohmique High Power Chip Resistor" H 5200 -360 60  0001 L CNN "Part Description"
-F 21 "YAGEO PHYCOMP" H 5200 -450 60  0001 L CNN "Manufacturer"
-F 22 "RL1206FR-7W0R47  (35051914707)" H 5200 -540 60  0001 L CNN "Manufacturer Part Number"
+F 21 "YAGEO" H 5200 -450 60  0001 L CNN "Manufacturer"
+F 22 "RL1206FR-7W0R47L" H 5200 -540 60  0001 L CNN "Manufacturer Part Number"
 F 23 "1206" H 5200 -630 60  0001 L CNN "Case"
 F 24 "No" H 5200 -720 60  0001 L CNN "PressFit"

Commit message: Mark more parts +standalone, like 8P8C and PoE
J1 J4 J15 U40 C353 C354 Cage1
Many others are also possible, but would make rework much harder, so don't do that now
R220 C37 R217 R218 Q20 Q21 D10 D11 R141 R164 R206 R207 R208 R211 R219 R226
U41 R281 D6 D7 D8 L35 L36 L37 L38 L39 L40 C350 D12
Parts:
- C353, C354, U40: config (none) -> +standalone
Changed lines of the file:
@@
 F 6 "Silvertel" H 6700 7900 50  0001 L CNN "Manufacturer"
 F 7 "AG5300" H 6700 7800 50  0001 L CNN "Manufacturer Part Number"
+F 8 "+standalone" H 5550 8300 50  0001 C CNN "config"
 	1    5550 8300
 	1    0    0    -1
@@
 F 37 "Capacitors THD" H 6200 4520 60  0001 L CNN "Library Name"
 F 38 "This work is licensed under the Creative Commons CC-BY-SA 4.0 License. To the extent that circuit schematics that use Licensed Material can be considered to be ‘Adapted Material’, then the copyright holder waives article 3.b of the license with respect to these schematics." H 6200 4430 60  0001 L CNN "License"
+F 39 "+standalone" H 6200 8200 50  0001 C CNN "config"
 	1    6200 8200
 	1    0    0    -1
@@
 F 37 "Capacitors THD" H 6200 5770 60  0001 L CNN "Library Name"
 F 38 "This work is licensed under the Creative Commons CC-BY-SA 4.0 License. To the extent that circuit schematics that use Licensed Material can be considered to be ‘Adapted Material’, then the copyright holder waives article 3.b of the license with respect to these schematics." H 6200 5680 60  0001 L CNN "License"
+F 39 "+standalone" H 6200 9450 50  0001 C CNN "config"
 	1    6200 9450
 	1    0    0    -1
