File: Power_SW.sch (KiCad schematic (older format))
At the start: 96 parts, among them J9 2057-PH1-04-UA-ND, Q10 FDMS7608S, Q11 FDMS7608S, Q12 FDMS7608S, Q13 FDMS7608S, Q26 BC847BV, Q27 BC847BV, U35 XRP7724ILB-F, U36 NCP186AMX180TAG, U37 NCP186AMX120TAG

Commit message: Rename library AMC_FMC_Carrier-PcbDoc-rescue as marble_misc
Parts:
- J9: symbol AMC_FMC_Carrier-PcbDoc-rescue:Conn_01x04_Male-Connector-AMC_FMC_Carrier-PcbDoc-rescue -> marble_misc:Conn_01x04_Male-Connector-AMC_FMC_Carrier-PcbDoc-rescue
- U36, U37: symbol AMC_FMC_Carrier-PcbDoc-rescue:NCP186AMX120TAG-powerMG-AMC_FMC_Carrier-PcbDoc-rescue -> marble_misc:NCP186AMX120TAG-powerMG-AMC_FMC_Carrier-PcbDoc-rescue
Changed lines of the file:
@@
 	6150 1050 6150 1700
 $Comp
-L AMC_FMC_Carrier-PcbDoc-rescue:Conn_01x04_Male-Connector-AMC_FMC_Carrier-PcbDoc-rescue J?
+L marble_misc:Conn_01x04_Male-Connector-AMC_FMC_Carrier-PcbDoc-rescue J?
 U 1 1 5DBB4777
 P 3900 2700
@@
 $EndComp
 $Comp
-L AMC_FMC_Carrier-PcbDoc-rescue:VCCAUX-powerMG-AMC_FMC_Carrier-PcbDoc-rescue #PWR?
+L marble_misc:VCCAUX-powerMG-AMC_FMC_Carrier-PcbDoc-rescue #PWR?
 U 1 1 5DBB8165
 P 9050 7950
@@
 $EndComp
 $Comp
-L AMC_FMC_Carrier-PcbDoc-rescue:VCCBRAM-powerMG-AMC_FMC_Carrier-PcbDoc-rescue #PWR?
+L marble_misc:VCCBRAM-powerMG-AMC_FMC_Carrier-PcbDoc-rescue #PWR?
 U 1 1 5DBB816B
 P 15300 7600
@@
 $EndComp
 $Comp
-L AMC_FMC_Carrier-PcbDoc-rescue:MGTAVCC-powerMG-AMC_FMC_Carrier-PcbDoc-rescue #PWR?
+L marble_misc:MGTAVCC-powerMG-AMC_FMC_Carrier-PcbDoc-rescue #PWR?
 U 1 1 5DBB8171
 P 15650 7600
@@
 	12650 2350 13550 2350
 $Comp
-L AMC_FMC_Carrier-PcbDoc-rescue:NCP186AMX120TAG-powerMG-AMC_FMC_Carrier-PcbDoc-rescue U?
+L marble_misc:NCP186AMX120TAG-powerMG-AMC_FMC_Carrier-PcbDoc-rescue U?
 U 1 1 5DBB8221
 P 6650 7700
@@
 Connection ~ 7950 10000
 $Comp
-L AMC_FMC_Carrier-PcbDoc-rescue:NCP186AMX120TAG-powerMG-AMC_FMC_Carrier-PcbDoc-rescue U?
+L marble_misc:NCP186AMX120TAG-powerMG-AMC_FMC_Carrier-PcbDoc-rescue U?
 U 1 1 5D300F70
 P 6650 9400
@@
 $EndComp
 $Comp
-L AMC_FMC_Carrier-PcbDoc-rescue:MGTAVTT-powerMG-AMC_FMC_Carrier-PcbDoc-rescue #PWR?
+L marble_misc:MGTAVTT-powerMG-AMC_FMC_Carrier-PcbDoc-rescue #PWR?
 U 1 1 5DBB815F
 P 9050 9650
@@
 NoConn ~ 7550 5100
 $Comp
-L AMC_FMC_Carrier-PcbDoc-rescue:MGTAVTT-powerMG-AMC_FMC_Carrier-PcbDoc-rescue #PWR?
+L marble_misc:MGTAVTT-powerMG-AMC_FMC_Carrier-PcbDoc-rescue #PWR?
 U 1 1 5CF3EE50
 P 3100 6450

Commit message: Strip extraneous AMC_FMC_Carrier-PcbDoc-rescue and powerMG from symbol names
Parts:
- J9: symbol marble_misc:Conn_01x04_Male-Connector-AMC_FMC_Carrier-PcbDoc-rescue -> marble_misc:Conn_01x04_Male-Connector
- U36, U37: symbol marble_misc:NCP186AMX120TAG-powerMG-AMC_FMC_Carrier-PcbDoc-rescue -> marble_misc:NCP186AMX120TAG
Changed lines of the file:
@@
 	6150 1050 6150 1700
 $Comp
-L marble_misc:Conn_01x04_Male-Connector-AMC_FMC_Carrier-PcbDoc-rescue J?
+L marble_misc:Conn_01x04_Male-Connector J?
 U 1 1 5DBB4777
 P 3900 2700
@@
 $EndComp
 $Comp
-L marble_misc:VCCAUX-powerMG-AMC_FMC_Carrier-PcbDoc-rescue #PWR?
+L marble_misc:VCCAUX #PWR?
 U 1 1 5DBB8165
 P 9050 7950
@@
 $EndComp
 $Comp
-L marble_misc:VCCBRAM-powerMG-AMC_FMC_Carrier-PcbDoc-rescue #PWR?
+L marble_misc:VCCBRAM #PWR?
 U 1 1 5DBB816B
 P 15300 7600
@@
 $EndComp
 $Comp
-L marble_misc:MGTAVCC-powerMG-AMC_FMC_Carrier-PcbDoc-rescue #PWR?
+L marble_misc:MGTAVCC #PWR?
 U 1 1 5DBB8171
 P 15650 7600
@@
 	12650 2350 13550 2350
 $Comp
-L marble_misc:NCP186AMX120TAG-powerMG-AMC_FMC_Carrier-PcbDoc-rescue U?
+L marble_misc:NCP186AMX120TAG U?
 U 1 1 5DBB8221
 P 6650 7700
@@
 Connection ~ 7950 10000
 $Comp
-L marble_misc:NCP186AMX120TAG-powerMG-AMC_FMC_Carrier-PcbDoc-rescue U?
+L marble_misc:NCP186AMX120TAG U?
 U 1 1 5D300F70
 P 6650 9400
@@
 $EndComp
 $Comp
-L marble_misc:MGTAVTT-powerMG-AMC_FMC_Carrier-PcbDoc-rescue #PWR?
+L marble_misc:MGTAVTT #PWR?
 U 1 1 5DBB815F
 P 9050 9650
@@
 NoConn ~ 7550 5100
 $Comp
-L marble_misc:MGTAVTT-powerMG-AMC_FMC_Carrier-PcbDoc-rescue #PWR?
+L marble_misc:MGTAVTT #PWR?
 U 1 1 5CF3EE50
 P 3100 6450

Commit message: SCH: rename +3.3VP, 3V3PM and +3V3MP to +3V3P
  * all of them refer to the same net
  * to make confusion perfect, all 3 power symbols on the schematic
    were an instance of the symbol `+3.3VP` with different
    value attributes
  * renamed the `+3.3VP` symbol to `+3V3P` for naming consistency
  * SCH: replaced all power symbols on the net by the new one
  * PCB: still needs to be synced up, as the net name has changed
Connections:
- net labels added: +3V3P
- net labels removed: +3V3MP
Other:
- note added: "D5 for programming supply path\nI2C_PM is forced to ground without +3V3P"
- note removed: "D5 for programming supply path\nI2C_PM is forced to ground without +3V3MP"
Changed lines of the file:
@@
 Connection ~ 4350 2600
 $Comp
-L power:+3.3VP #PWR?
+L power:+3V3P #PWR?
 U 1 1 5DBB47C4
 P 4750 2600
@@
 AR Path="/5DBB47C4" Ref="#PWR0254"  Part="1"
 F 0 "#PWR0254" H 4750 2450 50  0001 C CNN
-F 1 "+3V3MP" V 4750 2850 50  0000 C CNN
+F 1 "+3V3P" V 4750 2850 50  0000 C CNN
 F 2 "" H 4750 2600 50  0001 C CNN
 F 3 "" H 4750 2600 50  0001 C CNN
@@
 	2700 1600 4350 1600
 Text Notes 2050 2650 0    50   ~ 10
-D5 for programming supply path\nI2C_PM is forced to ground without +3V3MP
+D5 for programming supply path\nI2C_PM is forced to ground without +3V3P
 Connection ~ 4350 1900
 $Comp

Commit message: Add six test points
Parts:
- added TP3, TP4, TP5, TP6: TestPoint, Marble:TestPoint_Pad_D1.0mm, symbol Connector_Generic:TestPoint
Connections:
- wire segments 312 -> 319
Changed lines of the file:
@@
 Connection ~ 14400 5950
 Wire Wire Line
-	14400 5950 14700 5950
+	14400 5950 14550 5950
 $Comp
 L power:PWR_FLAG #FLG?
@@
 Connection ~ 14400 4150
 Wire Wire Line
-	14400 4150 14700 4150
+	14400 4150 14550 4150
 $Comp
 L power:PWR_FLAG #FLG?
@@
 Connection ~ 14400 2350
 Wire Wire Line
-	14400 2350 14700 2350
+	14400 2350 14500 2350
 $Comp
 L Diodes:BAT165 D?
@@
 Text Notes 10750 8250 0    50   ~ 0
 RDSon 7.2 mOhms
+$Comp
+L Connector_Generic:TestPoint TP3
+U 1 1 5ED7CF0D
+P 14500 2550
+F 0 "TP3" H 14442 2576 50  0000 R CNN
+F 1 "TestPoint" H 14442 2667 50  0000 R CNN
+F 2 "Marble:TestPoint_Pad_D1.0mm" H 14700 2550 50  0001 C CNN
+F 3 "" H 14700 2550 50  0001 C CNN
+	1    14500 2550
+	-1   0    0    1
+$EndComp
+$Comp
+L Connector_Generic:TestPoint TP4
+U 1 1 5ED7EA90
+P 14550 4300
+F 0 "TP4" H 14492 4326 50  0000 R CNN
+F 1 "TestPoint" H 14492 4417 50  0000 R CNN
+F 2 "Marble:TestPoint_Pad_D1.0mm" H 14750 4300 50  0001 C CNN
+F 3 "" H 14750 4300 50  0001 C CNN
+	1    14550 4300
+	-1   0    0    1
+$EndComp
+$Comp
+L Connector_Generic:TestPoint TP5
+U 1 1 5ED86CAA
+P 14550 6200
+F 0 "TP5" H 14492 6226 50  0000 R CNN
+F 1 "TestPoint" H 14492 6317 50  0000 R CNN
+F 2 "Marble:TestPoint_Pad_D1.0mm" H 14750 6200 50  0001 C CNN
+F 3 "" H 14750 6200 50  0001 C CNN
+	1    14550 6200
+	-1   0    0    1
+$EndComp
+$Comp
+L Connector_Generic:TestPoint TP6
+U 1 1 5ED8D8B0
+P 14650 8250
+F 0 "TP6" H 14592 8276 50  0000 R CNN
+F 1 "TestPoint" H 14592 8367 50  0000 R CNN
+F 2 "Marble:TestPoint_Pad_D1.0mm" H 14850 8250 50  0001 C CNN
+F 3 "" H 14850 8250 50  0001 C CNN
+	1    14650 8250
+	-1   0    0    1
+$EndComp
+Wire Wire Line
+	14650 8000 14650 8250
+Connection ~ 14650 8000
+Wire Wire Line
+	14550 6200 14550 5950
+Connection ~ 14550 5950
+Wire Wire Line
+	14550 5950 14700 5950
+Wire Wire Line
+	14550 4300 14550 4150
+Connection ~ 14550 4150
+Wire Wire Line
+	14550 4150 14700 4150
+Wire Wire Line
+	14500 2550 14500 2350
+Connection ~ 14500 2350
+Wire Wire Line
+	14500 2350 14700 2350
 $EndSCHEMATC

Commit message: Add four more testpoints to power nets
Parts:
- added TP7, TP8: TestPoint, Marble:TestPoint_Pad_D1.0mm, symbol Connector_Generic:TestPoint
Connections:
- wire segments 319 -> 323
Changed lines of the file:
@@
 Connection ~ 7700 8000
 Wire Wire Line
-	8750 8000 9050 8000
+	8750 8000 8900 8000
 Wire Wire Line
 	9050 8000 9050 7950
@@
 Wire Wire Line
 	14500 2350 14700 2350
+$Comp
+L Connector_Generic:TestPoint TP7
+U 1 1 5EC72B65
+P 8900 8150
+F 0 "TP7" H 8842 8176 50  0000 R CNN
+F 1 "TestPoint" H 8842 8267 50  0000 R CNN
+F 2 "Marble:TestPoint_Pad_D1.0mm" H 9100 8150 50  0001 C CNN
+F 3 "" H 9100 8150 50  0001 C CNN
+	1    8900 8150
+	-1   0    0    1
+$EndComp
+$Comp
+L Connector_Generic:TestPoint TP8
+U 1 1 5EC8839F
+P 9500 9800
+F 0 "TP8" H 9442 9826 50  0000 R CNN
+F 1 "TestPoint" H 9442 9917 50  0000 R CNN
+F 2 "Marble:TestPoint_Pad_D1.0mm" H 9700 9800 50  0001 C CNN
+F 3 "" H 9700 9800 50  0001 C CNN
+	1    9500 9800
+	-1   0    0    1
+$EndComp
+Wire Wire Line
+	8900 8150 8900 8000
+Connection ~ 8900 8000
+Wire Wire Line
+	8900 8000 9050 8000
+Wire Wire Line
+	9050 9700 9500 9700
+Wire Wire Line
+	9500 9700 9500 9800
 $EndSCHEMATC

Commit message: Convert all footprints to use Marble nickname
Includes both .sch and .lib files
Includes both bare footprint names and those with CERN-like nicknames
Parts:
- C105, C127, C139, C142, C143, C144, C159, C161, C195, C331, C347, C348, C349, C361: footprint CAPC1709X95N -> Marble:CAPC1709X95N
- C137, C138, C140, C147, C148, C149, C150, C362, C363: footprint CAPC1005X55N -> Marble:CAPC1005X55N
- C141: footprint CAPC3216X180N -> Marble:CAPC3216X180N
- C145, C146: footprint CAPC1709X100N -> Marble:CAPC1709X100N
- C151, C153, C155, C157: footprint CAPC2012X135N -> Marble:CAPC2012X135N
- C152, C154, C156, C158, C160, C194, C330, C340, C341, C345, C346: footprint CAPC2012X140N -> Marble:CAPC2012X140N
- D2, D5: footprint ICs And Semiconductors SMD:SOD2512X110N -> Marble:SOD2512X110N
- J9: footprint Connectors THD:SAMTEC_MTLW-104-07-L-S-250 -> Marble:SAMTEC_MTLW-104-07-L-S-250
- L14, L21, L22, L31, L32: footprint INDC4516X180N -> Marble:INDC4516X180N
- L15, L16, L33, L34: footprint INDC1608X65N -> Marble:INDC1608X65N
- L17, L18, L19, L20: footprint IND_BOURNS_SRP6540 -> Marble:IND_BOURNS_SRP6540
- LD10, LD4, LD5, LD6, LD7, LD8, LD9: footprint ICs And Semiconductors SMD:LED_KINGBRIGHT_KPH-1608CGCK -> Marble:LED_KINGBRIGHT_KPH-1608CGCK
- Q10, Q11, Q12, Q13: footprint FAIRCHILD_MLP08P -> Marble:FAIRCHILD_MLP08P
- Q26, Q27: footprint SOTFL50P160X60-6N -> Marble:SOTFL50P160X60-6N
- R157, R167, R168, R189, R190, R191, R192, R193, R194, R195, R196, R245, R247, R248, R249, R250, R251, R252, R253, R254, R255, R256, R257: footprint RESC1005X40N -> Marble:RESC1005X40N
- U35: footprint ICs And Semiconductors SMD:QFN50P700X700X80-45N-S520 -> Marble:QFN50P700X700X80-45N-S520
- U36, U37: footprint AG5300_2:SOIC-8 -> Marble:SOIC-8

Commit message: Replace Val=DNP with actual value for 6 resistors
Parts:
- R189, R196: ~ DNP -> (none)
Changed lines of the file:
@@
 F 2 "Marble:RESC1005X40N" H 7950 7280 60  0001 L CNN
 F 3 "\\\\cern.ch\\dfs\\Applications\\Altium\\Datasheets\\R0402_Phycomp_RC0402.pdf" H 7950 7910 60  0001 L CNN
-F 4 "DNP" V 8145 8360 50  0000 L CNN "~"
+F 4 "0" V 8145 8360 50  0000 L CNN "Val"
 F 5 "R0402_0R_JUMPER" H 7950 7820 60  0001 L CNN "Part Number"
 F 6 "Resistor" H 7950 7730 60  0001 L CNN "Library Ref"
@@
 F 2 "Marble:RESC1005X40N" H 7950 8980 60  0001 L CNN
 F 3 "\\\\cern.ch\\dfs\\Applications\\Altium\\Datasheets\\R0402_Phycomp_RC0402.pdf" H 7950 9610 60  0001 L CNN
-F 4 "DNP" V 8145 10060 50  0000 L CNN "~"
+F 4 "0" V 8145 10060 50  0000 L CNN "Val"
 F 5 "R0402_0R_JUMPER" H 7950 9520 60  0001 L CNN "Part Number"
 F 6 "Resistor" H 7950 9430 60  0001 L CNN "Library Ref"
