File: Power_SW.sch (KiCad schematic (older format))
At the start: 102 parts, among them J9 2057-PH1-04-UA-ND, Q10 FDMS7608S, Q11 FDMS7608S, Q12 FDMS7608S, Q13 FDMS7608S, Q26 BC847BV, Q27 BC847BV, U35 XRP7724ILB-F, U36 NCP186AMX180TAG, U37 NCP186AMX120TAG

Commit message: Manufacturer Part Number clean-up
Convert Manufacturer Part Number BAT165AX to BAT165
The AX suffix refers to Nexperia, and the Manufacturer we list is Infineon.
Digi-Key has both Nexperia BAT165AX and Infineon BAT165E6327HTSA1 in stock, and the two are fungible to us

Get rid of stray ,115 after BC857BV in a couple of places
Parts:
- D2, D5: Manufacturer Part Number BAT165AX -> BAT165
Changed lines of the file:
@@
 F 15 "Medium Power AF Schottky Diode" H 4350 310 60  0001 L CNN "Part Description"
 F 16 "INFINEON" H 4350 220 60  0001 L CNN "Manufacturer"
-F 17 "BAT165AX" H 4350 130 60  0001 L CNN "Manufacturer Part Number"
+F 17 "BAT165" H 4350 130 60  0001 L CNN "Manufacturer Part Number"
 F 18 "2" H 4350 40  60  0001 L CNN "Pin Count"
 F 19 "SOD323" H 4350 -50 60  0001 L CNN "Case"
@@
 F 15 "Medium Power AF Schottky Diode" H 4450 1010 60  0001 L CNN "Part Description"
 F 16 "INFINEON" H 4450 920 60  0001 L CNN "Manufacturer"
-F 17 "BAT165AX" H 4450 830 60  0001 L CNN "Manufacturer Part Number"
+F 17 "BAT165" H 4450 830 60  0001 L CNN "Manufacturer Part Number"
 F 18 "2" H 4450 740 60  0001 L CNN "Pin Count"
 F 19 "SOD323" H 4450 650 60  0001 L CNN "Case"

Commit message: Swap out 1206 ceramic caps for 0805
Only the schematic change is in this commit
Parts:
- C141: value CC1206_47UF_25V_20%_X5R -> CC0805_22UF_16V_10%_X5R; footprint Marble:CAPC3216X180N -> Marble:CAPC2012X135N; symbol Capacitors_SMD:CC1206_47UF_25V_20%_X5R -> Capacitors_SMD:CC0805_22UF_16V_10%_X5R; Case 1206 -> 0805; CreateDate 11/20/13 00:00:00 -> 10/25/12 00:00:00; Footprint Ref CAPC3216X180N -> CAPC2012X135N; LatestRevisionDate 03/14/17 00:00:00 -> 10/25/12 00:00:00; Manufacturer Part Number CC1206_47UF_25V_20%_X5R -> CC0805_22UF_16V_10%_X5R; Manufacturer1 ComponentHeight 1.8mm -> 1.35mm; Manufacturer1 Example TDK -> Murata; Manufacturer1 Part Number C3216X5R1E476M160AC -> GRM21BR61C226ME44L; Part Number CC1206_47UF_25V_20%_X5R -> CC0805_22UF_16V_10%_X5R; Status None -> Preferred; Tolerance ±20% -> ±10%; Val 47uF -> 22uF; Voltage 25V -> 16V
Changed lines of the file:
@@
 $EndComp
 $Comp
-L Capacitors_SMD:CC1206_47UF_25V_20%_X5R C141
+L Capacitors_SMD:CC0805_22UF_16V_10%_X5R C141
 U 1 1 5DAF13F0
 P 5850 1050
 F 0 "C141" V 5900 1050 50  0000 L CNN
-F 1 "CC1206_47UF_25V_20%_X5R" H 5850 790 60  0001 L CNN
-F 2 "Marble:CAPC3216X180N" H 5850 -20 60  0001 L CNN
+F 1 "CC0805_22UF_16V_10%_X5R" H 5850 790 60  0001 L CNN
+F 2 "Marble:CAPC2012X135N" H 5850 -20 60  0001 L CNN
 F 3 "\\\\cern.ch\\dfs\\Applications\\Altium\\Datasheets\\CC1206_X5R_TDK_C.pdf" H 5850 610 60  0001 L CNN
-F 4 "47uF" V 6100 1050 50  0000 L CNN "Val"
-F 5 "CC1206_47UF_25V_20%_X5R" H 5850 520 60  0001 L CNN "Part Number"
+F 4 "22uF" V 6100 1050 50  0000 L CNN "Val"
+F 5 "CC0805_22UF_16V_10%_X5R" H 5850 520 60  0001 L CNN "Part Number"
 F 6 "Capacitor - non polarized" H 5850 430 60  0001 L CNN "Library Ref"
 F 7 "SchLib\\Capacitors.SchLib" H 5850 340 60  0001 L CNN "Library Path"
@@
 F 11 "2" H 5850 -110 60  0001 L CNN "Pin Count"
 F 12 "PcbLib\\Capacitors SMD.PcbLib" H 5850 -200 60  0001 L CNN "Footprint Path"
-F 13 "CAPC3216X180N" H 5850 -290 60  0001 L CNN "Footprint Ref"
+F 13 "CAPC2012X135N" H 5850 -290 60  0001 L CNN "Footprint Ref"
 F 14 " " H 5850 -380 60  0001 L CNN "PackageDescription"
-F 15 "None" H 5850 -560 60  0001 L CNN "Status"
+F 15 "Preferred" H 5850 -560 60  0001 L CNN "Status"
 F 16 " " H 5850 -650 60  0001 L CNN "Status Comment"
-F 17 "25V" H 5850 -740 60  0001 L CNN "Voltage"
+F 17 "16V" H 5850 -740 60  0001 L CNN "Voltage"
 F 18 "X5R" H 5850 -830 60  0001 L CNN "TC"
-F 19 "±20%" H 5850 -920 60  0001 L CNN "Tolerance"
+F 19 "±10%" H 5850 -920 60  0001 L CNN "Tolerance"
 F 20 "SMD Multilayer Chip Ceramic Capacitor" H 5850 -1010 60  0001 L CNN "Part Description"
 F 21 "GENERIC" H 5850 -1100 60  0001 L CNN "Manufacturer"
-F 22 "CC1206_47UF_25V_20%_X5R" H 5850 -1190 60  0001 L CNN "Manufacturer Part Number"
-F 23 "1206" H 5850 -1280 60  0001 L CNN "Case"
+F 22 "CC0805_22UF_16V_10%_X5R" H 5850 -1190 60  0001 L CNN "Manufacturer Part Number"
+F 23 "0805" H 5850 -1280 60  0001 L CNN "Case"
 F 24 "Yes" H 5850 -1370 60  0001 L CNN "Mounted"
 F 25 "No" H 5850 -1460 60  0001 L CNN "Socket"
@@
 F 29 " " H 5850 -1820 60  0001 L CNN "Sense Comment"
 F 30 " " H 5850 -1910 60  0001 L CNN "ComponentHeight"
-F 31 "TDK" H 5850 -2000 60  0001 L CNN "Manufacturer1 Example"
-F 32 "C3216X5R1E476M160AC" H 5850 -2090 60  0001 L CNN "Manufacturer1 Part Number"
-F 33 "1.8mm" H 5850 -2180 60  0001 L CNN "Manufacturer1 ComponentHeight"
+F 31 "Murata" H 5850 -2000 60  0001 L CNN "Manufacturer1 Example"
+F 32 "GRM21BR61C226ME44L" H 5850 -2090 60  0001 L CNN "Manufacturer1 Part Number"
+F 33 "1.35mm" H 5850 -2180 60  0001 L CNN "Manufacturer1 ComponentHeight"
 F 34 "CERN DEM JLC" H 5850 -2360 60  0001 L CNN "Author"
-F 35 "11/20/13 00:00:00" H 5850 -2450 60  0001 L CNN "CreateDate"
-F 36 "03/14/17 00:00:00" H 5850 -2540 60  0001 L CNN "LatestRevisionDate"
+F 35 "10/25/12 00:00:00" H 5850 -2450 60  0001 L CNN "CreateDate"
+F 36 "10/25/12 00:00:00" H 5850 -2540 60  0001 L CNN "LatestRevisionDate"
 F 37 "Capacitors SMD" H 5850 -2630 60  0001 L CNN "Library Name"
 F 38 "This work is licensed under the Creative Commons CC-BY-SA 4.0 License. To the extent that circuit schematics that use Licensed Material can be considered to be ‘Adapted Material’, then the copyright holder waives article 3.b of the license with respect to these schematics." H 5850 -2720 60  0001 L CNN "License"

Commit message: Convert 7 x CC0805_22UF_16V_10%_X5R to CC0805_22UF_25V_20%_X5R
Yageo CC0805MKX5R8BB226, $0.24300 in 100s at Digi-Key
Parts:
- C141, C151, C153, C155, C157: value CC0805_22UF_16V_10%_X5R -> CC0805_22UF_25V_20%_X5R; symbol Capacitors_SMD:CC0805_22UF_16V_10%_X5R -> Capacitors_SMD:CC0805_22UF_25V_20%_X5R; LatestRevisionDate 10/25/12 00:00:00 -> 05/24/20 00:00:00; Manufacturer Part Number CC0805_22UF_16V_10%_X5R -> CC0805_22UF_25V_20%_X5R; Manufacturer1 Example Murata -> Yageo; Manufacturer1 Part Number GRM21BR61C226ME44L -> CC0805MKX5R8BB226; Part Number CC0805_22UF_16V_10%_X5R -> CC0805_22UF_25V_20%_X5R; Tolerance ±10% -> ±20%; Voltage 16V -> 25V

Commit message: Upgrade voltage rating on 0402 100nF
Convert 16 caps from CC0402_100NF_16V_10%_X5R to CC0402_100NF_25V_10%_X5R
C5 C61 C128 C130 C131 C134 C135 C137 C140 C147 C148 C149 C150 C357 C362 C363
Samsung CL05A104KA5NNNC, $0.00658 in 500s at Digi-Key
Parts:
- C137, C140, C147, C148, C149, C150, C362, C363: value CC0402_100NF_16V_10%_X5R -> CC0402_100NF_25V_10%_X5R; symbol Capacitors_SMD:CC0402_100NF_16V_10%_X5R -> Capacitors_SMD:CC0402_100NF_25V_10%_X5R; Manufacturer Part Number CC0402_100NF_16V_10%_X5R -> CC0402_100NF_25V_10%_X5R; Manufacturer1 Example MURATA -> Samsung; Manufacturer1 Part Number GRM155R61C104KA88D -> CL05A104KA5NNNC; Part Number CC0402_100NF_16V_10%_X5R -> CC0402_100NF_25V_10%_X5R; Voltage 16V -> 25V

Commit message: Upgrade voltage rating on 0603 4.7uF
Convert 26 caps from CC0603_4.7UF_16V_10%_X5R to CC0603_4.7UF_25V_10%_X5R
C57 C103 C105 C127 C129 C139 C142 C143 C144 C159 C161 C162 C167 C168 C173 C195 C331 C343 C344 C347 C348 C349 C360 C361 C364 C373
Samsung CL10A475KA8NQN, $0.11456 in 500s at Digi-Key
Parts:
- C105, C127, C139, C142, C143, C144, C159, C161, C195, C331, C347, C348, C349, C361: value CC0603_4.7UF_16V_10%_X5R -> CC0603_4.7UF_25V_10%_X5R; symbol Capacitors_SMD:CC0603_4.7UF_16V_10%_X5R -> Capacitors_SMD:CC0603_4.7UF_25V_10%_X5R; Manufacturer Part Number CC0603_4.7UF_16V_10%_X5R -> CC0603_4.7UF_25V_10%_X5R; Manufacturer1 Example TAIYO YUDEN -> Samsung; Manufacturer1 Part Number EMK107ABJ475KA-T -> CL10A475KA8NQN; Part Number CC0603_4.7UF_16V_10%_X5R -> CC0603_4.7UF_25V_10%_X5R; Voltage 16V -> 25V

Commit message: Start filling in more Manufacturer fields
Parts:
- U36, U37: Manufacturer (none) -> ON SEMICONDUCTOR
Changed lines of the file:
@@
 F 3 "" H 6650 7700 50  0001 C CNN
 F 4 "NCP186AMX180TAG" H 6650 7700 50  0001 C CNN "Manufacturer Part Number"
+F 5 "ON SEMICONDUCTOR" H 6650 7700 50  0001 C CNN "Manufacturer"
 	1    6650 7700
 	1    0    0    -1
@@
 F 3 "" H 6650 9400 50  0001 C CNN
 F 4 "NCP186AMX120TAG" H 6650 9400 50  0001 C CNN "Manufacturer Part Number"
+F 5 "ON SEMICONDUCTOR" H 6650 9400 50  0001 C CNN "Manufacturer"
 	1    6650 9400
 	1    0    0    -1

Commit message: Fill in Manufacturer for connectors
Parts:
- J9: Manufacturer (none) -> ADAM TECH; Manufacturer Part Number 2057-PH1-04-UA-ND -> PH1-04-UA
Changed lines of the file:
@@
 F 2 "Marble:SAMTEC_MTLW-104-07-L-S-250" H 3900 2700 50  0001 C CNN
 F 3 " " H 3900 2700 50  0001 C CNN
-F 4 "2057-PH1-04-UA-ND" H 3900 2700 50  0001 C CNN "Manufacturer Part Number"
+F 4 "PH1-04-UA" H 3900 2700 50  0001 C CNN "Manufacturer Part Number"
+F 5 "ADAM TECH" H 3900 2700 50  0001 C CNN "Manufacturer"
 	1    3900 2700
 	1    0    0    -1

Commit message: Part substitutions
Mercury VM53S3-25.000-2.5/-30+75 (Y2) => Taiten TXEAADSANF-25.000000 (Y1)
IQD LFVCXO026156 => Kyocera KV7050B20.0000C3GD00
Kingbright KPH-1608CGCK => Wurth 150060VS75000
Should make it easier to source parts in the USA in 2020
Also remove un-helpful (DC-10A) from Cliff FC68148;
Manufacturer part numbers now no longer have spaces; can't say the same about Manufacturer
Parts:
- LD10, LD4, LD5, LD6, LD7, LD8, LD9: Manufacturer KINGBRIGHT -> WURTH; Manufacturer Part Number KPH-1608CGCK -> 150060VS75000
Changed lines of the file:
@@
 F 14 " " H 1450 4900 60  0001 L CNN "Status"
 F 15 "SMD Green LED, Case 1.6mmX0.8mm(0603), 0.65mm Thickness" H 1450 4810 60  0001 L CNN "Part Description"
-F 16 "KINGBRIGHT" H 1450 4720 60  0001 L CNN "Manufacturer"
-F 17 "KPH-1608CGCK" H 1450 4630 60  0001 L CNN "Manufacturer Part Number"
+F 16 "WURTH" H 1450 4720 60  0001 L CNN "Manufacturer"
+F 17 "150060VS75000" H 1450 4630 60  0001 L CNN "Manufacturer Part Number"
 F 18 "2" H 1450 4540 60  0001 L CNN "Pin Count"
 F 19 " " H 1450 4450 60  0001 L CNN "Case"
@@
 F 14 " " H 2500 4900 60  0001 L CNN "Status"
 F 15 "SMD Green LED, Case 1.6mmX0.8mm(0603), 0.65mm Thickness" H 2500 4810 60  0001 L CNN "Part Description"
-F 16 "KINGBRIGHT" H 2500 4720 60  0001 L CNN "Manufacturer"
-F 17 "KPH-1608CGCK" H 2500 4630 60  0001 L CNN "Manufacturer Part Number"
+F 16 "WURTH" H 2500 4720 60  0001 L CNN "Manufacturer"
+F 17 "150060VS75000" H 2500 4630 60  0001 L CNN "Manufacturer Part Number"
 F 18 "2" H 2500 4540 60  0001 L CNN "Pin Count"
 F 19 " " H 2500 4450 60  0001 L CNN "Case"
@@
 F 14 " " H 3650 4900 60  0001 L CNN "Status"
 F 15 "SMD Green LED, Case 1.6mmX0.8mm(0603), 0.65mm Thickness" H 3650 4810 60  0001 L CNN "Part Description"
-F 16 "KINGBRIGHT" H 3650 4720 60  0001 L CNN "Manufacturer"
-F 17 "KPH-1608CGCK" H 3650 4630 60  0001 L CNN "Manufacturer Part Number"
+F 16 "WURTH" H 3650 4720 60  0001 L CNN "Manufacturer"
+F 17 "150060VS75000" H 3650 4630 60  0001 L CNN "Manufacturer Part Number"
 F 18 "2" H 3650 4540 60  0001 L CNN "Pin Count"
 F 19 " " H 3650 4450 60  0001 L CNN "Case"
@@
 F 14 " " H 4700 4900 60  0001 L CNN "Status"
 F 15 "SMD Green LED, Case 1.6mmX0.8mm(0603), 0.65mm Thickness" H 4700 4810 60  0001 L CNN "Part Description"
-F 16 "KINGBRIGHT" H 4700 4720 60  0001 L CNN "Manufacturer"
-F 17 "KPH-1608CGCK" H 4700 4630 60  0001 L CNN "Manufacturer Part Number"
+F 16 "WURTH" H 4700 4720 60  0001 L CNN "Manufacturer"
+F 17 "150060VS75000" H 4700 4630 60  0001 L CNN "Manufacturer Part Number"
 F 18 "2" H 4700 4540 60  0001 L CNN "Pin Count"
 F 19 " " H 4700 4450 60  0001 L CNN "Case"
@@
 F 14 " " H 5250 4900 60  0001 L CNN "Status"
 F 15 "SMD Green LED, Case 1.6mmX0.8mm(0603), 0.65mm Thickness" H 5250 4810 60  0001 L CNN "Part Description"
-F 16 "KINGBRIGHT" H 5250 4720 60  0001 L CNN "Manufacturer"
-F 17 "KPH-1608CGCK" H 5250 4630 60  0001 L CNN "Manufacturer Part Number"
+F 16 "WURTH" H 5250 4720 60  0001 L CNN "Manufacturer"
+F 17 "150060VS75000" H 5250 4630 60  0001 L CNN "Manufacturer Part Number"
 F 18 "2" H 5250 4540 60  0001 L CNN "Pin Count"
 F 19 " " H 5250 4450 60  0001 L CNN "Case"
@@
 F 14 " " H 1400 6500 60  0001 L CNN "Status"
 F 15 "SMD Green LED, Case 1.6mmX0.8mm(0603), 0.65mm Thickness" H 1400 6410 60  0001 L CNN "Part Description"
-F 16 "KINGBRIGHT" H 1400 6320 60  0001 L CNN "Manufacturer"
-F 17 "KPH-1608CGCK" H 1400 6230 60  0001 L CNN "Manufacturer Part Number"
+F 16 "WURTH" H 1400 6320 60  0001 L CNN "Manufacturer"
+F 17 "150060VS75000" H 1400 6230 60  0001 L CNN "Manufacturer Part Number"
 F 18 "2" H 1400 6140 60  0001 L CNN "Pin Count"
 F 19 " " H 1400 6050 60  0001 L CNN "Case"
@@
 F 14 " " H 2050 6500 60  0001 L CNN "Status"
 F 15 "SMD Green LED, Case 1.6mmX0.8mm(0603), 0.65mm Thickness" H 2050 6410 60  0001 L CNN "Part Description"
-F 16 "KINGBRIGHT" H 2050 6320 60  0001 L CNN "Manufacturer"
-F 17 "KPH-1608CGCK" H 2050 6230 60  0001 L CNN "Manufacturer Part Number"
+F 16 "WURTH" H 2050 6320 60  0001 L CNN "Manufacturer"
+F 17 "150060VS75000" H 2050 6230 60  0001 L CNN "Manufacturer Part Number"
 F 18 "2" H 2050 6140 60  0001 L CNN "Pin Count"
 F 19 " " H 2050 6050 60  0001 L CNN "Case"
