File: SDRAM.sch (KiCad schematic (older format))
At the start: 58 parts, among them U3 MT41K512M16HA-125_E, U31 TPS51200DRC

Commit message: Rename library AMC_FMC_Carrier-PcbDoc-rescue as marble_misc
Parts:
- U3: symbol AMC_FMC_Carrier-PcbDoc-rescue:MT41K512M16HA-125_E-Logic -> marble_misc:MT41K512M16HA-125_E-Logic
- U31: symbol AMC_FMC_Carrier-PcbDoc-rescue:TPS51200DRC-Regulator_Linear-AMC_FMC_Carrier-PcbDoc-rescue -> marble_misc:TPS51200DRC-Regulator_Linear-AMC_FMC_Carrier-PcbDoc-rescue
Changed lines of the file:
@@
 Connection ~ 3650 2850
 $Comp
-L AMC_FMC_Carrier-PcbDoc-rescue:MT41K512M16HA-125_E-Logic U3
+L marble_misc:MT41K512M16HA-125_E-Logic U3
 U 1 1 5C4F8488
 P 5000 950
@@
 	2950 3250 4800 3250
 $Comp
-L AMC_FMC_Carrier-PcbDoc-rescue:VTT_DDR3-powerMG-AMC_FMC_Carrier-PcbDoc-rescue #PWR0225
+L marble_misc:VTT_DDR3-powerMG-AMC_FMC_Carrier-PcbDoc-rescue #PWR0225
 U 1 1 5D9E969E
 P 3300 2750
@@
 $EndComp
 $Comp
-L AMC_FMC_Carrier-PcbDoc-rescue:VTT_DDR3-powerMG-AMC_FMC_Carrier-PcbDoc-rescue #PWR0224
+L marble_misc:VTT_DDR3-powerMG-AMC_FMC_Carrier-PcbDoc-rescue #PWR0224
 U 1 1 5DA46618
 P 2550 1050
@@
 Connection ~ 2550 1050
 $Comp
-L AMC_FMC_Carrier-PcbDoc-rescue:VTT_DDR3-powerMG-AMC_FMC_Carrier-PcbDoc-rescue #PWR0457
+L marble_misc:VTT_DDR3-powerMG-AMC_FMC_Carrier-PcbDoc-rescue #PWR0457
 U 1 1 5DA7582E
 P 10800 5200
@@
 	10400 5200 10800 5200
 $Comp
-L AMC_FMC_Carrier-PcbDoc-rescue:TPS51200DRC-Regulator_Linear-AMC_FMC_Carrier-PcbDoc-rescue U31
+L marble_misc:TPS51200DRC-Regulator_Linear-AMC_FMC_Carrier-PcbDoc-rescue U31
 U 1 1 5BDAE091
 P 8150 5400
@@
 $EndComp
 $Comp
-L AMC_FMC_Carrier-PcbDoc-rescue:VTT_DDR3-powerMG-AMC_FMC_Carrier-PcbDoc-rescue #PWR0653
+L marble_misc:VTT_DDR3-powerMG-AMC_FMC_Carrier-PcbDoc-rescue #PWR0653
 U 1 1 5CDF4563
 P 950 7250

Commit message: Strip extraneous AMC_FMC_Carrier-PcbDoc-rescue and powerMG from symbol names
Parts:
- U31: symbol marble_misc:TPS51200DRC-Regulator_Linear-AMC_FMC_Carrier-PcbDoc-rescue -> marble_misc:TPS51200DRC-Regulator_Linear
Changed lines of the file:
@@
 	2950 3250 4800 3250
 $Comp
-L marble_misc:VTT_DDR3-powerMG-AMC_FMC_Carrier-PcbDoc-rescue #PWR0225
+L marble_misc:VTT_DDR3 #PWR0225
 U 1 1 5D9E969E
 P 3300 2750
@@
 $EndComp
 $Comp
-L marble_misc:VTT_DDR3-powerMG-AMC_FMC_Carrier-PcbDoc-rescue #PWR0224
+L marble_misc:VTT_DDR3 #PWR0224
 U 1 1 5DA46618
 P 2550 1050
@@
 Connection ~ 2550 1050
 $Comp
-L marble_misc:VTT_DDR3-powerMG-AMC_FMC_Carrier-PcbDoc-rescue #PWR0457
+L marble_misc:VTT_DDR3 #PWR0457
 U 1 1 5DA7582E
 P 10800 5200
@@
 	10400 5200 10800 5200
 $Comp
-L marble_misc:TPS51200DRC-Regulator_Linear-AMC_FMC_Carrier-PcbDoc-rescue U31
+L marble_misc:TPS51200DRC-Regulator_Linear U31
 U 1 1 5BDAE091
 P 8150 5400
@@
 $EndComp
 $Comp
-L marble_misc:VTT_DDR3-powerMG-AMC_FMC_Carrier-PcbDoc-rescue #PWR0653
+L marble_misc:VTT_DDR3 #PWR0653
 U 1 1 5CDF4563
 P 950 7250

Commit message: Symbols lib. and schematic: update footprint fields
sync with layout is now possible without errors
Parts:
- U31: footprint ICs_And_Semiconductors_SMD:TEXAS_DRC (S-PVSON-N10) -> Marble:TEXAS_DRC(S-PVSON-N10)
Changed lines of the file:
@@
 F 0 "U31" H 8150 6078 50  0000 C CNN
 F 1 "TPS51200DRC" H 8150 5987 50  0000 C CNN
-F 2 "ICs_And_Semiconductors_SMD:TEXAS_DRC (S-PVSON-N10)" H 8150 6250 50  0001 C CNN
+F 2 "Marble:TEXAS_DRC(S-PVSON-N10)" H 8150 6250 50  0001 C CNN
 F 3 "http://www.ti.com/lit/ds/symlink/tps51200.pdf" H 8150 6250 50  0001 C CNN
 F 4 "TPS51200DRC" H 8150 5400 50  0001 C CNN "Manufacturer Part Number"

Commit message: Add four more testpoints to power nets
Parts:
- added TP9: TestPoint, Marble:TestPoint_Pad_D1.0mm, symbol Connector_Generic:TestPoint
Connections:
- wire segments 241 -> 243
Changed lines of the file:
@@
 $EndComp
 Wire Wire Line
-	9050 5200 10400 5200
+	9050 5200 10300 5200
 Connection ~ 9050 5200
 Connection ~ 10800 5200
@@
 Text Notes 1300 3800 0    50   ~ 0
 No need to control CS pin,
+$Comp
+L Connector_Generic:TestPoint TP9
+U 1 1 5ECF58E8
+P 10300 5050
+F 0 "TP9" H 10358 5168 50  0000 L CNN
+F 1 "TestPoint" H 10358 5077 50  0000 L CNN
+F 2 "Marble:TestPoint_Pad_D1.0mm" H 10500 5050 50  0001 C CNN
+F 3 "" H 10500 5050 50  0001 C CNN
+	1    10300 5050
+	1    0    0    -1
+$EndComp
+Wire Wire Line
+	10300 5050 10300 5200
 Wire Bus Line
 	10150 700  10150 1000
@@
 Wire Bus Line
 	10150 1150 10150 2750
+Connection ~ 10300 5200
+Wire Wire Line
+	10300 5200 10400 5200
 $EndSCHEMATC

Commit message: Convert all footprints to use Marble nickname
Includes both .sch and .lib files
Includes both bare footprint names and those with CERN-like nicknames
Parts:
- C14, C15, C16, C17, C18, C19, C20, C21, C23, C25, C365, C366, C367, C368, C369, C370, C371, C372: footprint CAPC0603X33N -> Marble:CAPC0603X33N
- C22, C26, C27: footprint CAPC1709X100N -> Marble:CAPC1709X100N
- C24: footprint CAPC1005X55N -> Marble:CAPC1005X55N
- C364, C373: footprint CAPC1709X95N -> Marble:CAPC1709X95N
- R1, R10, R106, R11, R12, R13, R14, R15, R16, R17, R18, R19, R2, R20, R21, R22, R23, R24, R25, R26, R27, R28, R29, R3, R30, R31, R4, R5, R6, R7, R8, R9: footprint RESC1005X40N -> Marble:RESC1005X40N
- U3: footprint BGA96C80P9X16_900X1400X120 -> Marble:BGA96C80P9X16_900X1400X120

Commit message: Get rid of "~" attribute in instances
This makes instances line up better with our library
Use a very short python program to rename "~" to "Val" and remove the old "Val".
Required a little pre-patch to correctly handle R297 R298 R299 R300 R162 R274 R197 R198, which had no "~" field.
No net changes to "Val" field contents.
Parts:
- C14, C15, C16, C17, C18, C19, C20, C21, C23, C25, C365, C366, C367, C368, C369, C370, C371, C372: ~ 100nF -> (none)
- C22, C26, C27: ~ 22uF -> (none)
- C24: ~ 1uF -> (none)
- C364, C373: ~ 4.7uF -> (none)
- R1, R2, R3: ~ 51 -> (none)
- R10, R106, R11, R12, R13, R14, R15, R16, R17, R18, R19, R20, R21, R22, R23, R27, R4, R5, R6, R7, R8, R9: ~ 40R2 -> (none)
- R24, R25, R26: ~ 5k1 -> (none)
- R28: ~ 240 -> (none)
- R29, R30, R31: ~ 10k -> (none)
