File: SDRAM.sch (KiCad schematic (older format))
At the start: 59 parts, among them U3 MT41K512M16HA-125_E, U31 TPS51200DRC

Commit message: Upgrade voltage rating on 0603 4.7uF
Convert 26 caps from CC0603_4.7UF_16V_10%_X5R to CC0603_4.7UF_25V_10%_X5R
C57 C103 C105 C127 C129 C139 C142 C143 C144 C159 C161 C162 C167 C168 C173 C195 C331 C343 C344 C347 C348 C349 C360 C361 C364 C373
Samsung CL10A475KA8NQN, $0.11456 in 500s at Digi-Key
Parts:
- C364, C373: value CC0603_4.7UF_16V_10%_X5R -> CC0603_4.7UF_25V_10%_X5R; symbol Capacitors_SMD:CC0603_4.7UF_16V_10%_X5R -> Capacitors_SMD:CC0603_4.7UF_25V_10%_X5R; Manufacturer Part Number CC0603_4.7UF_16V_10%_X5R -> CC0603_4.7UF_25V_10%_X5R; Manufacturer1 Example TAIYO YUDEN -> Samsung; Manufacturer1 Part Number EMK107ABJ475KA-T -> CL10A475KA8NQN; Part Number CC0603_4.7UF_16V_10%_X5R -> CC0603_4.7UF_25V_10%_X5R; Voltage 16V -> 25V
Changed lines of the file:
@@
 	950  5850 950  5900
 $Comp
-L Capacitors_SMD:CC0603_4.7UF_16V_10%_X5R C?
+L Capacitors_SMD:CC0603_4.7UF_25V_10%_X5R C?
 U 1 1 5D097270
 P 950 5550
@@
 AR Path="/5BD32060/5D097270" Ref="C364"  Part="1"
 F 0 "C364" V 1000 5550 50  0000 L CNN
-F 1 "CC0603_4.7UF_16V_10%_X5R" H 950 5290 60  0001 L CNN
+F 1 "CC0603_4.7UF_25V_10%_X5R" H 950 5290 60  0001 L CNN
 F 2 "Marble:CAPC1709X95N" H 950 4480 60  0001 L CNN
 F 3 "\\\\cern.ch\\dfs\\Applications\\Altium\\Datasheets\\CC0603_X7R_TAIYO-YUDEN_HIGH-VALUE.pdf" H 950 5110 60  0001 L CNN
 F 4 "4.7uF" V 1200 5550 50  0000 L CNN "Val"
-F 5 "CC0603_4.7UF_16V_10%_X5R" H 950 5020 60  0001 L CNN "Part Number"
+F 5 "CC0603_4.7UF_25V_10%_X5R" H 950 5020 60  0001 L CNN "Part Number"
 F 6 "Capacitor - non polarized" H 950 4930 60  0001 L CNN "Library Ref"
 F 7 "SchLib\\Capacitors.SchLib" H 950 4840 60  0001 L CNN "Library Path"
@@
 F 15 "None" H 950 3940 60  0001 L CNN "Status"
 F 16 " " H 950 3850 60  0001 L CNN "Status Comment"
-F 17 "16V" H 950 3760 60  0001 L CNN "Voltage"
+F 17 "25V" H 950 3760 60  0001 L CNN "Voltage"
 F 18 "X5R" H 950 3670 60  0001 L CNN "TC"
 F 19 "±10%" H 950 3580 60  0001 L CNN "Tolerance"
 F 20 "SMD Multilayer Chip Ceramic Capacitor" H 950 3490 60  0001 L CNN "Part Description"
 F 21 "GENERIC" H 950 3400 60  0001 L CNN "Manufacturer"
-F 22 "CC0603_4.7UF_16V_10%_X5R" H 950 3310 60  0001 L CNN "Manufacturer Part Number"
+F 22 "CC0603_4.7UF_25V_10%_X5R" H 950 3310 60  0001 L CNN "Manufacturer Part Number"
 F 23 "0603" H 950 3220 60  0001 L CNN "Case"
 F 24 "Yes" H 950 3130 60  0001 L CNN "Mounted"
@@
 F 29 " " H 950 2680 60  0001 L CNN "Sense Comment"
 F 30 " " H 950 2590 60  0001 L CNN "ComponentHeight"
-F 31 "TAIYO YUDEN" H 950 2500 60  0001 L CNN "Manufacturer1 Example"
-F 32 "EMK107ABJ475KA-T" H 950 2410 60  0001 L CNN "Manufacturer1 Part Number"
+F 31 "Samsung" H 950 2500 60  0001 L CNN "Manufacturer1 Example"
+F 32 "CL10A475KA8NQN" H 950 2410 60  0001 L CNN "Manufacturer1 Part Number"
 F 33 "0.95mm" H 950 2320 60  0001 L CNN "Manufacturer1 ComponentHeight"
 F 34 "CERN DEM JLC" H 950 2140 60  0001 L CNN "Author"
@@
 	2300 5850 1850 5850
 $Comp
-L Capacitors_SMD:CC0603_4.7UF_16V_10%_X5R C?
+L Capacitors_SMD:CC0603_4.7UF_25V_10%_X5R C?
 U 1 1 5DA50D23
 P 1400 5550
@@
 AR Path="/5BD32060/5DA50D23" Ref="C373"  Part="1"
 F 0 "C373" V 1450 5550 50  0000 L CNN
-F 1 "CC0603_4.7UF_16V_10%_X5R" H 1400 5290 60  0001 L CNN
+F 1 "CC0603_4.7UF_25V_10%_X5R" H 1400 5290 60  0001 L CNN
 F 2 "Marble:CAPC1709X95N" H 1400 4480 60  0001 L CNN
 F 3 "\\\\cern.ch\\dfs\\Applications\\Altium\\Datasheets\\CC0603_X7R_TAIYO-YUDEN_HIGH-VALUE.pdf" H 1400 5110 60  0001 L CNN
 F 4 "4.7uF" V 1650 5550 50  0000 L CNN "Val"
-F 5 "CC0603_4.7UF_16V_10%_X5R" H 1400 5020 60  0001 L CNN "Part Number"
+F 5 "CC0603_4.7UF_25V_10%_X5R" H 1400 5020 60  0001 L CNN "Part Number"
 F 6 "Capacitor - non polarized" H 1400 4930 60  0001 L CNN "Library Ref"
 F 7 "SchLib\\Capacitors.SchLib" H 1400 4840 60  0001 L CNN "Library Path"
@@
 F 15 "None" H 1400 3940 60  0001 L CNN "Status"
 F 16 " " H 1400 3850 60  0001 L CNN "Status Comment"
-F 17 "16V" H 1400 3760 60  0001 L CNN "Voltage"
+F 17 "25V" H 1400 3760 60  0001 L CNN "Voltage"
 F 18 "X5R" H 1400 3670 60  0001 L CNN "TC"
 F 19 "±10%" H 1400 3580 60  0001 L CNN "Tolerance"
 F 20 "SMD Multilayer Chip Ceramic Capacitor" H 1400 3490 60  0001 L CNN "Part Description"
 F 21 "GENERIC" H 1400 3400 60  0001 L CNN "Manufacturer"
-F 22 "CC0603_4.7UF_16V_10%_X5R" H 1400 3310 60  0001 L CNN "Manufacturer Part Number"
+F 22 "CC0603_4.7UF_25V_10%_X5R" H 1400 3310 60  0001 L CNN "Manufacturer Part Number"
 F 23 "0603" H 1400 3220 60  0001 L CNN "Case"
 F 24 "Yes" H 1400 3130 60  0001 L CNN "Mounted"
@@
 F 29 " " H 1400 2680 60  0001 L CNN "Sense Comment"
 F 30 " " H 1400 2590 60  0001 L CNN "ComponentHeight"
-F 31 "TAIYO YUDEN" H 1400 2500 60  0001 L CNN "Manufacturer1 Example"
-F 32 "EMK107ABJ475KA-T" H 1400 2410 60  0001 L CNN "Manufacturer1 Part Number"
+F 31 "Samsung" H 1400 2500 60  0001 L CNN "Manufacturer1 Example"
+F 32 "CL10A475KA8NQN" H 1400 2410 60  0001 L CNN "Manufacturer1 Part Number"
 F 33 "0.95mm" H 1400 2320 60  0001 L CNN "Manufacturer1 ComponentHeight"
 F 34 "CERN DEM JLC" H 1400 2140 60  0001 L CNN "Author"

Commit message: Start filling in more Manufacturer fields
Parts:
- U31: Manufacturer (none) -> TEXAS INSTRUMENTS
Changed lines of the file:
@@
 F 3 "http://www.ti.com/lit/ds/symlink/tps51200.pdf" H 8150 6250 50  0001 C CNN
 F 4 "TPS51200DRC" H 8150 5400 50  0001 C CNN "Manufacturer Part Number"
+F 5 "TEXAS INSTRUMENTS" H 8150 5400 50  0001 C CNN "Manufacturer"
 	1    8150 5400
 	1    0    0    -1

Commit message: A little more clarity on Manufacturer and Part Number
Adjustments to DDR3 memory, a resistor, and a push-button
Parts:
- U3: Manufacturer MICRON TECHNOLOGY -> ALLIANCE; Manufacturer Part Number MT41K512M16HA-125:E (AS4C512M16D3L-12BCN) -> AS4C512M16D3L-12BCN
Changed lines of the file:
@@
 F 12 " " H 5000 -6120 60  0001 L CNN "Status"
 F 13 "+1.35V, 8Gb (64 Meg x 16 x 8 banks) DDR3L SDRAM" H 5000 -6210 60  0001 L CNN "Part Description"
-F 14 "MICRON TECHNOLOGY" H 5000 -6300 60  0001 L CNN "Manufacturer"
-F 15 "MT41K512M16HA-125:E (AS4C512M16D3L-12BCN)" H 5000 -6390 60  0001 L CNN "Manufacturer Part Number"
+F 14 "ALLIANCE" H 5000 -6300 60  0001 L CNN "Manufacturer"
+F 15 "AS4C512M16D3L-12BCN" H 5000 -6390 60  0001 L CNN "Manufacturer Part Number"
 F 16 "96" H 5000 -6480 60  0001 L CNN "Pin Count"
 F 17 "BGA96" H 5000 -6570 60  0001 L CNN "Case"
