File: AMC_connector.sch (KiCad schematic (older format))
At the start: 2 parts, among them P3 CMP-0001-00058-2

Commit message: SCH: PWR_FLAG cosmetics, update annotation
Changed lines of the file:
@@
 	1    0    0    -1
 $EndComp
-Wire Wire Line
-	1750 6493 1750 6500
-Connection ~ 1750 6500
-Wire Wire Line
-	1750 6500 1750 7700
 $Comp
 L marble_misc:+12V_AMC #PWR031
@@
 Wire Wire Line
 	9200 3250 10000 3250
+Wire Wire Line
+	1750 6500 1750 6550
 Wire Bus Line
 	10026 4346 10026 4546
+$Comp
+L power:PWR_FLAG #FLG0110
+U 1 1 5EDB0932
+P 1750 6550
+F 0 "#FLG0110" H 1750 6625 50  0001 C CNN
+F 1 "PWR_FLAG" V 1750 6677 50  0000 L CNN
+F 2 "" H 1750 6550 50  0001 C CNN
+F 3 "" H 1750 6550 50  0001 C CNN
+	1    1750 6550
+	0    -1   -1   0
+$EndComp
+Connection ~ 1750 6550
+Wire Wire Line
+	1750 6550 1750 7700
 $EndSCHEMATC

Commit message: Convert all footprints to use Marble nickname
Includes both .sch and .lib files
Includes both bare footprint names and those with CERN-like nicknames
Parts:
- D1: footprint DIOM5127X229N -> Marble:DIOM5127X229N
Changed lines of the file:
@@
 F 0 "D1" V 12196 5310 50  0000 R CNN
 F 1 "SS16" V 12105 5310 50  0000 R CNN
-F 2 "DIOM5127X229N" H 12000 4260 60  0001 L CNN
+F 2 "Marble:DIOM5127X229N" H 12000 4260 60  0001 L CNN
 F 3 "\\\\cern.ch\\dfs\\Applications\\Altium\\Datasheets\\SS16.pdf" H 12000 4980 60  0001 L CNN
 F 4 "SS16" H 12000 4890 60  0001 L CNN "Part Number"

Commit message: Convert "~" and "~~" in .sch and .lib files to " "
Parts:
- D1: ComponentLink1Description ~~ -> (none); ComponentLink1URL ~~ -> (none); ComponentLink2Description ~~ -> (none); ComponentLink2URL ~~ -> (none); Sense Comment ~~ -> (none); Status ~~ -> (none); Status Comment ~~ -> (none)
Changed lines of the file:
@@
 F 12 "60V" H 12000 4080 60  0001 L CNN "Voltage"
 F 13 "1A" H 12000 3990 60  0001 L CNN "Power"
-F 14 "~~" H 12000 3900 60  0001 L CNN "Status"
+F 14 " " H 12000 3900 60  0001 L CNN "Status"
 F 15 "Surface Mount Schottky Barrier Rectifier" H 12000 3810 60  0001 L CNN "Part Description"
 F 16 "VISHAY GENERAL SEMICONDUCTOR" H 12000 3720 60  0001 L CNN "Manufacturer"
@@
 F 23 "No" H 12000 3090 60  0001 L CNN "PressFit"
 F 24 "No" H 12000 3000 60  0001 L CNN "Sense"
-F 25 "~~" H 12000 2910 60  0001 L CNN "Sense Comment"
+F 25 " " H 12000 2910 60  0001 L CNN "Sense Comment"
 F 26 "No" H 12000 2820 60  0001 L CNN "Bonding"
-F 27 "~~" H 12000 2730 60  0001 L CNN "Status Comment"
+F 27 " " H 12000 2730 60  0001 L CNN "Status Comment"
 F 28 "2.29mm" H 12000 2640 60  0001 L CNN "ComponentHeight"
 F 29 "PcbLib\\ICs And Semiconductors SMD.PcbLib" H 12000 2550 60  0001 L CNN "Footprint Path"
 F 30 "DIOM5127X229N" H 12000 2460 60  0001 L CNN "Footprint Ref"
 F 31 "\\\\cern.ch\\dfs\\Applications\\Altium\\Datasheets\\SS16.pdf" H 12000 2370 60  0001 L CNN "HelpURL"
-F 32 "~~" H 12000 2280 60  0001 L CNN "ComponentLink1URL"
-F 33 "~~" H 12000 2190 60  0001 L CNN "ComponentLink1Description"
-F 34 "~~" H 12000 2100 60  0001 L CNN "ComponentLink2URL"
-F 35 "~~" H 12000 2010 60  0001 L CNN "ComponentLink2Description"
+F 32 " " H 12000 2280 60  0001 L CNN "ComponentLink1URL"
+F 33 " " H 12000 2190 60  0001 L CNN "ComponentLink1Description"
+F 34 " " H 12000 2100 60  0001 L CNN "ComponentLink2URL"
+F 35 " " H 12000 2010 60  0001 L CNN "ComponentLink2Description"
 F 36 "CERN DEM JLC" H 12000 1920 60  0001 L CNN "Author"
 F 37 "07/15/08 00:00:00" H 12000 1830 60  0001 L CNN "CreateDate"

Commit message: Trash HelpURL ComponentLink1URL ComponentLink2URL attributes
Removes 1056 useless and library-mismatched attributes
Parts:
- D1: ComponentLink1URL (none) -> (none); ComponentLink2URL (none) -> (none); HelpURL \\\\cern.ch\\dfs\\Applications\\Altium\\Datasheets\\SS16.pdf -> (none)
Changed lines of the file:
@@
 F 29 "PcbLib\\ICs And Semiconductors SMD.PcbLib" H 12000 2550 60  0001 L CNN "Footprint Path"
 F 30 "DIOM5127X229N" H 12000 2460 60  0001 L CNN "Footprint Ref"
-F 31 "\\\\cern.ch\\dfs\\Applications\\Altium\\Datasheets\\SS16.pdf" H 12000 2370 60  0001 L CNN "HelpURL"
-F 32 " " H 12000 2280 60  0001 L CNN "ComponentLink1URL"
 F 33 " " H 12000 2190 60  0001 L CNN "ComponentLink1Description"
-F 34 " " H 12000 2100 60  0001 L CNN "ComponentLink2URL"
 F 35 " " H 12000 2010 60  0001 L CNN "ComponentLink2Description"
 F 36 "CERN DEM JLC" H 12000 1920 60  0001 L CNN "Author"
