File: FPGA_PWR&MISC.sch (KiCad schematic (older format))
At the start: 102 parts, among them Q19 BSS138LT1G, U1 XC7A100T-2FGG484C

Commit message: Convert "~" and "~~" in .sch and .lib files to " "
Parts:
- C1, C2, C216, C217, C218, C219, C220, C221, C222, C223, C224, C225, C226, C227, C228, C229, C230, C231, C232, C233, C234, C235, C236, C237, C238, C239, C240, C241, C242, C243, C244, C245, C246, C247, C248, C249, C250, C251, C252, C253, C254, C255, C256, C257, C258, C259, C260, C261, C262, C263, C264, C265, C266, C267, C268, C269, C270, C271, C272, C273, C274, C275, C276, C277, C278, C279, C280, C281, C282, C283, C284, C285, C286, C287, C3, C332, C333, C334, C335, C336, C337, C338, C339, C4: ComponentHeight ~~ -> (none); PackageDescription ~~ -> (none); PressFit ~~ -> (none); Sense Comment ~~ -> (none); Status Comment ~~ -> (none)
- L27, L28: PackageDescription ~~ -> (none); Sense Comment ~~ -> (none); Status Comment ~~ -> (none)
- LD3: Case ~~ -> (none); Comment ~~ -> (none); ComponentLink1Description ~~ -> (none); ComponentLink1URL ~~ -> (none); ComponentLink2Description ~~ -> (none); ComponentLink2URL ~~ -> (none); Device ~~ -> (none); Sense Comment ~~ -> (none); Status ~~ -> (none); Status Comment ~~ -> (none)
- PB1: Case ~~ -> (none); Comment ~~ -> (none); ComponentLink1Description ~~ -> (none); ComponentLink1URL ~~ -> (none); ComponentLink2Description ~~ -> (none); ComponentLink2URL ~~ -> (none); Manufacturer1 ComponentHeight ~~ -> (none); Manufacturer1 Example ~~ -> (none); Manufacturer1 Part Number ~~ -> (none); SCEM ~~ -> (none); Sense Comment ~~ -> (none); Status Comment ~~ -> (none)
- Q19: ComponentLink1URL ~~ -> (none); ComponentLink2URL ~~ -> (none)
- R159, R286, R287, R288: ComponentHeight ~~ -> (none); PackageDescription ~~ -> (none); Power ~~ -> (none); Sense Comment ~~ -> (none); Status Comment ~~ -> (none); TC ~~ -> (none); Tolerance ~~ -> (none); Voltage ~~ -> (none)
- R160, R162, R163, R282, R283, R284, R285: ComponentHeight ~~ -> (none); PackageDescription ~~ -> (none); Sense Comment ~~ -> (none); Status Comment ~~ -> (none); Voltage ~~ -> (none)
- R161: ComponentHeight ~~ -> (none); PackageDescription ~~ -> (none); Sense Comment ~~ -> (none); Status Comment ~~ -> (none)

Commit message: Sanitize pin counts in schematics
A lot of them were listed as 2.0000000000000000e+00
Parts:
- C1, C2, C216, C217, C218, C219, C220, C221, C222, C223, C224, C225, C226, C227, C228, C229, C230, C231, C232, C233, C234, C235, C236, C237, C238, C239, C240, C241, C242, C243, C244, C245, C246, C247, C248, C249, C250, C251, C252, C253, C254, C255, C256, C257, C258, C259, C260, C261, C262, C263, C264, C265, C266, C267, C268, C269, C270, C271, C272, C273, C274, C275, C276, C277, C278, C279, C280, C281, C282, C283, C284, C285, C286, C287, C3, C332, C333, C334, C335, C336, C337, C338, C339, C4, L27, L28: Pin Count 2.0000000000000000e+00 -> 2

Commit message: Trash HelpURL ComponentLink1URL ComponentLink2URL attributes
Removes 1056 useless and library-mismatched attributes
Parts:
- C1, C222, C225, C280, C281, C282, C283: HelpURL \\\\cern.ch\\dfs\\Applications\\Altium\\Datasheets\\CC0603_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 -> (none)
- C2, C239, C265, C266: HelpURL \\\\cern.ch\\dfs\\Applications\\Altium\\Datasheets\\CC1210_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 -> (none)
- C216, C217, C218, C219, C220, C221, C223, C224, C226, C227, C228, C229, C230, C231, C232, C234, C236, C238, C244, C245, C246, C247, C248, C249, C250, C251, C256, C257, C258, C259, C260, C261, C262, C263, C264, C267, C269, C271, C273, C275, C277, C279, C3, C332, C333, C334, C335, C336, C337, C338, C339, C4: HelpURL \\\\cern.ch\\dfs\\Applications\\Altium\\Datasheets\\CC0201_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 -> (none)
- C233, C235, C237, C240, C241, C242, C243, C252, C253, C254, C255, C268, C270, C272, C274, C276, C278, C284, C285, C286, C287: HelpURL \\\\cern.ch\\dfs\\Applications\\Altium\\Datasheets\\CC0805_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 -> (none)
- L27, L28: HelpURL \\\\cern.ch\\dfs\\Applications\\Altium\\Datasheets\\IND0603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 -> (none)
- LD3: ComponentLink1URL (none) -> (none); ComponentLink2URL (none) -> (none); HelpURL \\\\cern.ch\\dfs\\Applications\\Altium\\Datasheets\\LED_KIN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 -> (none)
- PB1: ComponentLink1URL (none) -> (none); ComponentLink2URL (none) -> (none); HelpURL \\\\cern.ch\\dfs\\Applications\\Altium\\Datasheets\\PB_TYCO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 -> (none)
- Q19: ComponentLink1URL (none) -> (none); ComponentLink2URL (none) -> (none); HelpURL \\\\cern.ch\\dfs\\Applications\\Altium\\Datasheets\\BSS138L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 -> (none)
- R159, R160, R161, R162, R163, R282, R283, R284, R285, R286, R287, R288: HelpURL \\\\cern.ch\\dfs\\Applications\\Altium\\Datasheets\\R0402_P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 -> (none)

Commit message: Trash "Footprint Library" and "Database Table Name" attributes
Takes 100 attributes out of schematic, 174 out of library
Parts:
- Q19: Database Table Name Transistors -> (none); Footprint Library ICs And Semiconductors SMD -> (none)
Changed lines of the file:
@@
 F 37 "ICs And Semiconductors SMD" H 15150 1560 60  0001 L CNN "Library Name"
 F 38 "This work is licensed under the Creative Commons CC-BY-SA 4.0 License. To the extent that circuit schematics that use Licensed Material can be considered to be ‘Adapted Material’, then the copyright holder waives article 3.b of the license with respect to these schematics." H 15150 1470 60  0001 L CNN "License"
-F 39 "Transistors" H 15150 5200 50  0001 C CNN "Database Table Name"
-F 40 "ICs And Semiconductors SMD" H 15150 5200 50  0001 C CNN "Footprint Library"
 F 41 " " H 15150 5200 50  0001 C CNN "SCEM"
 	1    15150 5200

Commit message: Trash SCEM attribute
Parts:
- PB1, Q19: SCEM (none) -> (none)
Changed lines of the file:
@@
 F 23 "None" H 11350 4400 60  0001 L CNN "Status"
 F 24 " " H 11350 4310 60  0001 L CNN "Status Comment"
-F 25 " " H 11350 4220 60  0001 L CNN "SCEM"
 F 26 "12VDC 50mA SPST Tactile  Push-Button Switch" H 11350 4130 60  0001 L CNN "Part Description"
 F 27 "TYCO ELECTRONICS" H 11350 4040 60  0001 L CNN "Manufacturer"
@@
 F 37 "ICs And Semiconductors SMD" H 15150 1560 60  0001 L CNN "Library Name"
 F 38 "This work is licensed under the Creative Commons CC-BY-SA 4.0 License. To the extent that circuit schematics that use Licensed Material can be considered to be ‘Adapted Material’, then the copyright holder waives article 3.b of the license with respect to these schematics." H 15150 1470 60  0001 L CNN "License"
-F 41 " " H 15150 5200 50  0001 C CNN "SCEM"
 	1    15150 5200
 	1    0    0    -1
