File: SFP4.sch (KiCad schematic (older format))
At the start: 19 parts, among them J8 TYCO_1888247-1

Commit message: Convert "~" and "~~" in .sch and .lib files to " "
Parts:
- C100, C101, C94, C95, C96, C97, C98, C99: ComponentHeight ~~ -> (none); PackageDescription ~~ -> (none); PressFit ~~ -> (none); Sense Comment ~~ -> (none); Status Comment ~~ -> (none)
- J8: ComponentLink1URL ~~ -> (none); ComponentLink2URL ~~ -> (none)
- L7, L8: PackageDescription ~~ -> (none); Sense Comment ~~ -> (none); Status Comment ~~ -> (none)
- R186, R85, R87, R88, R89, R90: ComponentHeight ~~ -> (none); PackageDescription ~~ -> (none); Sense Comment ~~ -> (none); Status Comment ~~ -> (none); Voltage ~~ -> (none)
- R86: ComponentHeight ~~ -> (none); PackageDescription ~~ -> (none); Power ~~ -> (none); Sense Comment ~~ -> (none); Status Comment ~~ -> (none); TC ~~ -> (none); Tolerance ~~ -> (none); Voltage ~~ -> (none)

Commit message: Sanitize pin counts in schematics
A lot of them were listed as 2.0000000000000000e+00
Parts:
- C100, C101, C94, C95, C96, C97, C98, C99, L7, L8: Pin Count 2.0000000000000000e+00 -> 2
Changed lines of the file:
@@
 F 9 "Standard" H 1150 1060 60  0001 L CNN "Component Kind"
 F 10 "Standard" H 1150 970 60  0001 L CNN "Component Type"
-F 11 "2.0000000000000000e+00" H 1150 790 60  0001 L CNN "Pin Count"
+F 11 "2" H 1150 790 60  0001 L CNN "Pin Count"
 F 12 "PcbLib\\Capacitors SMD.PcbLib" H 1150 700 60  0001 L CNN "Footprint Path"
 F 13 "CAPC0603X33N" H 1150 610 60  0001 L CNN "Footprint Ref"
@@
 F 9 "Standard" H 3100 1060 60  0001 L CNN "Component Kind"
 F 10 "Standard" H 3100 970 60  0001 L CNN "Component Type"
-F 11 "2.0000000000000000e+00" H 3100 790 60  0001 L CNN "Pin Count"
+F 11 "2" H 3100 790 60  0001 L CNN "Pin Count"
 F 12 "PcbLib\\Capacitors SMD.PcbLib" H 3100 700 60  0001 L CNN "Footprint Path"
 F 13 "CAPC0603X33N" H 3100 610 60  0001 L CNN "Footprint Ref"
@@
 F 9 "Standard" H 3500 1060 60  0001 L CNN "Component Kind"
 F 10 "Standard" H 3500 970 60  0001 L CNN "Component Type"
-F 11 "2.0000000000000000e+00" H 3500 790 60  0001 L CNN "Pin Count"
+F 11 "2" H 3500 790 60  0001 L CNN "Pin Count"
 F 12 "PcbLib\\Capacitors SMD.PcbLib" H 3500 700 60  0001 L CNN "Footprint Path"
 F 13 "CAPC0603X33N" H 3500 610 60  0001 L CNN "Footprint Ref"
@@
 F 9 "Standard" H 3850 2060 60  0001 L CNN "Component Kind"
 F 10 "Standard" H 3850 1970 60  0001 L CNN "Component Type"
-F 11 "2.0000000000000000e+00" H 3850 1790 60  0001 L CNN "Pin Count"
+F 11 "2" H 3850 1790 60  0001 L CNN "Pin Count"
 F 12 "PcbLib\\Capacitors SMD.PcbLib" H 3850 1700 60  0001 L CNN "Footprint Path"
 F 13 "CAPC0603X33N" H 3850 1610 60  0001 L CNN "Footprint Ref"
@@
 F 10 "Standard" H 1850 1040 60  0001 L CNN "Component Type"
 F 11 " " H 1850 860 60  0001 L CNN "PackageDescription"
-F 12 "2.0000000000000000e+00" H 1850 770 60  0001 L CNN "Pin Count"
+F 12 "2" H 1850 770 60  0001 L CNN "Pin Count"
 F 13 "PcbLib\\Inductors SMD.PcbLib" H 1850 680 60  0001 L CNN "Footprint Path"
 F 14 "INDC1608X65N" H 1850 590 60  0001 L CNN "Footprint Ref"
@@
 F 10 "Standard" H 3100 2040 60  0001 L CNN "Component Type"
 F 11 " " H 3100 1860 60  0001 L CNN "PackageDescription"
-F 12 "2.0000000000000000e+00" H 3100 1770 60  0001 L CNN "Pin Count"
+F 12 "2" H 3100 1770 60  0001 L CNN "Pin Count"
 F 13 "PcbLib\\Inductors SMD.PcbLib" H 3100 1680 60  0001 L CNN "Footprint Path"
 F 14 "INDC1608X65N" H 3100 1590 60  0001 L CNN "Footprint Ref"
@@
 F 9 "Standard" H 1600 1060 60  0001 L CNN "Component Kind"
 F 10 "Standard" H 1600 970 60  0001 L CNN "Component Type"
-F 11 "2.0000000000000000e+00" H 1600 790 60  0001 L CNN "Pin Count"
+F 11 "2" H 1600 790 60  0001 L CNN "Pin Count"
 F 12 "PcbLib\\Capacitors SMD.PcbLib" H 1600 700 60  0001 L CNN "Footprint Path"
 F 13 "CAPC1005X55N" H 1600 610 60  0001 L CNN "Footprint Ref"
@@
 F 9 "Standard" H 2700 1060 60  0001 L CNN "Component Kind"
 F 10 "Standard" H 2700 970 60  0001 L CNN "Component Type"
-F 11 "2.0000000000000000e+00" H 2700 790 60  0001 L CNN "Pin Count"
+F 11 "2" H 2700 790 60  0001 L CNN "Pin Count"
 F 12 "PcbLib\\Capacitors SMD.PcbLib" H 2700 700 60  0001 L CNN "Footprint Path"
 F 13 "CAPC1005X55N" H 2700 610 60  0001 L CNN "Footprint Ref"
@@
 F 9 "Standard" H 2300 1360 60  0001 L CNN "Component Kind"
 F 10 "Standard" H 2300 1270 60  0001 L CNN "Component Type"
-F 11 "2.0000000000000000e+00" H 2300 1090 60  0001 L CNN "Pin Count"
+F 11 "2" H 2300 1090 60  0001 L CNN "Pin Count"
 F 12 "PcbLib\\Capacitors SMD.PcbLib" H 2300 1000 60  0001 L CNN "Footprint Path"
 F 13 "CAPC1608X87N" H 2300 910 60  0001 L CNN "Footprint Ref"
@@
 F 9 "Standard" H 3450 2360 60  0001 L CNN "Component Kind"
 F 10 "Standard" H 3450 2270 60  0001 L CNN "Component Type"
-F 11 "2.0000000000000000e+00" H 3450 2090 60  0001 L CNN "Pin Count"
+F 11 "2" H 3450 2090 60  0001 L CNN "Pin Count"
 F 12 "PcbLib\\Capacitors SMD.PcbLib" H 3450 2000 60  0001 L CNN "Footprint Path"
 F 13 "CAPC1608X87N" H 3450 1910 60  0001 L CNN "Footprint Ref"

Commit message: Trash HelpURL ComponentLink1URL ComponentLink2URL attributes
Removes 1056 useless and library-mismatched attributes
Parts:
- C100, C101, C94, C98: HelpURL \\\\cern.ch\\dfs\\Applications\\Altium\\Datasheets\\CC0201_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 -> (none)
- C95, C97: HelpURL \\\\cern.ch\\dfs\\Applications\\Altium\\Datasheets\\CC0402_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 -> (none)
- C96, C99: HelpURL \\\\cern.ch\\dfs\\Applications\\Altium\\Datasheets\\CC0603_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 -> (none)
- J8: ComponentLink1URL (none) -> (none); ComponentLink2URL (none) -> (none); HelpURL \\\\cern.ch\\dfs\\Applications\\Altium\\Datasheets\\TYCO_18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 -> (none)
- L7, L8: HelpURL \\\\cern.ch\\dfs\\Applications\\Altium\\Datasheets\\IND0603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 -> (none)
- R186, R187, R85, R86, R87, R88, R89, R90: HelpURL \\\\cern.ch\\dfs\\Applications\\Altium\\Datasheets\\R0402_P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 -> (none)
Changed lines of the file:
@@
 F 33 "232270591001L" H 7750 670 60  0001 L CNN "Manufacturer1 Part Number"
 F 34 "0.4mm" H 7750 580 60  0001 L CNN "Manufacturer1 ComponentHeight"
-F 35 "\\\\cern.ch\\dfs\\Applications\\Altium\\Datasheets\\R0402_Phycomp_RC0402.pdf" H 7750 490 60  0001 L CNN "HelpURL"
 F 36 "CERN DEM JLC" H 7750 400 60  0001 L CNN "Author"
 F 37 "12/03/07 00:00:00" H 7750 310 60  0001 L CNN "CreateDate"
@@
 F 33 "232270671003L" H 7450 -530 60  0001 L CNN "Manufacturer1 Part Number"
 F 34 "0.4mm" H 7450 -620 60  0001 L CNN "Manufacturer1 ComponentHeight"
-F 35 "\\\\cern.ch\\dfs\\Applications\\Altium\\Datasheets\\R0402_Phycomp_RC0402.pdf" H 7450 -710 60  0001 L CNN "HelpURL"
 F 36 "CERN DEM JLC" H 7450 -800 60  0001 L CNN "Author"
 F 37 "12/03/07 00:00:00" H 7450 -890 60  0001 L CNN "CreateDate"
@@
 F 33 "232270671003L" H 7700 -530 60  0001 L CNN "Manufacturer1 Part Number"
 F 34 "0.4mm" H 7700 -620 60  0001 L CNN "Manufacturer1 ComponentHeight"
-F 35 "\\\\cern.ch\\dfs\\Applications\\Altium\\Datasheets\\R0402_Phycomp_RC0402.pdf" H 7700 -710 60  0001 L CNN "HelpURL"
 F 36 "CERN DEM JLC" H 7700 -800 60  0001 L CNN "Author"
 F 37 "12/03/07 00:00:00" H 7700 -890 60  0001 L CNN "CreateDate"
@@
 F 32 "02016D104KAT2A" H 1150 -1190 60  0001 L CNN "Manufacturer1 Part Number"
 F 33 "0.33mm" H 1150 -1280 60  0001 L CNN "Manufacturer1 ComponentHeight"
-F 34 "\\\\cern.ch\\dfs\\Applications\\Altium\\Datasheets\\CC0201_X5R_AVX.pdf" H 1150 -1370 60  0001 L CNN "HelpURL"
 F 35 "CERN DEM JLC" H 1150 -1460 60  0001 L CNN "Author"
 F 36 "12/03/07 00:00:00" H 1150 -1550 60  0001 L CNN "CreateDate"
@@
 F 32 "02016D104KAT2A" H 3100 -1190 60  0001 L CNN "Manufacturer1 Part Number"
 F 33 "0.33mm" H 3100 -1280 60  0001 L CNN "Manufacturer1 ComponentHeight"
-F 34 "\\\\cern.ch\\dfs\\Applications\\Altium\\Datasheets\\CC0201_X5R_AVX.pdf" H 3100 -1370 60  0001 L CNN "HelpURL"
 F 35 "CERN DEM JLC" H 3100 -1460 60  0001 L CNN "Author"
 F 36 "12/03/07 00:00:00" H 3100 -1550 60  0001 L CNN "CreateDate"
@@
 F 32 "02016D104KAT2A" H 3500 -1190 60  0001 L CNN "Manufacturer1 Part Number"
 F 33 "0.33mm" H 3500 -1280 60  0001 L CNN "Manufacturer1 ComponentHeight"
-F 34 "\\\\cern.ch\\dfs\\Applications\\Altium\\Datasheets\\CC0201_X5R_AVX.pdf" H 3500 -1370 60  0001 L CNN "HelpURL"
 F 35 "CERN DEM JLC" H 3500 -1460 60  0001 L CNN "Author"
 F 36 "12/03/07 00:00:00" H 3500 -1550 60  0001 L CNN "CreateDate"
@@
 F 32 "02016D104KAT2A" H 3850 -190 60  0001 L CNN "Manufacturer1 Part Number"
 F 33 "0.33mm" H 3850 -280 60  0001 L CNN "Manufacturer1 ComponentHeight"
-F 34 "\\\\cern.ch\\dfs\\Applications\\Altium\\Datasheets\\CC0201_X5R_AVX.pdf" H 3850 -370 60  0001 L CNN "HelpURL"
 F 35 "CERN DEM JLC" H 3850 -460 60  0001 L CNN "Author"
 F 36 "12/03/07 00:00:00" H 3850 -550 60  0001 L CNN "CreateDate"
@@
 F 28 " " H 1850 -760 60  0001 L CNN "Status Comment"
 F 29 "0.65mm" H 1850 -850 60  0001 L CNN "ComponentHeight"
-F 30 "\\\\cern.ch\\dfs\\Applications\\Altium\\Datasheets\\IND0603_MURATA_BLM18S.pdf" H 1850 -940 60  0001 L CNN "HelpURL"
 F 31 "CERN DEM JLC" H 1850 -1030 60  0001 L CNN "Author"
 F 32 "07/23/14 00:00:00" H 1850 -1120 60  0001 L CNN "CreateDate"
@@
 F 28 " " H 3100 240 60  0001 L CNN "Status Comment"
 F 29 "0.65mm" H 3100 150 60  0001 L CNN "ComponentHeight"
-F 30 "\\\\cern.ch\\dfs\\Applications\\Altium\\Datasheets\\IND0603_MURATA_BLM18S.pdf" H 3100 60  60  0001 L CNN "HelpURL"
 F 31 "CERN DEM JLC" H 3100 -30 60  0001 L CNN "Author"
 F 32 "07/23/14 00:00:00" H 3100 -120 60  0001 L CNN "CreateDate"
@@
 F 32 "C1005X5R1C105KT" H 1600 -1190 60  0001 L CNN "Manufacturer1 Part Number"
 F 33 "0.55mm" H 1600 -1280 60  0001 L CNN "Manufacturer1 ComponentHeight"
-F 34 "\\\\cern.ch\\dfs\\Applications\\Altium\\Datasheets\\CC0402_X5R_TDK_C.pdf" H 1600 -1370 60  0001 L CNN "HelpURL"
 F 35 "CERN DEM JLC" H 1600 -1460 60  0001 L CNN "Author"
 F 36 "10/25/12 00:00:00" H 1600 -1550 60  0001 L CNN "CreateDate"
@@
 F 32 "C1005X5R1C105KT" H 2700 -1190 60  0001 L CNN "Manufacturer1 Part Number"
 F 33 "0.55mm" H 2700 -1280 60  0001 L CNN "Manufacturer1 ComponentHeight"
-F 34 "\\\\cern.ch\\dfs\\Applications\\Altium\\Datasheets\\CC0402_X5R_TDK_C.pdf" H 2700 -1370 60  0001 L CNN "HelpURL"
 F 35 "CERN DEM JLC" H 2700 -1460 60  0001 L CNN "Author"
 F 36 "10/25/12 00:00:00" H 2700 -1550 60  0001 L CNN "CreateDate"
@@
 F 32 "C0603C106M9PAC" H 2300 -890 60  0001 L CNN "Manufacturer1 Part Number"
 F 33 "0.95mm" H 2300 -980 60  0001 L CNN "Manufacturer1 ComponentHeight"
-F 34 "\\\\cern.ch\\dfs\\Applications\\Altium\\Datasheets\\CC0603_X5R_KEMET.pdf" H 2300 -1070 60  0001 L CNN "HelpURL"
 F 35 "CERN DEM JLC" H 2300 -1160 60  0001 L CNN "Author"
 F 36 "12/03/07 00:00:00" H 2300 -1250 60  0001 L CNN "CreateDate"
@@
 F 32 "C0603C106M9PAC" H 3450 110 60  0001 L CNN "Manufacturer1 Part Number"
 F 33 "0.95mm" H 3450 20  60  0001 L CNN "Manufacturer1 ComponentHeight"
-F 34 "\\\\cern.ch\\dfs\\Applications\\Altium\\Datasheets\\CC0603_X5R_KEMET.pdf" H 3450 -70 60  0001 L CNN "HelpURL"
 F 35 "CERN DEM JLC" H 3450 -160 60  0001 L CNN "Author"
 F 36 "12/03/07 00:00:00" H 3450 -250 60  0001 L CNN "CreateDate"
@@
 F 33 "232270671003L" H 7200 -530 60  0001 L CNN "Manufacturer1 Part Number"
 F 34 "0.4mm" H 7200 -620 60  0001 L CNN "Manufacturer1 ComponentHeight"
-F 35 "\\\\cern.ch\\dfs\\Applications\\Altium\\Datasheets\\R0402_Phycomp_RC0402.pdf" H 7200 -710 60  0001 L CNN "HelpURL"
 F 36 "CERN DEM JLC" H 7200 -800 60  0001 L CNN "Author"
 F 37 "12/03/07 00:00:00" H 7200 -890 60  0001 L CNN "CreateDate"
@@
 F 33 "232270671003L" H 6950 -530 60  0001 L CNN "Manufacturer1 Part Number"
 F 34 "0.4mm" H 6950 -620 60  0001 L CNN "Manufacturer1 ComponentHeight"
-F 35 "\\\\cern.ch\\dfs\\Applications\\Altium\\Datasheets\\R0402_Phycomp_RC0402.pdf" H 6950 -710 60  0001 L CNN "HelpURL"
 F 36 "CERN DEM JLC" H 6950 -800 60  0001 L CNN "Author"
 F 37 "12/03/07 00:00:00" H 6950 -890 60  0001 L CNN "CreateDate"
@@
 F 33 "232270671003L" H 6700 -530 60  0001 L CNN "Manufacturer1 Part Number"
 F 34 "0.4mm" H 6700 -620 60  0001 L CNN "Manufacturer1 ComponentHeight"
-F 35 "\\\\cern.ch\\dfs\\Applications\\Altium\\Datasheets\\R0402_Phycomp_RC0402.pdf" H 6700 -710 60  0001 L CNN "HelpURL"
 F 36 "CERN DEM JLC" H 6700 -800 60  0001 L CNN "Author"
 F 37 "12/03/07 00:00:00" H 6700 -890 60  0001 L CNN "CreateDate"
@@
 F 33 "232270671003L" H 6100 720 60  0001 L CNN "Manufacturer1 Part Number"
 F 34 "0.4mm" H 6100 630 60  0001 L CNN "Manufacturer1 ComponentHeight"
-F 35 "\\\\cern.ch\\dfs\\Applications\\Altium\\Datasheets\\R0402_Phycomp_RC0402.pdf" H 6100 540 60  0001 L CNN "HelpURL"
 F 36 "CERN DEM JLC" H 6100 450 60  0001 L CNN "Author"
 F 37 "12/03/07 00:00:00" H 6100 360 60  0001 L CNN "CreateDate"
@@
 F 33 "232270591001L" H 6250 720 60  0001 L CNN "Manufacturer1 Part Number"
 F 34 "0.4mm" H 6250 630 60  0001 L CNN "Manufacturer1 ComponentHeight"
-F 35 "\\\\cern.ch\\dfs\\Applications\\Altium\\Datasheets\\R0402_Phycomp_RC0402.pdf" H 6250 540 60  0001 L CNN "HelpURL"
 F 36 "CERN DEM JLC" H 6250 450 60  0001 L CNN "Author"
 F 37 "12/03/07 00:00:00" H 6250 360 60  0001 L CNN "CreateDate"
@@
 F 29 "1888247-1" H 4500 -2660 60  0001 L CNN "Manufacturer Part Number"
 F 30 "5.4mm" H 4500 -2750 60  0001 L CNN "ComponentHeight"
-F 31 " " H 4500 -2840 60  0001 L CNN "ComponentLink1URL"
 F 32 " " H 4500 -2930 60  0001 L CNN "ComponentLink1Description"
-F 33 " " H 4500 -3020 60  0001 L CNN "ComponentLink2URL"
 F 34 " " H 4500 -3110 60  0001 L CNN "ComponentLink2Description"
-F 35 "\\\\cern.ch\\dfs\\Applications\\Altium\\Datasheets\\TYCO_1888247-1.pdf" H 4500 -3200 60  0001 L CNN "HelpURL"
 F 36 "CERN DEM JLC" H 4500 -3290 60  0001 L CNN "Author"
 F 37 "02/27/12 00:00:00" H 4500 -3380 60  0001 L CNN "CreateDate"

Commit message: Trash "Footprint Library" and "Database Table Name" attributes
Takes 100 attributes out of schematic, 174 out of library
Parts:
- J8: Database Table Name TYCO -> (none); Footprint Library TYCO SMD -> (none)
- R187: Database Table Name Resistors SMD -> (none); Footprint Library Resistors SMD -> (none)
Changed lines of the file:
@@
 F 39 "Resistors SMD" H 7750 130 60  0001 L CNN "Library Name"
 F 40 "This work is licensed under the Creative Commons CC-BY-SA 4.0 License. To the extent that circuit schematics that use Licensed Material can be considered to be ‘Adapted Material’, then the copyright holder waives article 3.b of the license with respect to these schematics." H 7750 40  60  0001 L CNN "License"
-F 41 "Resistors SMD" H 7750 3850 50  0001 C CNN "Database Table Name"
-F 42 "Resistors SMD" H 7750 3850 50  0001 C CNN "Footprint Library"
 F 43 "dnf" V 7950 4100 50  0000 C CNN "config"
 	1    7750 3850
@@
 F 39 "Connectors.DbLib" H 4500 -3560 60  0001 L CNN "Library Name"
 F 40 "This work is licensed under the Creative Commons CC-BY-SA 4.0 License. To the extent that circuit schematics that use Licensed Material can be considered to be ‘Adapted Material’, then the copyright holder waives article 3.b of the license with respect to these schematics." H 4500 -3650 60  0001 L CNN "License"
-F 41 "TYCO" H 4500 1850 50  0001 C CNN "Database Table Name"
-F 42 "TYCO SMD" H 4500 1850 50  0001 C CNN "Footprint Library"
 	1    4500 1850
 	1    0    0    -1

Commit message: Trash SCEM attribute
Parts:
- J8: SCEM (none) -> (none)
Changed lines of the file:
@@
 F 23 "None" H 4500 -2120 60  0001 L CNN "Status"
 F 24 " " H 4500 -2210 60  0001 L CNN "Status Comment"
-F 25 " " H 4500 -2300 60  0001 L CNN "SCEM"
 F 26 " " H 4500 -2390 60  0001 L CNN "Device"
 F 27 "20 Position, Pitch 0.8mm SFP+ Receptacle (Small Form-factor Pluggable)" H 4500 -2480 60  0001 L CNN "Part Description"
