File: FPGA_34_35.sch (KiCad schematic (older format))
At the start: 1 part, among them U1 XC7A100T-2FGG484C

Commit message: Rename library AMC_FMC_Carrier-PcbDoc-rescue as marble_misc
Parts:
- U1: symbol AMC_FMC_Carrier-PcbDoc-rescue:XC7A200T-FBG484-FPGA_Xilinx_Artix7-AMC_FMC_Carrier-PcbDoc-rescue -> marble_misc:XC7A200T-FBG484-FPGA_Xilinx_Artix7-AMC_FMC_Carrier-PcbDoc-rescue
Changed lines of the file:
@@
 $EndDescr
 $Comp
-L AMC_FMC_Carrier-PcbDoc-rescue:XC7A200T-FBG484-FPGA_Xilinx_Artix7-AMC_FMC_Carrier-PcbDoc-rescue U?
+L marble_misc:XC7A200T-FBG484-FPGA_Xilinx_Artix7-AMC_FMC_Carrier-PcbDoc-rescue U?
 U 3 1 5C8DFB5E
 P 8350 4650

Commit message: Strip extraneous AMC_FMC_Carrier-PcbDoc-rescue and powerMG from symbol names
Parts:
- U1: symbol marble_misc:XC7A200T-FBG484-FPGA_Xilinx_Artix7-AMC_FMC_Carrier-PcbDoc-rescue -> marble_misc:XC7A200T-FBG484-FPGA_Xilinx_Artix7
Changed lines of the file:
@@
 $EndDescr
 $Comp
-L marble_misc:XC7A200T-FBG484-FPGA_Xilinx_Artix7-AMC_FMC_Carrier-PcbDoc-rescue U?
+L marble_misc:XC7A200T-FBG484-FPGA_Xilinx_Artix7 U?
 U 3 1 5C8DFB5E
 P 8350 4650

Commit message: Convert all footprints to use Marble nickname
Includes both .sch and .lib files
Includes both bare footprint names and those with CERN-like nicknames
Parts:
- U1: footprint ICs And Semiconductors SMD_BGA:BGA484C100P22X22_2300X2300X240 -> Marble:BGA484C100P22X22_2300X2300X240
Changed lines of the file:
@@
 F 0 "U1" H 8350 1676 50  0000 C CNN
 F 1 "XC7A100T-2FGG484C" H 8350 1585 50  0000 C CNN
-F 2 "ICs And Semiconductors SMD_BGA:BGA484C100P22X22_2300X2300X240" H 8350 4650 50  0001 C CNN
+F 2 "Marble:BGA484C100P22X22_2300X2300X240" H 8350 4650 50  0001 C CNN
 F 3 "" H 8350 4650 50  0000 C CNN
 F 4 "XC7A100T-2FGG484C" H 8350 4650 50  0001 C CNN "Manufacturer Part Number"

Commit message: Start filling in more Manufacturer fields
Parts:
- U1: Manufacturer (none) -> Xilinx
Changed lines of the file:
@@
 F 3 "" H 8350 4650 50  0000 C CNN
 F 4 "XC7A100T-2FGG484C" H 8350 4650 50  0001 C CNN "Manufacturer Part Number"
+F 5 "Xilinx" H 8350 4650 50  0001 C CNN "Manufacturer"
 	3    8350 4650
 	1    0    0    -1
